File: Hardware/MCU.kicad_sch (KiCad schematic)
At the start: 25 parts, among them SW301 RESET, U301 STM32F722ZETx, Y301 24MHz

Commit message: Checkpoint
Parts:
- C303, C304: value 4.7uF -> 2.2uF; footprint (none) -> Capacitor_SMD:C_0805_2012Metric
- C305, C306, C307, C308, C309, C310, C311, C312, C313, C314, C315, C316, C318, C319: footprint (none) -> Capacitor_SMD:C_0603_1608Metric
- C317: footprint (none) -> Capacitor_SMD:C_1206_3216Metric
- C320, C321: footprint (none) -> Capacitor_SMD:C_0805_2012Metric
- R301: footprint (none) -> Resistor_SMD:R_0603_1608Metric
Changed lines of the file:
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@@
       (effects (font (size 1.27 1.27)) (justify left))
     )
-    (property "Footprint" "" (at 307.34 139.7 0)
+    (property "Footprint" "Capacitor_SMD:C_0603_1608Metric" (at 307.34 139.7 0)
       (effects (font (size 1.27 1.27)) hide)
     )
@@
       (effects (font (size 1.27 1.27)))
     )
-    (property "Footprint" "" (at 360.68 246.38 0)
+    (property "Footprint" "Capacitor_SMD:C_0603_1608Metric" (at 360.68 246.38 0)
       (effects (font (size 1.27 1.27)) hide)
     )
@@
       (effects (font (size 1.27 1.27)) (justify left))
     )
-    (property "Footprint" "" (at 368.3 83.82 0)
+    (property "Footprint" "Capacitor_SMD:C_0805_2012Metric" (at 368.3 83.82 0)
       (effects (font (size 1.27 1.27)) hide)
     )
@@
       (effects (font (size 1.27 1.27)) (justify left))
     )
-    (property "Footprint" "" (at 320.04 111.76 0)
+    (property "Footprint" "Capacitor_SMD:C_0603_1608Metric" (at 320.04 111.76 0)
       (effects (font (size 1.27 1.27)) hide)
     )
@@
       (effects (font (size 1.27 1.27)) (justify left))
     )
-    (property "Footprint" "" (at 307.34 111.76 0)
+    (property "Footprint" "Capacitor_SMD:C_0603_1608Metric" (at 307.34 111.76 0)
       (effects (font (size 1.27 1.27)) hide)
     )
@@
       (effects (font (size 1.27 1.27)) (justify left))
     )
-    (property "Footprint" "" (at 320.04 139.7 0)
+    (property "Footprint" "Capacitor_SMD:C_0603_1608Metric" (at 320.04 139.7 0)
       (effects (font (size 1.27 1.27)) hide)
     )
@@
       (effects (font (size 1.27 1.27)) (justify right))
     )
-    (property "Value" "4.7uF" (at 109.22 245.1036 0)
+    (property "Value" "2.2uF" (at 109.22 245.1036 0)
       (effects (font (size 1.27 1.27)) (justify right))
     )
-    (property "Footprint" "" (at 111.76 243.84 0)
+    (property "Footprint" "Capacitor_SMD:C_0805_2012Metric" (at 111.76 243.84 0)
       (effects (font (size 1.27 1.27)) hide)
     )
@@
       (effects (font (size 1.27 1.27)) (justify left))
     )
-    (property "Footprint" "" (at 294.64 111.76 0)
+    (property "Footprint" "Capacitor_SMD:C_0603_1608Metric" (at 294.64 111.76 0)
       (effects (font (size 1.27 1.27)) hide)
     )
@@
       (effects (font (size 1.27 1.27)) (justify left))
     )
-    (property "Footprint" "" (at 350.52 111.76 0)
+    (property "Footprint" "Capacitor_SMD:C_0603_1608Metric" (at 350.52 111.76 0)
       (effects (font (size 1.27 1.27)) hide)
     )
@@
       (effects (font (size 1.27 1.27)) (justify left))
     )
-    (property "Footprint" "" (at 350.52 83.82 0)
+    (property "Footprint" "Capacitor_SMD:C_1206_3216Metric" (at 350.52 83.82 0)
       (effects (font (size 1.27 1.27)) hide)
     )
@@
       (effects (font (size 1.27 1.27)) (justify left))
     )
-    (property "Footprint" "" (at 332.74 111.76 0)
+    (property "Footprint" "Capacitor_SMD:C_0603_1608Metric" (at 332.74 111.76 0)
       (effects (font (size 1.27 1.27)) hide)
     )
@@
       (effects (font (size 1.27 1.27)) (justify left))
     )
-    (property "Footprint" "" (at 332.74 139.7 0)
+    (property "Footprint" "Capacitor_SMD:C_0603_1608Metric" (at 332.74 139.7 0)
       (effects (font (size 1.27 1.27)) hide)
     )
@@
       (effects (font (size 1.27 1.27)) (justify left))
     )
-    (property "Footprint" "" (at 332.74 83.82 0)
+    (property "Footprint" "Capacitor_SMD:C_0603_1608Metric" (at 332.74 83.82 0)
       (effects (font (size 1.27 1.27)) hide)
     )
@@
       (effects (font (size 1.27 1.27)) (justify left))
     )
-    (property "Footprint" "" (at 320.04 83.82 0)
+    (property "Footprint" "Capacitor_SMD:C_0603_1608Metric" (at 320.04 83.82 0)
       (effects (font (size 1.27 1.27)) hide)
     )
@@
       (effects (font (size 1.27 1.27)) (justify right))
     )
-    (property "Value" "4.7uF" (at 119.38 245.1036 0)
+    (property "Value" "2.2uF" (at 119.38 245.1036 0)
       (effects (font (size 1.27 1.27)) (justify right))
     )
-    (property "Footprint" "" (at 116.84 243.84 0)
+    (property "Footprint" "Capacitor_SMD:C_0805_2012Metric" (at 116.84 243.84 0)
       (effects (font (size 1.27 1.27)) hide)
     )
@@
       (effects (font (size 1.27 1.27)) (justify left))
     )
-    (property "Footprint" "" (at 294.64 139.7 0)
+    (property "Footprint" "Capacitor_SMD:C_0603_1608Metric" (at 294.64 139.7 0)
       (effects (font (size 1.27 1.27)) hide)
     )
@@
       (effects (font (size 1.27 1.27)))
     )
-    (property "Footprint" "" (at 391.16 246.38 0)
+    (property "Footprint" "Resistor_SMD:R_0603_1608Metric" (at 391.16 246.38 0)
       (effects (font (size 1.27 1.27)) hide)
     )
@@
       (effects (font (size 1.27 1.27)) (justify left))
     )
-    (property "Footprint" "" (at 294.64 83.82 0)
+    (property "Footprint" "Capacitor_SMD:C_0603_1608Metric" (at 294.64 83.82 0)
       (effects (font (size 1.27 1.27)) hide)
     )
@@
       (effects (font (size 1.27 1.27)) (justify left))
     )
-    (property "Footprint" "" (at 307.34 83.82 0)
+    (property "Footprint" "Capacitor_SMD:C_0603_1608Metric" (at 307.34 83.82 0)
       (effects (font (size 1.27 1.27)) hide)
     )
@@
       (effects (font (size 1.27 1.27)) (justify left))
     )
-    (property "Footprint" "" (at 363.22 111.76 0)
-      (effects (font (size 1.27 1.27)) hide)
-    )
+    (property "Footprint" "Capacitor_SMD:C_0805_2012Metric" (at 363.22 111.76 0)
+      (effects (font (size 1.27 1.27)) hide)
+    )
