File: Hardware/MCU.kicad_sch (KiCad schematic)
At the start: 25 parts, among them SW301 RESET, U301 STM32F722ZETx, Y301 24MHz

Commit message: Checkpoint
Connections:
- net GPIO_PD1: now reaches U301.115 (PD1)
- net GPIO_PF14: now reaches U301.54 (PF14)
- net GPIO_PF15: now reaches U301.55 (PF15)
- net GPIO_PG0: now reaches U301.56 (PG0)
- net GPIO_PG1: now reaches U301.57 (PG1)
- no-connect marks 31 -> 26
Changed lines of the file:
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@@
   (junction (at 101.6 99.06) (diameter 0) (color 0 0 0 0)
   )
-  (no_connect (at 121.92 182.88))
-  (no_connect (at 121.92 104.14))
   (no_connect (at 121.92 180.34))
   (no_connect (at 121.92 177.8))
-  (no_connect (at 121.92 185.42))
-  (no_connect (at 121.92 119.38))
   (no_connect (at 182.88 109.22))
-  (no_connect (at 121.92 124.46))
   (no_connect (at 182.88 91.44))
-  (no_connect (at 182.88 210.82))
   (no_connect (at 182.88 134.62))
   (no_connect (at 121.92 175.26))
@@
   (no_connect (at 182.88 81.28))
   (no_connect (at 121.92 220.98))
+  (no_connect (at 121.92 121.92))
   (no_connect (at 182.88 236.22))
   (no_connect (at 121.92 218.44))
-  (no_connect (at 121.92 106.68))
-  (no_connect (at 121.92 121.92))
+  (no_connect (at 121.92 119.38))
   (no_connect (at 182.88 93.98))
   (no_connect (at 182.88 215.9))
   (no_connect (at 182.88 139.7))
   (no_connect (at 182.88 121.92))
+  (no_connect (at 121.92 124.46))
   (no_connect (at 182.88 233.68))
   (no_connect (at 182.88 96.52))
@@
     (effects (font (size 1.27 1.27)) (justify left))
   )
+  (hierarchical_label "GPIO_PF15" (shape output) (at 121.92 185.42 180) (fields_autoplaced)
+    (effects (font (size 1.27 1.27)) (justify right))
+  )
+  (hierarchical_label "GPIO_PG0" (shape output) (at 121.92 104.14 180) (fields_autoplaced)
+    (effects (font (size 1.27 1.27)) (justify right))
+  )
   (hierarchical_label "QUADSPI_BK1_IO[0..3]" (shape bidirectional) (at 381 25.4 0) (fields_autoplaced)
     (effects (font (size 1.27 1.27)) (justify left))
@@
     (effects (font (size 1.27 1.27)) (justify left))
   )
+  (hierarchical_label "GPIO_PG1" (shape output) (at 121.92 106.68 180) (fields_autoplaced)
+    (effects (font (size 1.27 1.27)) (justify right))
+  )
   (hierarchical_label "QUADSPI_CLK" (shape output) (at 182.88 127 0) (fields_autoplaced)
     (effects (font (size 1.27 1.27)) (justify left))
   )
+  (hierarchical_label "GPIO_PF14" (shape input) (at 121.92 182.88 180) (fields_autoplaced)
+    (effects (font (size 1.27 1.27)) (justify right))
+  )
   (hierarchical_label "VDD" (shape passive) (at 294.64 132.08 90) (fields_autoplaced)
     (effects (font (size 1.27 1.27)) (justify left))
@@
     (effects (font (size 1.27 1.27)) (justify right))
   )
+  (hierarchical_label "GPIO_PD1" (shape output) (at 182.88 210.82 0) (fields_autoplaced)
+    (effects (font (size 1.27 1.27)) (justify left))
+  )
   (hierarchical_label "GPIO_PA0+EXTI0+TIM2_CH1+TIM2_ETR+TIM5_CH1" (shape bidirectional) (at 182.88 78.74 0) (fields_autoplaced)

Commit message: Checkpoint
Parts:
- SW301: footprint (none) -> Button_Switch_THT:SW_PUSH_6mm_H5mm
Changed lines of the file:
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@@
       (effects (font (size 1.27 1.27)))
     )
-    (property "Footprint" "" (at 360.68 231.14 0)
+    (property "Footprint" "Button_Switch_THT:SW_PUSH_6mm_H5mm" (at 360.68 231.14 0)
       (effects (font (size 1.27 1.27)) hide)
     )

Commit message: Checkpoint
Parts:
- added NT301: LOOP, symbol Device:NetTie_2
Connections:
- net SPI4_MISO: now also U301.66 (PE13); no longer U301.4 (PE5)
- net SPI4_MOSI: now also U301.67 (PE14); no longer U301.5 (PE6)
- net SPI4_SCK: now also U301.65 (PE12); no longer U301.1 (PE2)
- net TIM9_CH2: now also U301.5 (PE6); no longer U301.37 (PA3)
- net GPIO_PD3+EXTI3: now reaches U301.117 (PD3)
- net GPIO_PG15: now reaches U301.132 (PG15)
- net TIM2_CH2: now reaches U301.35 (PA1)
- net SPI1_SCK: now reaches U301.41 (PA5)
- net SPI1_MISO: now reaches U301.42 (PA6)
- net SPI1_MOSI: now reaches U301.43 (PA7)
- net ADC1_IN8: now reaches U301.46 (PB0)
- net ADC1_IN9: now reaches U301.47 (PB1)
- net GPIO_PF11: now reaches U301.49 (PF11)
- net GPIO_PF12: now reaches U301.50 (PF12)
- net GPIO_PF13: now reaches U301.53 (PF13)
- net GPIO_PE11: now reaches U301.64 (PE11)
- net GPIO_PB12+EXTI12: now reaches U301.73 (PB12)
- net GPIO_PD10: now reaches U301.79 (PD10)
- net GPIO_PD11: now reaches U301.80 (PD11)
- net GPIO_PG6+EXTI6: now reaches U301.91 (PG6)
- net ADC1_IN10 renamed ADC2_IN10
- net GPIO_PA0+EXTI0+TIM2_CH1+TIM2_ETR+TIM5_CH1 renamed TIM2_CH1
- net GPIO_PA2+EXTI2+TIM2_CH2+TIM5_CH3+USART2_TX renamed TIM2_CH3
- net GPIO_PC1+EXTI1 renamed ADC2_IN11
- net GPIO_PC14+EXTI14: no longer names the net of U301.8 (PC14)
- net GPIO_PC14+EXTI14: now also NT301.2
- net GPIO_PC15+EXTI15: no longer names the net of U301.9 (PC15)
- net GPIO_PC15+EXTI15: now also NT301.1
- net GPIO_PD5+EXTI5: no longer names the net of U301.119 (PD5)
- net GPIO_PE15 renamed GPIO_PE15+EXTI15
- net GPIO_PE3+EXTI3 renamed GPIO_PE3
- net GPIO_PF2 renamed GPIO_PF2+EXTI2
- net GPIO_PG1 renamed GPIO_PG1+EXTI1
- net GPIO_PG13 renamed GPIO_PG13+EXTI13
- net GPIO_PG2: no longer names the net of U301.87 (PG2)
- net GPIO_PG3: no longer names the net of U301.88 (PG3)
- net SPI2_MISO renamed ADC2_IN12
- net SPI2_MOSI renamed ADC2_IN13
- net SPI2_SCK renamed GPIO_PB10+EXTI10
- net UART8_RX renamed UART8_RX+EXTI0
- net USART3_RX+EXTI9 renamed USART3_RX
- new net GPIO_PE5+EXTI5: U301.4 (PE5)
- new net TIM2_CH4: U301.37 (PA3)
- no-connect marks 26 -> 11

Commit message: Checkpoint
Parts:
- removed NT301: LOOP, symbol Device:NetTie_2
- added R?: 2.2K, Resistor_SMD:R_0805_2012Metric, symbol Device:R_Small
- renumbered R301 to R302
Connections:
- net at U301.9 (PC15): now also R?.2
- net LOOP: now reaches U301.8 (PC14)
- net LOOP: now also R?.1
Changed lines of the file:
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@@
+    (stroke (width 0) (type default))
+  )
+  (wire (pts (xy 203.2 203.2) (xy 205.74 203.2))
     (stroke (width 0) (type default))
   )
@@
     (stroke (width 0) (type default))
   )
+  (wire (pts (xy 182.88 203.2) (xy 198.12 203.2))
+    (stroke (width 0) (type default))
+  )
   (wire (pts (xy 147.32 68.58) (xy 147.32 71.12))
     (stroke (width 0) (type default))
@@
     (stroke (width 0) (type default))
   )
-  (wire (pts (xy 195.58 200.66) (xy 195.58 198.12))
-    (stroke (width 0) (type default))
-  )
   (wire (pts (xy 111.76 248.92) (xy 111.76 246.38))
     (stroke (width 0) (type default))
@@
     (stroke (width 0) (type default))
   )
+  (wire (pts (xy 182.88 200.66) (xy 205.74 200.66))
+    (stroke (width 0) (type default))
+  )
   (wire (pts (xy 294.64 134.62) (xy 294.64 132.08))
     (stroke (width 0) (type default))
   )
-  (wire (pts (xy 182.88 200.66) (xy 195.58 200.66))
-    (stroke (width 0) (type default))
-  )
   (wire (pts (xy 350.52 76.2) (xy 350.52 81.28))
     (stroke (width 0) (type default))
@@
     (stroke (width 0) (type default))
   )
-  (wire (pts (xy 195.58 198.12) (xy 198.12 198.12))
-    (stroke (width 0) (type default))
-  )
   (wire (pts (xy 142.24 68.58) (xy 144.78 68.58))
     (stroke (width 0) (type default))
@@
     (stroke (width 0) (type default))
   )
-  (wire (pts (xy 182.88 203.2) (xy 198.12 203.2))
-    (stroke (width 0) (type default))
-  )
   (wire (pts (xy 294.64 88.9) (xy 307.34 88.9))
     (stroke (width 0) (type default))
@@
     (stroke (width 0) (type default))
   )
+  (wire (pts (xy 205.74 200.66) (xy 205.74 203.2))
+    (stroke (width 0) (type default))
+  )
   (text "VDDSDMMC" (at 365.76 83.82 90)
     (effects (font (size 1.27 1.27)) (justify left bottom))
@@
   (label "QUADSPI_BK1_IO[0..3]" (at 330.2 25.4 0) (fields_autoplaced)
     (effects (font (size 1.27 1.27)) (justify left bottom))
+  )
+  (label "LOOP" (at 203.2 200.66 180) (fields_autoplaced)
+    (effects (font (size 1.27 1.27)) (justify right bottom))
   )
   (label "QUADSPI_BK1_IO3" (at 76.2 162.56 0) (fields_autoplaced)
@@
     )
   )
+  (symbol (lib_id "Device:R_Small") (at 200.66 203.2 270) (mirror x) (unit 1)
+    (in_bom yes) (on_board yes) (dnp no)
+    (property "Reference" "R?" (at 200.66 208.28 90)
+      (effects (font (size 1.27 1.27)))
+    )
+    (property "Value" "2.2K" (at 200.66 205.74 90)
+      (effects (font (size 1.27 1.27)))
+    )
+    (property "Footprint" "Resistor_SMD:R_0805_2012Metric" (at 200.66 203.2 0)
+      (effects (font (size 1.27 1.27)) hide)
+    )
+    (property "Datasheet" "~" (at 200.66 203.2 0)
+      (effects (font (size 1.27 1.27)) hide)
+    )
+    (pin "1")
+    (pin "2")
+    (instances
+      (project "Avionus_Flight_Controller"
+        (path "/ddc7e940-0588-4587-8902-8ced9e615ace/07011d92-7eb9-4cfe-9164-8ccacd4ef57f"
+          (reference "R?") (unit 1)
+        )
+        (path "/ddc7e940-0588-4587-8902-8ced9e615ace/fb82246b-9ed4-401c-b8a1-7e9ae6260bc5"
+          (reference "R301") (unit 1)
+        )
+      )
+    )
+  )
   (symbol (lib_id "Device:Crystal_Small") (at 101.6 93.98 90) (unit 1)
     (in_bom yes) (on_board yes) (dnp no) (fields_autoplaced)
@@
         (path "/ddc7e940-0588-4587-8902-8ced9e615ace/fb82246b-9ed4-401c-b8a1-7e9ae6260bc5"
           (reference "Y301") (unit 1)
-        )
-      )
-    )
-  )
-  (symbol (lib_id "Device:NetTie_2") (at 198.12 200.66 90) (unit 1)
-    (in_bom no) (on_board yes) (dnp no) (fields_autoplaced)
-    (property "Reference" "NT301" (at 199.39 199.39 90)
-      (effects (font (size 1.27 1.27)) (justify right))
-    )
-    (property "Value" "LOOP" (at 199.39 201.93 90)
-      (effects (font (size 1.27 1.27)) (justify right))
-    )
-    (property "Footprint" "" (at 198.12 200.66 0)
-      (effects (font (size 1.27 1.27)) hide)
-    )
-    (property "Datasheet" "~" (at 198.12 200.66 0)
-      (effects (font (size 1.27 1.27)) hide)
-    )
-    (pin "1")
-    (pin "2")
-    (instances
-      (project "Avionus_Flight_Controller"
-        (path "/ddc7e940-0588-4587-8902-8ced9e615ace/fb82246b-9ed4-401c-b8a1-7e9ae6260bc5"
-          (reference "NT301") (unit 1)
         )
       )
@@
   (symbol (lib_id "Device:R_Small") (at 391.16 246.38 270) (unit 1)
     (in_bom yes) (on_board yes) (dnp no) (fields_autoplaced)
-    (property "Reference" "R301" (at 391.16 241.3 90)
+    (property "Reference" "R302" (at 391.16 241.3 90)
       (effects (font (size 1.27 1.27)))
     )
@@
       (project "Avionus_Flight_Controller"
         (path "/ddc7e940-0588-4587-8902-8ced9e615ace/fb82246b-9ed4-401c-b8a1-7e9ae6260bc5"
-          (reference "R301") (unit 1)
-        )
-      )
+          (reference "R302") (unit 1)
+        )
+      )

Commit message: Checkpoint
Connections:
- net GPIO_PA12: now reaches U301.104 (PA12)
- net ADC1_IN8: no longer names the net of U301.46 (PB0)
- net ADC1_IN9: no longer names the net of U301.47 (PB1)
- no-connect marks 11 -> 12
Changed lines of the file:
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@@
   (no_connect (at 121.92 109.22))
   (no_connect (at 182.88 134.62))
-  (no_connect (at 182.88 109.22))
   (no_connect (at 121.92 111.76))
+  (no_connect (at 182.88 124.46))
+  (no_connect (at 182.88 121.92))
   (no_connect (at 182.88 139.7))
   (no_connect (at 121.92 121.92))
@@
     (effects (font (size 1.27 1.27)) (justify left))
   )
-  (hierarchical_label "ADC1_IN9" (shape input) (at 182.88 124.46 0) (fields_autoplaced)
-    (effects (font (size 1.27 1.27)) (justify left))
-  )
   (hierarchical_label "SPI4_SCK" (shape output) (at 121.92 220.98 180) (fields_autoplaced)
     (effects (font (size 1.27 1.27)) (justify right))
@@
     (effects (font (size 1.27 1.27)) (justify left))
   )
-  (hierarchical_label "ADC1_IN8" (shape input) (at 182.88 121.92 0) (fields_autoplaced)
-    (effects (font (size 1.27 1.27)) (justify left))
-  )
   (hierarchical_label "SDMMC2_D[0..3]" (shape bidirectional) (at 381 38.1 0) (fields_autoplaced)
     (effects (font (size 1.27 1.27)) (justify left))
@@
     (effects (font (size 1.27 1.27)) (justify left))
   )
+  (hierarchical_label "GPIO_PA12" (shape input) (at 182.88 109.22 0) (fields_autoplaced)
+    (effects (font (size 1.27 1.27)) (justify left))
+  )

Commit message: Checkpoint
Parts:
- added TP301, TP302, TP303, TP304, TP305, TP306, TP307, TP308, TP309, TP310, TP311, TP312: ~, TestPoint:TestPoint_Pad_D1.0mm, symbol Connector:TestPoint
Connections:
- net at U301.1 (PE2): now also TP305.1
- net at U301.119 (PD5): now also TP312.1
- net at U301.134 (PB4): now also TP308.1
- net at U301.135 (PB5): now also TP309.1
- net at U301.137 (PB7): now also TP310.1
- net at U301.139 (PB8): now also TP311.1
- net at U301.46 (PB0): now also TP306.1
- net at U301.47 (PB1): now also TP307.1
- net at U301.87 (PG2): now also TP301.1
- net at U301.88 (PG3): now also TP302.1
- net at U301.92 (PG7): now also TP303.1
- net at U301.93 (PG8): now also TP304.1
- no-connect marks 12 -> 0

Commit message: Misc routing
Parts:
- removed R?: 2.2K, Resistor_SMD:R_0805_2012Metric, symbol Device:R_Small
- added R301, R303: 10K, Resistor_SMD:R_0603_1608Metric, symbol Device:R_Small
Connections:
- net LOOP: now also R301.1, R303.1; no longer U301.8 (PC14)
- net at U301.9 (PC15): now also R303.2
- new net: R301.2, U301.8 (PC14)
Changed lines of the file:
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@@
-    (stroke (width 0) (type default))
-  )
-  (wire (pts (xy 182.88 200.66) (xy 205.74 200.66))
     (stroke (width 0) (type default))
   )
@@
     (stroke (width 0) (type default))
   )
+  (wire (pts (xy 182.88 200.66) (xy 198.12 200.66))
+    (stroke (width 0) (type default))
+  )
   (wire (pts (xy 294.64 88.9) (xy 294.64 91.44))
     (stroke (width 0) (type default))
@@
     (stroke (width 0) (type default))
   )
+  (wire (pts (xy 203.2 200.66) (xy 205.74 200.66))
+    (stroke (width 0) (type default))
+  )
   (wire (pts (xy 363.22 116.84) (xy 350.52 116.84))
     (stroke (width 0) (type default))
@@
     (effects (font (size 1.27 1.27)) (justify left bottom))
   )
-  (label "LOOP" (at 203.2 200.66 180) (fields_autoplaced)
-    (effects (font (size 1.27 1.27)) (justify right bottom))
+  (label "LOOP" (at 205.74 203.2 0) (fields_autoplaced)
+    (effects (font (size 1.27 1.27)) (justify left bottom))
   )
   (label "QUADSPI_BK1_IO3" (at 76.2 162.56 0) (fields_autoplaced)
@@
     )
   )
-  (symbol (lib_id "Device:R_Small") (at 200.66 203.2 270) (mirror x) (unit 1)
-    (in_bom yes) (on_board yes) (dnp no)
-    (property "Reference" "R?" (at 200.66 208.28 90)
-      (effects (font (size 1.27 1.27)))
-    )
-    (property "Value" "2.2K" (at 200.66 205.74 90)
-      (effects (font (size 1.27 1.27)))
-    )
-    (property "Footprint" "Resistor_SMD:R_0805_2012Metric" (at 200.66 203.2 0)
-      (effects (font (size 1.27 1.27)) hide)
-    )
-    (property "Datasheet" "~" (at 200.66 203.2 0)
-      (effects (font (size 1.27 1.27)) hide)
-    )
-    (pin "1")
-    (pin "2")
-    (instances
-      (project "Avionus_Flight_Controller"
-        (path "/ddc7e940-0588-4587-8902-8ced9e615ace/07011d92-7eb9-4cfe-9164-8ccacd4ef57f"
-          (reference "R?") (unit 1)
-        )
-        (path "/ddc7e940-0588-4587-8902-8ced9e615ace/fb82246b-9ed4-401c-b8a1-7e9ae6260bc5"
-          (reference "R301") (unit 1)
-        )
-      )
-    )
-  )
   (symbol (lib_id "Connector:TestPoint") (at 182.88 139.7 270) (unit 1)
     (in_bom yes) (on_board yes) (dnp no) (fields_autoplaced)
@@
         (path "/ddc7e940-0588-4587-8902-8ced9e615ace/fb82246b-9ed4-401c-b8a1-7e9ae6260bc5"
           (reference "TP304") (unit 1)
+        )
+      )
+    )
+  )
+  (symbol (lib_id "Device:R_Small") (at 200.66 200.66 270) (unit 1)
+    (in_bom yes) (on_board yes) (dnp no)
+    (property "Reference" "R301" (at 200.66 195.58 90)
+      (effects (font (size 1.27 1.27)))
+    )
+    (property "Value" "10K" (at 200.66 198.12 90)
+      (effects (font (size 1.27 1.27)))
+    )
+    (property "Footprint" "Resistor_SMD:R_0603_1608Metric" (at 200.66 200.66 0)
+      (effects (font (size 1.27 1.27)) hide)
+    )
+    (property "Datasheet" "~" (at 200.66 200.66 0)
+      (effects (font (size 1.27 1.27)) hide)
+    )
+    (pin "1")
+    (pin "2")
+    (instances
+      (project "Avionus_Flight_Controller"
+        (path "/ddc7e940-0588-4587-8902-8ced9e615ace/fb82246b-9ed4-401c-b8a1-7e9ae6260bc5"
+          (reference "R301") (unit 1)
         )
       )
@@
         )
       )
+    )
+  )
+  (symbol (lib_id "Device:R_Small") (at 200.66 203.2 270) (mirror x) (unit 1)
+    (in_bom yes) (on_board yes) (dnp no)
+    (property "Reference" "R303" (at 200.66 208.28 90)
+      (effects (font (size 1.27 1.27)))
+    )
+    (property "Value" "10K" (at 200.66 205.74 90)
+      (effects (font (size 1.27 1.27)))
+    )
+    (property "Footprint" "Resistor_SMD:R_0603_1608Metric" (at 200.66 203.2 0)
+      (effects (font (size 1.27 1.27)) hide)
+    )
+    (property "Datasheet" "~" (at 200.66 203.2 0)
+      (effects (font (size 1.27 1.27)) hide)
+    )
+    (pin "1")
+    (pin "2")
+    (instances
+      (project "Avionus_Flight_Controller"
+        (path "/ddc7e940-0588-4587-8902-8ced9e615ace/fb82246b-9ed4-401c-b8a1-7e9ae6260bc5"
+          (reference "R303") (unit 1)
+        )
+      )

Commit message: More routing
Parts:
- added R304: 10K, Resistor_SMD:R_0603_1608Metric, symbol Device:R_Small
Connections:
- net GPIO_PD1 is gone; now on an unnamed net: U301.115 (PD1)
- net USB_OTG_HS_VBUS: now also R304.1; no longer U301.74 (PB13)
- net at TP305.1: no longer U301.1 (PE2)
- new net: R304.2, U301.74 (PB13)
- new net GPIO_PE2: U301.1 (PE2)
Other:
- moved on the sheet: TP305
Changed lines of the file:
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@@
+    (stroke (width 0) (type default))
+  )
+  (wire (pts (xy 182.88 154.94) (xy 203.2 154.94))
     (stroke (width 0) (type default))
   )
@@
     (effects (font (size 1.27 1.27)) (justify left))
   )
-  (hierarchical_label "USB_OTG_HS_VBUS" (shape bidirectional) (at 182.88 154.94 0) (fields_autoplaced)
+  (hierarchical_label "USB_OTG_HS_VBUS" (shape bidirectional) (at 208.28 154.94 0) (fields_autoplaced)
     (effects (font (size 1.27 1.27)) (justify left))
   )
@@
     (effects (font (size 1.27 1.27)) (justify right))
   )
-  (hierarchical_label "GPIO_PD1" (shape output) (at 182.88 210.82 0) (fields_autoplaced)
-    (effects (font (size 1.27 1.27)) (justify left))
+  (hierarchical_label "GPIO_PE2" (shape output) (at 121.92 195.58 180) (fields_autoplaced)
+    (effects (font (size 1.27 1.27)) (justify right))
   )
   (hierarchical_label "TIM4_CH4" (shape output) (at 182.88 246.38 0) (fields_autoplaced)
@@
         (path "/ddc7e940-0588-4587-8902-8ced9e615ace/fb82246b-9ed4-401c-b8a1-7e9ae6260bc5"
           (reference "C306") (unit 1)
+        )
+      )
+    )
+  )
+  (symbol (lib_id "Device:R_Small") (at 205.74 154.94 270) (mirror x) (unit 1)
+    (in_bom yes) (on_board yes) (dnp no)
+    (property "Reference" "R304" (at 205.74 160.02 90)
+      (effects (font (size 1.27 1.27)))
+    )
+    (property "Value" "10K" (at 205.74 157.48 90)
+      (effects (font (size 1.27 1.27)))
+    )
+    (property "Footprint" "Resistor_SMD:R_0603_1608Metric" (at 205.74 154.94 0)
+      (effects (font (size 1.27 1.27)) hide)
+    )
+    (property "Datasheet" "~" (at 205.74 154.94 0)
+      (effects (font (size 1.27 1.27)) hide)
+    )
+    (pin "1")
+    (pin "2")
+    (instances
+      (project "Avionus_Flight_Controller"
+        (path "/ddc7e940-0588-4587-8902-8ced9e615ace/fb82246b-9ed4-401c-b8a1-7e9ae6260bc5"
+          (reference "R304") (unit 1)
         )
       )
@@
     )
   )
-  (symbol (lib_id "Connector:TestPoint") (at 121.92 195.58 90) (unit 1)
-    (in_bom yes) (on_board yes) (dnp no) (fields_autoplaced)
-    (property "Reference" "TP305" (at 116.84 195.58 90)
-      (effects (font (size 1.27 1.27)) (justify left))
-    )
-    (property "Value" "~" (at 116.84 194.31 90)
-      (effects (font (size 1.27 1.27)) (justify left))
-    )
-    (property "Footprint" "TestPoint:TestPoint_Pad_D1.0mm" (at 121.92 190.5 0)
-      (effects (font (size 1.27 1.27)) hide)
-    )
-    (property "Datasheet" "~" (at 121.92 190.5 0)
-      (effects (font (size 1.27 1.27)) hide)
-    )
+  (symbol (lib_id "Connector:TestPoint") (at 182.88 210.82 270) (unit 1)
+    (in_bom yes) (on_board yes) (dnp no) (fields_autoplaced)
+    (property "Reference" "TP305" (at 187.96 210.82 90)
+      (effects (font (size 1.27 1.27)) (justify left))
+    )
+    (property "Value" "~" (at 187.96 212.09 90)
+      (effects (font (size 1.27 1.27)) (justify left))
+    )
+    (property "Footprint" "TestPoint:TestPoint_Pad_D1.0mm" (at 182.88 215.9 0)
+      (effects (font (size 1.27 1.27)) hide)
+    )
+    (property "Datasheet" "~" (at 182.88 215.9 0)
+      (effects (font (size 1.27 1.27)) hide)
+    )
