File: Hardware/Avionus_Flight_Controller.kicad_sch (KiCad schematic)
At the start: 0 parts

Commit message: Checkpoint
Other:
- sheet MCU ports: added ADC1_IN8, ADC1_IN9, ADC2_IN10, ADC2_IN11, ADC2_IN12, ADC2_IN13, GPIO_PB10+EXTI10, GPIO_PB12+EXTI12, GPIO_PD10, GPIO_PD11, GPIO_PD3+EXTI3, GPIO_PE11, GPIO_PE15+EXTI15, GPIO_PE3, GPIO_PE5+EXTI5, GPIO_PF11, GPIO_PF12, GPIO_PF13, GPIO_PF2+EXTI2, GPIO_PG1+EXTI1, GPIO_PG13+EXTI13, GPIO_PG15, GPIO_PG6+EXTI6, SPI1_MISO, SPI1_MOSI, SPI1_SCK, TIM2_CH1, TIM2_CH2, TIM2_CH3, TIM2_CH4, UART8_RX+EXTI0, USART3_RX; removed ADC1_IN10, GPIO_PA0+EXTI0+TIM2_CH1+TIM2_ETR+TIM5_CH1, GPIO_PA2+EXTI2+TIM2_CH2+TIM5_CH3+USART2_TX, GPIO_PC1+EXTI1, GPIO_PC14+EXTI14, GPIO_PC15+EXTI15, GPIO_PD5+EXTI5, GPIO_PE15, GPIO_PE3+EXTI3, GPIO_PF2, GPIO_PG1, GPIO_PG13, GPIO_PG2, GPIO_PG3, SPI2_MISO, SPI2_MOSI, SPI2_SCK, UART8_RX, USART3_RX+EXTI9
- sheet POWER ports: added D0_VBAT, D3_3V3, D3_EN, D4_3V3, D4_EN, D5_5V, D5_EN, MEAS_D1_5V, ~{D5_FAULT}; removed D0_3V3_BACKUP, D1_5V
- sheet RF ports: added BUSY, DIO1, DIO2, DIO3, RX_SWITCH, TX_SWITCH; removed DIO[0..5]
- sheet SERVO ports: added CH[0..15]; removed CH[0..11]

Commit message: Checkpoint
Other:
- sheet POWER ports: added MEAS_D2_1V8, MEAS_D2_3V3, MEAS_D3_3V3, MEAS_D4_3V3, SERVO_5V_AUX_EN; removed ~{SERVO_5V_AUX_EN}
Changed lines of the file:
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@@
   (junction (at 66.04 157.48) (diameter 0) (color 0 0 0 0)
   )
-  (junction (at 106.68 243.84) (diameter 0) (color 0 0 0 0)
-  )
-  (junction (at 109.22 241.3) (diameter 0) (color 0 0 0 0)
-  )
   (junction (at 63.5 124.46) (diameter 0) (color 0 0 0 0)
   )
@@
   (junction (at 276.86 83.82) (diameter 0) (color 0 0 0 0)
   )
-  (junction (at 111.76 238.76) (diameter 0) (color 0 0 0 0)
-  )
   (junction (at 106.68 73.66) (diameter 0) (color 0 0 0 0)
   )
@@
   (junction (at 307.34 86.36) (diameter 0) (color 0 0 0 0)
   )
-  (junction (at 114.3 236.22) (diameter 0) (color 0 0 0 0)
-  )
   (junction (at 66.04 223.52) (diameter 0) (color 0 0 0 0)
   )
@@
     (stroke (width 0) (type default))
   )
-  (wire (pts (xy 111.76 223.52) (xy 111.76 238.76))
-    (stroke (width 0) (type default))
-  )
   (wire (pts (xy 254 190.5) (xy 279.4 190.5))
     (stroke (width 0) (type default))
@@
     (stroke (width 0) (type default))
   )
-  (wire (pts (xy 60.96 238.76) (xy 111.76 238.76))
+  (wire (pts (xy 60.96 238.76) (xy 312.42 238.76))
     (stroke (width 0) (type default))
   )
@@
     (stroke (width 0) (type default))
   )
-  (wire (pts (xy 114.3 226.06) (xy 114.3 236.22))
+  (wire (pts (xy 101.6 226.06) (xy 127 226.06))
     (stroke (width 0) (type default))
   )
@@
     (stroke (width 0) (type default))
   )
-  (wire (pts (xy 63.5 236.22) (xy 114.3 236.22))
+  (wire (pts (xy 63.5 236.22) (xy 309.88 236.22))
     (stroke (width 0) (type default))
   )
@@
     (stroke (width 0) (type default))
   )
-  (wire (pts (xy 106.68 218.44) (xy 106.68 243.84))
-    (stroke (width 0) (type default))
-  )
   (wire (pts (xy 187.96 231.14) (xy 187.96 228.6))
     (stroke (width 0) (type default))
@@
     (stroke (width 0) (type default))
   )
-  (wire (pts (xy 106.68 243.84) (xy 317.5 243.84))
-    (stroke (width 0) (type default))
-  )
   (wire (pts (xy 106.68 73.66) (xy 127 73.66))
     (stroke (width 0) (type default))
@@
     (stroke (width 0) (type default))
   )
-  (wire (pts (xy 127 223.52) (xy 111.76 223.52))
-    (stroke (width 0) (type default))
-  )
   (wire (pts (xy 254 172.72) (xy 279.4 172.72))
     (stroke (width 0) (type default))
@@
     (stroke (width 0) (type default))
   )
-  (wire (pts (xy 127 226.06) (xy 114.3 226.06))
-    (stroke (width 0) (type default))
-  )
   (wire (pts (xy 101.6 190.5) (xy 127 190.5))
     (stroke (width 0) (type default))
@@
     (stroke (width 0) (type default))
   )
-  (wire (pts (xy 109.22 220.98) (xy 109.22 241.3))
-    (stroke (width 0) (type default))
-  )
   (bus (pts (xy 104.14 129.54) (xy 104.14 132.08))
     (stroke (width 0) (type default))
@@
     (stroke (width 0) (type default))
   )
-  (wire (pts (xy 127 220.98) (xy 109.22 220.98))
-    (stroke (width 0) (type default))
-  )
   (wire (pts (xy 254 81.28) (xy 279.4 81.28))
     (stroke (width 0) (type default))
   )
-  (wire (pts (xy 127 218.44) (xy 106.68 218.44))
-    (stroke (width 0) (type default))
-  )
   (wire (pts (xy 101.6 175.26) (xy 127 175.26))
     (stroke (width 0) (type default))
@@
     (stroke (width 0) (type default))
   )
-  (wire (pts (xy 111.76 238.76) (xy 312.42 238.76))
-    (stroke (width 0) (type default))
-  )
   (wire (pts (xy 254 175.26) (xy 279.4 175.26))
     (stroke (width 0) (type default))
@@
     (stroke (width 0) (type default))
   )
-  (wire (pts (xy 55.88 243.84) (xy 106.68 243.84))
+  (wire (pts (xy 55.88 243.84) (xy 317.5 243.84))
     (stroke (width 0) (type default))
   )
@@
     (stroke (width 0) (type default))
   )
-  (wire (pts (xy 58.42 241.3) (xy 109.22 241.3))
-    (stroke (width 0) (type default))
-  )
   (bus (pts (xy 104.14 154.94) (xy 104.14 157.48))
     (stroke (width 0) (type default))
@@
     (stroke (width 0) (type default))
   )
+  (wire (pts (xy 101.6 220.98) (xy 127 220.98))
+    (stroke (width 0) (type default))
+  )
   (wire (pts (xy 73.66 172.72) (xy 76.2 172.72))
     (stroke (width 0) (type default))
@@
     (stroke (width 0) (type default))
   )
-  (wire (pts (xy 114.3 236.22) (xy 309.88 236.22))
-    (stroke (width 0) (type default))
-  )
   (bus (pts (xy 104.14 134.62) (xy 104.14 137.16))
     (stroke (width 0) (type default))
@@
     (stroke (width 0) (type default))
   )
+  (wire (pts (xy 101.6 223.52) (xy 127 223.52))
+    (stroke (width 0) (type default))
+  )
   (wire (pts (xy 101.6 185.42) (xy 127 185.42))
     (stroke (width 0) (type default))
@@
     (stroke (width 0) (type default))
   )
-  (wire (pts (xy 109.22 241.3) (xy 314.96 241.3))
+  (wire (pts (xy 58.42 241.3) (xy 314.96 241.3))
     (stroke (width 0) (type default))
   )
@@
   )
   (wire (pts (xy 254 53.34) (xy 279.4 53.34))
+    (stroke (width 0) (type default))
+  )
+  (wire (pts (xy 101.6 218.44) (xy 127 218.44))
     (stroke (width 0) (type default))
   )
@@
       (effects (font (size 1.27 1.27)) (justify right))
     )
-    (pin "~{SERVO_5V_AUX_EN}" input (at 101.6 187.96 0)
+    (pin "SERVO_5V_AUX_EN" input (at 101.6 187.96 0)
       (effects (font (size 1.27 1.27)) (justify right))
     )
@@
       (effects (font (size 1.27 1.27)) (justify right))
     )
+    (pin "MEAS_D4_3V3" output (at 101.6 226.06 0)
+      (effects (font (size 1.27 1.27)) (justify right))
+    )
+    (pin "MEAS_D2_1V8" output (at 101.6 220.98 0)
+      (effects (font (size 1.27 1.27)) (justify right))
+    )
+    (pin "MEAS_D3_3V3" output (at 101.6 223.52 0)
+      (effects (font (size 1.27 1.27)) (justify right))
+    )
+    (pin "MEAS_D2_3V3" output (at 101.6 218.44 0)
+      (effects (font (size 1.27 1.27)) (justify right))
+    )

Commit message: Checkpoint
Parts:
- added SYM101: ~, leptunKicadLib:AMOGUS_exposed_copper, symbol Graphic:Logo_Open_Hardware_Small
Changed lines of the file:
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@@
     (effects (font (size 1.27 1.27)) (justify left bottom))
+  )
+  (symbol (lib_id "Graphic:Logo_Open_Hardware_Small") (at 25.4 25.4 0) (unit 1)
+    (in_bom no) (on_board yes) (dnp no) (fields_autoplaced)
+    (property "Reference" "SYM101" (at 25.4 18.415 0)
+      (effects (font (size 1.27 1.27)) hide)
+    )
+    (property "Value" "~" (at 25.4 31.115 0)
+      (effects (font (size 1.27 1.27)) hide)
+    )
+    (property "Footprint" "leptunKicadLib:AMOGUS_exposed_copper" (at 25.4 25.4 0)
+      (effects (font (size 1.27 1.27)) hide)
+    )
+    (property "Datasheet" "~" (at 25.4 25.4 0)
+      (effects (font (size 1.27 1.27)) hide)
+    )
+    (property "Sim.Enable" "0" (at 25.4 25.4 0)
+      (effects (font (size 1.27 1.27)) hide)
+    )
+    (instances
+      (project "Avionus_Flight_Controller"
+        (path "/ddc7e940-0588-4587-8902-8ced9e615ace"
+          (reference "SYM101") (unit 1)
+        )
+      )
+    )
   )
   (sheet (at 76.2 134.62) (size 25.4 27.94) (fields_autoplaced)

Commit message: Checkpoint
Changed lines of the file:
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@@
     (effects (font (size 1.27 1.27)) (justify left bottom))
+  )
+  (label "USB_D+" (at 127 43.18 180) (fields_autoplaced)
+    (effects (font (size 1.27 1.27)) (justify right bottom))
   )
   (label "CH15" (at 106.68 129.54 0) (fields_autoplaced)
@@
     (effects (font (size 1.27 1.27)) (justify left bottom))
   )
+  (label "USB_D-" (at 127 45.72 180) (fields_autoplaced)
+    (effects (font (size 1.27 1.27)) (justify right bottom))
+  )
   (label "CH10" (at 106.68 142.24 0) (fields_autoplaced)

Commit message: Checkpoint
Other:
- sheet DEBUG ports: added GNDDetect; removed none
- sheet MCU ports: added GPIO_PA12; removed ADC1_IN8, ADC1_IN9
- sheet POWER ports: added MEAS_D5_5V, MEAS_I_D1_5V, MEAS_I_SERVO_5V5, MEAS_POWER_IN, SERVO_ESC; removed MEAS_S[1..6]
- sheet SERVO ports: added VDD_ESC; removed none

Commit message: Checkpoint routing
Parts:
- SYM101: footprint leptunKicadLib:AMOGUS_exposed_copper -> leptunKicadLib:AMOGUS
Changed lines of the file:
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@@
       (effects (font (size 1.27 1.27)) hide)
     )
-    (property "Footprint" "leptunKicadLib:AMOGUS_exposed_copper" (at 25.4 25.4 0)
+    (property "Footprint" "leptunKicadLib:AMOGUS" (at 25.4 25.4 0)
       (effects (font (size 1.27 1.27)) hide)
     )

Commit message: Finalize schematic and some more routing
Other:
- sheet UI ports: added VDD_5V; removed VDD_3V3
Changed lines of the file:
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@@
   (junction (at 60.96 124.46) (diameter 0) (color 0 0 0 0)
   )
+  (junction (at 60.96 210.82) (diameter 0) (color 0 0 0 0)
+  )
   (junction (at 104.14 71.12) (diameter 0) (color 0 0 0 0)
   )
@@
   (junction (at 63.5 223.52) (diameter 0) (color 0 0 0 0)
   )
-  (junction (at 307.34 175.26) (diameter 0) (color 0 0 0 0)
-  )
   (junction (at 58.42 218.44) (diameter 0) (color 0 0 0 0)
   )
@@
     (stroke (width 0) (type default))
   )
+  (wire (pts (xy 320.04 246.38) (xy 320.04 175.26))
+    (stroke (width 0) (type default))
+  )
   (wire (pts (xy 254 167.64) (xy 279.4 167.64))
     (stroke (width 0) (type default))
@@
     (stroke (width 0) (type default))
   )
+  (wire (pts (xy 50.8 246.38) (xy 320.04 246.38))
+    (stroke (width 0) (type default))
+  )
   (wire (pts (xy 106.68 152.4) (xy 127 152.4))
     (stroke (width 0) (type default))
@@
     (stroke (width 0) (type default))
   )
+  (wire (pts (xy 304.8 175.26) (xy 320.04 175.26))
+    (stroke (width 0) (type default))
+  )
   (wire (pts (xy 106.68 160.02) (xy 127 160.02))
     (stroke (width 0) (type default))
@@
     (stroke (width 0) (type default))
   )
-  (wire (pts (xy 307.34 233.68) (xy 307.34 175.26))
+  (wire (pts (xy 307.34 104.14) (xy 307.34 233.68))
     (stroke (width 0) (type default))
   )
@@
     (stroke (width 0) (type default))
   )
+  (wire (pts (xy 60.96 210.82) (xy 50.8 210.82))
+    (stroke (width 0) (type default))
+  )
   (wire (pts (xy 254 68.58) (xy 279.4 68.58))
     (stroke (width 0) (type default))
@@
     (stroke (width 0) (type default))
   )
+  (wire (pts (xy 50.8 210.82) (xy 50.8 246.38))
+    (stroke (width 0) (type default))
+  )
   (wire (pts (xy 68.58 55.88) (xy 127 55.88))
     (stroke (width 0) (type default))
@@
     (stroke (width 0) (type default))
   )
-  (wire (pts (xy 307.34 175.26) (xy 307.34 104.14))
-    (stroke (width 0) (type default))
-  )
   (wire (pts (xy 254 218.44) (xy 279.4 218.44))
     (stroke (width 0) (type default))
@@
   )
   (wire (pts (xy 254 129.54) (xy 279.4 129.54))
-    (stroke (width 0) (type default))
-  )
-  (wire (pts (xy 304.8 175.26) (xy 307.34 175.26))
     (stroke (width 0) (type default))
   )
@@
       (effects (font (size 1.27 1.27)) (justify left top))
     )
-    (pin "VDD_3V3" passive (at 304.8 175.26 0)
-      (effects (font (size 1.27 1.27)) (justify right))
-    )
     (pin "~{BUZZER}" input (at 279.4 175.26 180)
       (effects (font (size 1.27 1.27)) (justify left))
@@
       (effects (font (size 1.27 1.27)) (justify left))
     )
+    (pin "VDD_5V" passive (at 304.8 175.26 0)
+      (effects (font (size 1.27 1.27)) (justify right))
+    )
     (instances

Commit message: Lots of routing
Changed lines of the file:
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@@
       (effects (font (size 1.27 1.27)) (justify left))
     )
-    (pin "TX_SWITCH" input (at 279.4 142.24 180)
-      (effects (font (size 1.27 1.27)) (justify left))
-    )
-    (pin "RX_SWITCH" input (at 279.4 144.78 180)
+    (pin "TX_SWITCH" input (at 279.4 144.78 180)
+      (effects (font (size 1.27 1.27)) (justify left))
+    )
+    (pin "RX_SWITCH" input (at 279.4 142.24 180)
       (effects (font (size 1.27 1.27)) (justify left))
     )
@@
       (effects (font (size 1.27 1.27)) (justify left))
     )
-    (pin "TIM2_CH4" output (at 127 129.54 180)
-      (effects (font (size 1.27 1.27)) (justify left))
-    )
-    (pin "TIM2_CH1" output (at 127 137.16 180)
-      (effects (font (size 1.27 1.27)) (justify left))
-    )
-    (pin "TIM2_CH2" output (at 127 134.62 180)
-      (effects (font (size 1.27 1.27)) (justify left))
-    )
-    (pin "TIM2_CH3" output (at 127 132.08 180)
-      (effects (font (size 1.27 1.27)) (justify left))
-    )
+    (pin "TIM2_CH4" output (at 127 137.16 180)
+      (effects (font (size 1.27 1.27)) (justify left))
+    )
+    (pin "TIM2_CH1" output (at 127 129.54 180)
+      (effects (font (size 1.27 1.27)) (justify left))
+    )
+    (pin "TIM2_CH2" output (at 127 132.08 180)
+      (effects (font (size 1.27 1.27)) (justify left))
+    )
+    (pin "TIM2_CH3" output (at 127 134.62 180)
+      (effects (font (size 1.27 1.27)) (justify left))
+    )
