File: Hardware/POWER.kicad_sch (KiCad schematic)
At the start: 65 parts, among them J15 5V_USB, J17 Battery IN, Q1 RE1C002UN, U11 AOZ1212AI, U5 AP2112K-3.3, U5 AP2151W, U6 AP2112K-1.8, U7 AP2112K-3.3

Commit message: Checkpoint
Changed lines of the file:
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@@
     )
   )
-  (symbol (lib_id "Device:R_Small") (at 93.98 185.42 270) (unit 1)
-    (in_bom yes) (on_board yes) (dnp no) (fields_autoplaced)
-    (property "Reference" "R39" (at 93.98 187.96 90)
-      (effects (font (size 1.27 1.27)))
-    )
-    (property "Value" "1K" (at 93.98 190.5 90)
+  (symbol (lib_id "Device:R_Small") (at 93.98 185.42 270) (mirror x) (unit 1)
+    (in_bom yes) (on_board yes) (dnp no)
+    (property "Reference" "R39" (at 93.98 182.88 90)
+      (effects (font (size 1.27 1.27)))
+    )
+    (property "Value" "1K" (at 93.98 180.34 90)
       (effects (font (size 1.27 1.27)))
     )
@@
     )
   )
-  (symbol (lib_id "Device:R_Small") (at 93.98 177.8 270) (unit 1)
-    (in_bom yes) (on_board yes) (dnp no) (fields_autoplaced)
-    (property "Reference" "R38" (at 93.98 180.34 90)
-      (effects (font (size 1.27 1.27)))
-    )
-    (property "Value" "1K" (at 93.98 182.88 90)
+  (symbol (lib_id "Device:R_Small") (at 93.98 177.8 270) (mirror x) (unit 1)
+    (in_bom yes) (on_board yes) (dnp no)
+    (property "Reference" "R38" (at 93.98 175.26 90)
+      (effects (font (size 1.27 1.27)))
+    )
+    (property "Value" "1K" (at 93.98 172.72 90)
       (effects (font (size 1.27 1.27)))
     )
@@
   )
   (symbol (lib_id "Device:R_Small") (at 93.98 170.18 270) (unit 1)
-    (in_bom yes) (on_board yes) (dnp no) (fields_autoplaced)
+    (in_bom yes) (on_board yes) (dnp no)
     (property "Reference" "R34" (at 93.98 165.1 90)
       (effects (font (size 1.27 1.27)))

Commit message: Checkpoint
Changed lines of the file:
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@@
   (junction (at 208.28 76.2) (diameter 0) (color 0 0 0 0)
   )
+  (junction (at 35.56 190.5) (diameter 0) (color 0 0 0 0)
+  )
   (junction (at 144.78 114.3) (diameter 0) (color 0 0 0 0)
   )
@@
   (junction (at 165.1 144.78) (diameter 0) (color 0 0 0 0)
   )
+  (junction (at 256.54 106.68) (diameter 0) (color 0 0 0 0)
+  )
   (junction (at 165.1 175.26) (diameter 0) (color 0 0 0 0)
   )
@@
   (junction (at 45.72 43.18) (diameter 0) (color 0 0 0 0)
   )
+  (wire (pts (xy 35.56 190.5) (xy 38.1 190.5))
+    (stroke (width 0) (type default))
+  )
   (wire (pts (xy 43.18 27.94) (xy 30.48 27.94))
     (stroke (width 0) (type default))
@@
     (stroke (width 0) (type default))
   )
+  (wire (pts (xy 256.54 106.68) (xy 259.08 106.68))
+    (stroke (width 0) (type default))
+  )
   (wire (pts (xy 243.84 121.92) (xy 246.38 121.92))
     (stroke (width 0) (type default))
@@
     (stroke (width 0) (type default))
   )
+  (wire (pts (xy 254 106.68) (xy 256.54 106.68))
+    (stroke (width 0) (type default))
+  )
   (wire (pts (xy 165.1 127) (xy 165.1 124.46))
     (stroke (width 0) (type default))
@@
     (stroke (width 0) (type default))
   )
+  (wire (pts (xy 33.02 190.5) (xy 35.56 190.5))
+    (stroke (width 0) (type default))
+  )
   (wire (pts (xy 104.14 50.8) (xy 104.14 53.34))
     (stroke (width 0) (type default))
@@
     (effects (font (size 1.27 1.27)) (justify left))
   )
-  (hierarchical_label "D0_3V3_BACKUP" (shape passive) (at 38.1 190.5 180) (fields_autoplaced)
+  (hierarchical_label "D0_3V3_BACKUP" (shape passive) (at 33.02 190.5 180) (fields_autoplaced)
     (effects (font (size 1.27 1.27)) (justify right))
   )
@@
     )
   )
+  (symbol (lib_id "power:PWR_FLAG") (at 35.56 190.5 180) (unit 1)
+    (in_bom yes) (on_board yes) (dnp no) (fields_autoplaced)
+    (property "Reference" "#FLG01" (at 35.56 192.405 0)
+      (effects (font (size 1.27 1.27)) hide)
+    )
+    (property "Value" "PWR_FLAG" (at 35.56 195.58 0)
+      (effects (font (size 1.27 1.27)))
+    )
+    (property "Footprint" "" (at 35.56 190.5 0)
+      (effects (font (size 1.27 1.27)) hide)
+    )
+    (property "Datasheet" "~" (at 35.56 190.5 0)
+      (effects (font (size 1.27 1.27)) hide)
+    )
+    (pin "1")
+    (instances
+      (project "Avionus_Flight_Controller"
+        (path "/ddc7e940-0588-4587-8902-8ced9e615ace/26f6db01-be5b-4944-aca8-25d2b5bac430"
+          (reference "#FLG01") (unit 1)
+        )
+      )
+    )
+  )
   (symbol (lib_id "Device:L_Small") (at 96.52 43.18 90) (unit 1)
     (in_bom yes) (on_board yes) (dnp no) (fields_autoplaced)
@@
     )
   )
+  (symbol (lib_id "power:PWR_FLAG") (at 256.54 106.68 180) (unit 1)
+    (in_bom yes) (on_board yes) (dnp no) (fields_autoplaced)
+    (property "Reference" "#FLG05" (at 256.54 108.585 0)
+      (effects (font (size 1.27 1.27)) hide)
+    )
+    (property "Value" "PWR_FLAG" (at 256.54 111.76 0)
+      (effects (font (size 1.27 1.27)))
+    )
+    (property "Footprint" "" (at 256.54 106.68 0)
+      (effects (font (size 1.27 1.27)) hide)
+    )
+    (property "Datasheet" "~" (at 256.54 106.68 0)
+      (effects (font (size 1.27 1.27)) hide)
+    )
+    (pin "1")
+    (instances
+      (project "Avionus_Flight_Controller"
+        (path "/ddc7e940-0588-4587-8902-8ced9e615ace/26f6db01-be5b-4944-aca8-25d2b5bac430"
+          (reference "#FLG05") (unit 1)
+        )
+      )
+    )
+  )
   (symbol (lib_id "Device:R_Small") (at 165.1 66.04 90) (mirror x) (unit 1)
     (in_bom yes) (on_board yes) (dnp no) (fields_autoplaced)
@@
     )
   )
+  (symbol (lib_id "power:PWR_FLAG") (at 43.18 22.86 0) (unit 1)
+    (in_bom yes) (on_board yes) (dnp no) (fields_autoplaced)
+    (property "Reference" "#FLG06" (at 43.18 20.955 0)
+      (effects (font (size 1.27 1.27)) hide)
+    )
+    (property "Value" "PWR_FLAG" (at 43.18 17.78 0)
+      (effects (font (size 1.27 1.27)))
+    )
+    (property "Footprint" "" (at 43.18 22.86 0)
+      (effects (font (size 1.27 1.27)) hide)
+    )
+    (property "Datasheet" "~" (at 43.18 22.86 0)
+      (effects (font (size 1.27 1.27)) hide)
+    )
+    (pin "1")
+    (instances
+      (project "Avionus_Flight_Controller"
+        (path "/ddc7e940-0588-4587-8902-8ced9e615ace/26f6db01-be5b-4944-aca8-25d2b5bac430"
+          (reference "#FLG06") (unit 1)
+        )
+      )
+    )
+  )
   (symbol (lib_id "Connector:TestPoint") (at 256.54 45.72 90) (unit 1)
     (in_bom yes) (on_board yes) (dnp no) (fields_autoplaced)
@@
     )
   )
+  (symbol (lib_id "power:PWR_FLAG") (at 248.92 91.44 90) (unit 1)
+    (in_bom yes) (on_board yes) (dnp no) (fields_autoplaced)
+    (property "Reference" "#FLG04" (at 247.015 91.44 0)
+      (effects (font (size 1.27 1.27)) hide)
+    )
+    (property "Value" "PWR_FLAG" (at 245.11 91.44 90)
+      (effects (font (size 1.27 1.27)) (justify left))
+    )
+    (property "Footprint" "" (at 248.92 91.44 0)
+      (effects (font (size 1.27 1.27)) hide)
+    )
+    (property "Datasheet" "~" (at 248.92 91.44 0)
+      (effects (font (size 1.27 1.27)) hide)
+    )
+    (pin "1")
+    (instances
+      (project "Avionus_Flight_Controller"
+        (path "/ddc7e940-0588-4587-8902-8ced9e615ace/26f6db01-be5b-4944-aca8-25d2b5bac430"
+          (reference "#FLG04") (unit 1)
+        )
+      )
+    )
+  )
   (symbol (lib_id "Device:C_Small") (at 144.78 182.88 0) (mirror y) (unit 1)
     (in_bom yes) (on_board yes) (dnp no) (fields_autoplaced)
@@
     )
   )
+  (symbol (lib_id "power:PWR_FLAG") (at 119.38 43.18 0) (unit 1)
+    (in_bom yes) (on_board yes) (dnp no) (fields_autoplaced)
+    (property "Reference" "#FLG03" (at 119.38 41.275 0)
+      (effects (font (size 1.27 1.27)) hide)
+    )
+    (property "Value" "PWR_FLAG" (at 119.38 38.1 0)
+      (effects (font (size 1.27 1.27)))
+    )
+    (property "Footprint" "" (at 119.38 43.18 0)
+      (effects (font (size 1.27 1.27)) hide)
+    )
+    (property "Datasheet" "~" (at 119.38 43.18 0)
+      (effects (font (size 1.27 1.27)) hide)
+    )
+    (pin "1")
+    (instances
+      (project "Avionus_Flight_Controller"
+        (path "/ddc7e940-0588-4587-8902-8ced9e615ace/26f6db01-be5b-4944-aca8-25d2b5bac430"
+          (reference "#FLG03") (unit 1)
+        )
+      )
+    )
+  )
   (symbol (lib_id "power:GND") (at 259.08 127 0) (unit 1)
     (in_bom yes) (on_board yes) (dnp no) (fields_autoplaced)
@@
     )
   )
-  (symbol (lib_id "power:GND") (at 259.08 106.68 270) (mirror x) (unit 1)
+  (symbol (lib_id "power:GND") (at 254 106.68 270) (mirror x) (unit 1)
     (in_bom yes) (on_board yes) (dnp no) (fields_autoplaced)
-    (property "Reference" "#PWR034" (at 252.73 106.68 0)
+    (property "Reference" "#PWR034" (at 247.65 106.68 0)
       (effects (font (size 1.27 1.27)) hide)
     )
-    (property "Value" "GND" (at 255.27 106.68 90)
+    (property "Value" "GND" (at 250.19 106.68 90)
       (effects (font (size 1.27 1.27)) (justify right))
     )
-    (property "Footprint" "" (at 259.08 106.68 0)
+    (property "Footprint" "" (at 254 106.68 0)
       (effects (font (size 1.27 1.27)) hide)
     )
-    (property "Datasheet" "" (at 259.08 106.68 0)
+    (property "Datasheet" "" (at 254 106.68 0)
       (effects (font (size 1.27 1.27)) hide)
     )

Commit message: Checkpoint
Parts:
- BT201: renamed from BT1; footprint (none) -> leptunKicadLib:DS1092-12-N8S
- C202: renamed from C8; footprint Capacitor_SMD:C_1210_3225Metric -> (none)
- C206: renamed from C11; footprint Capacitor_SMD:C_1210_3225Metric -> (none)
- J201: renamed from J15; footprint (none) -> Connector_PinHeader_2.54mm:PinHeader_1x02_P2.54mm_Vertical
- R?: renamed from R28; footprint Resistor_SMD:R_1206_3216Metric -> (none)
- R?: renamed from R29; footprint Resistor_SMD:R_1206_3216Metric -> (none)
- renumbered C48 to C201, C49 to C203, C9 to C204, C10 to C205, C13 to C207, C15 to C208, C17 to C209, C14 to C210, C16 to C211, C18 to C212, C19 to C213, C20 to C214, C21 to C215, C22 to C216, C12 to C217, D5 to D201, D6 to D202, D1 to D203, D2 to D204, D3 to D205, F1 to F?, J17 to J202, L2 to L201, Q1 to Q?, R41 to R201, R33 to R202, R42 to R203, R40 to R204, R67 to R205, R32 to R206, R34 to R207, R38 to R208, R39 to R209, R51 to R212, R50 to R213, R49 to R214, R48 to R215, R47 to R216, R46 to R217, R52 to R218, R53 to R219, R54 to R220, R55 to R221, R56 to R222, R57 to R223, R58 to R224, R59 to R225, TP2 to TP201, TP3 to TP202, TP4 to TP203, TP5 to TP204, TP6 to TP205, TP7 to TP206, U5 to U202, U6 to U203, U7 to U204, U5 to U?, U11 to U?

Commit message: Checkpoint
Parts:
- removed C214, C216: 100nF, symbol Device:C_Small
- removed U? (x2): AP2151W, Package_TO_SOT_SMD:SOT-23-5, symbol leptunKicadLib:AP2151W
- added J201: 5V_SEL, Connector_PinHeader_2.54mm:PinHeader_2x03_P2.54mm_Vertical, symbol Connector_Generic:Conn_02x03_Odd_Even
- added J203: POWER IN, symbol Connector:Conn_01x02_Socket
- added SW201: START, symbol Switch:SW_Push
- added U205: AP22814BW5, Package_TO_SOT_SMD:SOT-23-5, symbol Power_Management:AP22814BW5
- C201: footprint (none) -> Capacitor_SMD:C_1206_3216Metric
- C202: value 22uF -> 100uF; footprint (none) -> Capacitor_THT:C_Radial_D8.0mm_H11.5mm_P3.50mm; symbol Device:C_Small -> Device:C_Polarized_Small; Rating (none) -> 50V
- C203, C209: footprint (none) -> Capacitor_SMD:C_0805_2012Metric
- C204: value 27nF -> 51pF; footprint (none) -> Capacitor_SMD:C_0402_1005Metric
- C205, C213: footprint (none) -> Capacitor_SMD:C_0603_1608Metric
- C206: renamed from C207; footprint (none) -> Capacitor_SMD:C_0805_2012Metric
- C207: renamed from C210; footprint (none) -> Capacitor_SMD:C_0805_2012Metric
- C208: renamed from C206; footprint (none) -> Capacitor_SMD:C_1210_3225Metric
- C210: renamed from C208; footprint (none) -> Capacitor_SMD:C_0805_2012Metric
- C211: renamed from C212; footprint (none) -> Capacitor_SMD:C_0805_2012Metric
- C212: renamed from C211; footprint (none) -> Capacitor_SMD:C_0805_2012Metric
- C214: renamed from C215; footprint (none) -> Capacitor_SMD:C_0603_1608Metric
- C215: renamed from C217; symbol Device:C_Small -> Device:C_Polarized_Small
- J202: renamed from J201; value 5V_USB -> E5V
- J204: renamed from J202; value Battery IN -> Battery
- R201, R202, R203, R204, R206, R207, R208, R209, R212, R213, R214, R215, R216, R217, R218: footprint (none) -> Resistor_SMD:R_0805_2012Metric
- R205: value 23K -> 22K; footprint (none) -> Resistor_SMD:R_0805_2012Metric
- R219, R220, R221, R222, R223, R224, R225, R? (x2): footprint (none) -> Resistor_SMD:R_0603_1608Metric
- renumbered U204 to U203, U203 to U204
Connections:
- net BATT_S6: no longer F?.2
- net D1_5V: now also R203.2, J201.1 (Pin_1), J201.3 (Pin_3), J201.5 (Pin_5), U205.5 (IN); no longer C208.1, J202.2 (Pin_2), L201.2, R?.1
- net GND: now also J202.1 (Pin_1), J203.1 (Pin_1), U205.2 (GND); no longer R203.2
- net SERVO_5V5: now also U205.1 (OUT)
- net USB_5V: now also J201.6 (Pin_6); no longer J202.1 (Pin_1)
- net at C202.1, F?.1, U?.7 (VIN): now also SW201.2; no longer D201.2
- net SERVO_5V_AUX_EN renamed ~{SERVO_5V_AUX_EN}
- net ~{SERVO_5V_AUX_EN}: now also U205.4 (~{EN})
- new net: J201.4 (Pin_4), J202.2 (Pin_2)
- new net: D201.2, SW201.1
- new net 5V_BUCK: C208.1, J201.2 (Pin_2), L201.2, R?.1
- new net PWR_IN: F?.2, J203.2 (Pin_2)
- new net ~{SERVO_5V_AUX_FAULT}: U205.3 (~{FLG})
Other:
- moved on the sheet: C203, C204, C206, C207, C209, C210, C211, C212, C213, C214, J202, J204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

Commit message: Checkpoint
Parts:
- F?: footprint Fuse:Fuse_1206_3216Metric -> (none)
- J203: footprint (none) -> Connector_AMASS:AMASS_XT30UPB-M_1x02_P5.0mm_Vertical
- J204: footprint (none) -> Connector_PinHeader_2.54mm:PinHeader_1x07_P2.54mm_Vertical
- TP201, TP202, TP203, TP204, TP205, TP206: footprint (none) -> TestPoint:TestPoint_Pad_D2.0mm
Changed lines of the file:
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@@
       (effects (font (size 1.27 1.27)) (justify left))
     )
-    (property "Footprint" "" (at 226.06 101.6 0)
+    (property "Footprint" "Connector_AMASS:AMASS_XT30UPB-M_1x02_P5.0mm_Vertical" (at 226.06 101.6 0)
       (effects (font (size 1.27 1.27)) hide)
     )
@@
       (effects (font (size 1.27 1.27)) hide)
     )
-    (property "Footprint" "" (at 256.54 45.72 0)
+    (property "Footprint" "TestPoint:TestPoint_Pad_D2.0mm" (at 256.54 45.72 0)
       (effects (font (size 1.27 1.27)) hide)
     )
@@
       (effects (font (size 1.27 1.27)) hide)
     )
-    (property "Footprint" "" (at 256.54 50.8 0)
+    (property "Footprint" "TestPoint:TestPoint_Pad_D2.0mm" (at 256.54 50.8 0)
       (effects (font (size 1.27 1.27)) hide)
     )
@@
       (effects (font (size 1.27 1.27)) hide)
     )
-    (property "Footprint" "" (at 256.54 40.64 0)
+    (property "Footprint" "TestPoint:TestPoint_Pad_D2.0mm" (at 256.54 40.64 0)
       (effects (font (size 1.27 1.27)) hide)
     )
@@
       (effects (font (size 1.27 1.27)) hide)
     )
-    (property "Footprint" "" (at 256.54 55.88 0)
+    (property "Footprint" "TestPoint:TestPoint_Pad_D2.0mm" (at 256.54 55.88 0)
       (effects (font (size 1.27 1.27)) hide)
     )
@@
       (effects (font (size 1.27 1.27)) hide)
     )
-    (property "Footprint" "" (at 256.54 66.04 0)
+    (property "Footprint" "TestPoint:TestPoint_Pad_D2.0mm" (at 256.54 66.04 0)
       (effects (font (size 1.27 1.27)) hide)
     )
@@
       (effects (font (size 1.27 1.27)) (justify left))
     )
-    (property "Footprint" "" (at 271.78 101.6 0)
+    (property "Footprint" "Connector_PinHeader_2.54mm:PinHeader_1x07_P2.54mm_Vertical" (at 271.78 101.6 0)
       (effects (font (size 1.27 1.27)) hide)
     )
@@
       (effects (font (size 1.27 1.27)))
     )
-    (property "Footprint" "Fuse:Fuse_1206_3216Metric" (at 29.21 24.13 0)
+    (property "Footprint" "" (at 29.21 24.13 0)
       (effects (font (size 1.27 1.27)) (justify left) hide)
     )
@@
       (effects (font (size 1.27 1.27)) hide)
     )
-    (property "Footprint" "" (at 256.54 60.96 0)
-      (effects (font (size 1.27 1.27)) hide)
-    )
+    (property "Footprint" "TestPoint:TestPoint_Pad_D2.0mm" (at 256.54 60.96 0)
+      (effects (font (size 1.27 1.27)) hide)
+    )

Commit message: Checkpoint
Parts:
- D203, D204, D205: footprint (none) -> LED_SMD:LED_1206_3216Metric
- F?: footprint (none) -> Fuse:Fuse_1812_4532Metric
- SW201: footprint (none) -> Button_Switch_THT:SW_PUSH_6mm_H5mm
- renumbered R204 to R201, R205 to R202, R206 to R203, R207 to R204, R208 to R205, R209 to R206, R212 to R209, R213 to R210, R214 to R211, R215 to R212, R216 to R213, R217 to R214, R218 to R215, R225 to R216, R224 to R217, R223 to R218, R222 to R219, R221 to R220, R220 to R221, R219 to R222, R201 to R223, R202 to R224, R203 to R225
Other:
- moved on the sheet: BT201, R209, R210, R211, R212, R213, R214, R215, R216, R217, R218, R219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

Commit message: Checkpoint
Parts:
- added C201, C203, C211, C217: 1uF, Capacitor_SMD:C_0805_2012Metric, symbol Device:C_Small
- added C204, C212: 100nF, Capacitor_SMD:C_0603_1608Metric, symbol Device:C_Small
- added C214: 22uF, Capacitor_SMD:C_1210_3225Metric, symbol Device:C_Small
- added D206, D207, D208: ~, LED_SMD:LED_1206_3216Metric, symbol Device:LED_Small
- added R202, R203, R208, R216: 100K, Resistor_SMD:R_0805_2012Metric, symbol Device:R_Small
- added R224: 10K, Resistor_SMD:R_0603_1608Metric, symbol Device:R_Small
- added R231, R232, R233: 1K, Resistor_SMD:R_0805_2012Metric, symbol Device:R_Small
- added TP201, TP202: ~, TestPoint:TestPoint_Pad_D2.0mm, symbol Connector:TestPoint
- added U201, U206: AP2112K-3.3, Package_TO_SOT_SMD:SOT-23-5, symbol Regulator_Linear:AP2112K-3.3
- added U203: AP2151W, Package_TO_SOT_SMD:SOT-23-5, symbol leptunKicadLib:AP2151W
- renumbered C201 to C202, C202 to C205, C203 to C206, C204 to C207, C205 to C208, C206 to C213, C211 to C215, C212 to C216, C207 to C218, C208 to C219, C213 to C220, C214 to C221, C215 to C222, J204 to J201, J203 to J202, J201 to J203, J202 to J204, R202 to R204, R223 to R207, R225 to R209, R209 to R210, R210 to R211, R211 to R212, R212 to R213, R213 to R214, R214 to R215, R215 to R217, R216 to R218, R217 to R219, R218 to R220, R219 to R221, R220 to R222, R221 to R223, R222 to R225, R203 to R226, R224 to R227, R204 to R228, R205 to R229, R206 to R230, TP201 to TP204, TP202 to TP205, TP204 to TP206, TP206 to TP207, TP205 to TP208, U203 to U204, U204 to U205, U202 to U207, U205 to U208
Connections:
- net D1_3V3: now also TP206.1
- net D1_5V: now also R228.1, TP208.1, C201.1, C204.1, C211.1, R216.1, U201.1 (VIN), U203.5 (IN), U206.1 (VIN); no longer TP205.1
- net D1_EN: no longer R228.1
- net D2_1V8: now also TP204.1; no longer TP206.1
- net D2_3V3: now also R229.1
- net D2_EN: no longer R229.1
- net GND: now also C201.2, C203.2, C204.2, C211.2, C212.2, C214.2, C217.2, R202.1, R203.2, R208.2, R224.2, U201.2 (GND), U203.2 (GND), U206.2 (GND)
- net SERVO_5V5: now also R233.1
- net USB_5V: no longer TP208.1
- net ~{SERVO_5V_AUX_EN}: no longer R230.1
- net at D203.1 (K), D204.1 (K), D205.1 (K)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: now also D206.1 (K), D207.1 (K), D208.1 (K)
- net D0_3V3_BACKUP renamed D0_VBAT
- net D0_VBAT: no longer TP204.1
- new net: D207.2 (A), R232.2
- new net: D208.2 (A), R233.2
- new net: D206.2 (A), R231.2
- new net D3_3V3: C203.1, R230.1, TP201.1, U201.5 (VOUT)
- new net D3_EN: R203.1, U201.3 (EN)
- new net D4_3V3: C217.1, R231.1, TP205.1, U206.5 (VOUT)
- new net D4_EN: R208.1, U206.3 (EN)
- new net D5_5V: C212.1, C214.1, R232.1, TP202.1, U203.1 (OUT)
- new net D5_EN: R202.2, U203.4 (EN)
- new net MEAS_D1_5V: R216.2, R224.1
- new net ~{D5_FAULT}: U203.3 (~{FLG})
Other:
- moved on the sheet: BT201, C202, C205, C206, C207, C208, C209, C210, C213, C215, C216, C218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

Commit message: Checkpoint
Parts:
- removed F?: 2000mA, Fuse:Fuse_1812_4532Metric, symbol Device:Polyfuse
- removed U208: AP22814BW5, Package_TO_SOT_SMD:SOT-23-5, symbol Power_Management:AP22814BW5
- added R234, R235, R236, R237: 10K, Resistor_SMD:R_0603_1608Metric, symbol Device:R_Small
- added U209: AP2171W, Package_TO_SOT_SMD:SOT-23-5, symbol Power_Management:AP2171W
- renumbered R227 to R226, R226 to R227
Connections:
- net ~{SERVO_5V_AUX_EN} is gone; now on net GND: R209.1
- net D1_5V: now also U209.5 (IN); no longer R209.2
- net D2_1V8: now also R235.1
- net D2_3V3: now also R234.1
- net D3_3V3: now also R236.1
- net D4_3V3: now also R237.1
- net GND: now also U209.2 (GND)
- net PWR_IN: now also C205.1, SW201.2, U?.7 (VIN)
- net SERVO_5V5: now also U209.1 (OUT)
- net ~{SERVO_5V_AUX_FAULT}: now also U209.3 (~{FLG})
- new net MEAS_D2_1V8: R235.2
- new net MEAS_D2_3V3: R234.2
- new net MEAS_D3_3V3: R236.2
- new net MEAS_D4_3V3: R237.2
- new net SERVO_5V_AUX_EN: R209.2, U209.4 (EN)
Other:
- moved on the sheet: C220, C221, C222, R209, R216, R217, R224, R225, TP207
