File: Hardware/Avionus_Flight_Controller.kicad_pcb (KiCad board)
At the start: 4 copper layers, 101.6 x 101.6 mm, 0 parts

Commit message: Checkpoint
Parts:
- added AE1001: SR4G080, leptunKicadLib:SR4G080, F.Cu at (30.2, 25.4)
- added BT201: Battery_Cell, leptunKicadLib:DS1092-12-N8S, F.Cu at (47.0, 43.8)
- added C1001: 4.3pF, Capacitor_SMD:C_0402_1005Metric_Pad0.74x0.62mm_HandSolder, F.Cu at (35.1, 36.1)
- added C1002: 3.6pF, Capacitor_SMD:C_0402_1005Metric_Pad0.74x0.62mm_HandSolder, F.Cu at (35.1, 32.5)
- added C1501: 100nF, Capacitor_SMD:C_0603_1608Metric, F.Cu at (75.9, 59.5)
- added C1502: 100nF, Capacitor_SMD:C_0603_1608Metric, F.Cu at (75.9, 62.0)
- added C1503: 100nF, Capacitor_SMD:C_0603_1608Metric, F.Cu at (75.9, 64.5)
- added C201: 1uF, Capacitor_SMD:C_0805_2012Metric, F.Cu at (131.6, 98.2)
- added C202: 4.7uF, Capacitor_SMD:C_1206_3216Metric, F.Cu at (177.4, 14.9)
- added C203: 1uF, Capacitor_SMD:C_0805_2012Metric, F.Cu at (131.6, 101.2)
- added C204: 100nF, Capacitor_SMD:C_0603_1608Metric, F.Cu at (44.9, 119.4)
- added C205: 100uF, Capacitor_THT:C_Radial_D8.0mm_H11.5mm_P3.50mm, F.Cu at (177.2, 25.8)
- added C206: 1uF, Capacitor_SMD:C_0805_2012Metric, F.Cu at (182.4, 19.2)
- added C207: 51pF, Capacitor_SMD:C_0402_1005Metric, F.Cu at (186.1, 18.7)
- added C208: 100nF, Capacitor_SMD:C_0603_1608Metric, F.Cu at (185.8, 22.3)
- added C209: 1uF, Capacitor_SMD:C_0805_2012Metric, F.Cu at (37.7, 15.3)
- added C210: 1uF, Capacitor_SMD:C_0805_2012Metric, F.Cu at (83.8, 68.1)
- added C211: 1uF, Capacitor_SMD:C_0805_2012Metric, F.Cu at (192.1, 111.0)
- added C212: 100nF, Capacitor_SMD:C_0603_1608Metric, F.Cu at (44.9, 121.9)
- added C213: 1uF, Capacitor_SMD:C_0805_2012Metric, F.Cu at (202.8, 23.6)
- added C214: 22uF, Capacitor_SMD:C_1210_3225Metric, F.Cu at (40.6, 116.0)
- added C215: 1uF, Capacitor_SMD:C_0805_2012Metric, F.Cu at (37.7, 18.4)
- added C216: 1uF, Capacitor_SMD:C_0805_2012Metric, F.Cu at (83.8, 71.1)
- added C217: 1uF, Capacitor_SMD:C_0805_2012Metric, F.Cu at (196.6, 105.0)
- added C218: 1uF, Capacitor_SMD:C_0805_2012Metric, F.Cu at (202.8, 26.6)
- added C219: 22uF, Capacitor_SMD:C_1210_3225Metric, F.Cu at (177.4, 18.7)
- added C220: 100nF, Capacitor_SMD:C_0603_1608Metric, F.Cu at (179.9, 103.2)
- added C221: 100nF, Capacitor_SMD:C_0603_1608Metric, F.Cu at (179.9, 105.7)
- added C222: 120uF, Capacitor_THT:C_Radial_D6.3mm_H11.0mm_P2.50mm, F.Cu at (204.8, 124.5)
- added C301: 15pF, Capacitor_SMD:C_0805_2012Metric, F.Cu at (91.8, 78.7)
- added C302: 15pF, Capacitor_SMD:C_0805_2012Metric, F.Cu at (91.8, 81.8)
- added C303: 2.2uF, Capacitor_SMD:C_0805_2012Metric, F.Cu at (42.9, 151.3)
- added C304: 2.2uF, Capacitor_SMD:C_0805_2012Metric, F.Cu at (42.9, 154.3)
- added C305: 100nF, Capacitor_SMD:C_0603_1608Metric, F.Cu at (31.0, 142.3)
- added C306: 100nF, Capacitor_SMD:C_0603_1608Metric, F.Cu at (31.0, 144.8)
- added C307: 100nF, Capacitor_SMD:C_0603_1608Metric, F.Cu at (31.0, 147.3)
- added C308: 100nF, Capacitor_SMD:C_0603_1608Metric, F.Cu at (31.0, 149.9)
- added C309: 100nF, Capacitor_SMD:C_0603_1608Metric, F.Cu at (31.0, 152.4)
- added C310: 100nF, Capacitor_SMD:C_0603_1608Metric, F.Cu at (35.0, 142.3)
- added C311: 100nF, Capacitor_SMD:C_0603_1608Metric, F.Cu at (35.0, 144.8)
- added C312: 100nF, Capacitor_SMD:C_0603_1608Metric, F.Cu at (35.0, 147.3)
- added C313: 100nF, Capacitor_SMD:C_0603_1608Metric, F.Cu at (35.0, 149.9)
- added C314: 100nF, Capacitor_SMD:C_0603_1608Metric, F.Cu at (35.0, 152.4)
- added C315: 100nF, Capacitor_SMD:C_0603_1608Metric, F.Cu at (39.0, 142.3)
- added C316: 100nF, Capacitor_SMD:C_0603_1608Metric, F.Cu at (39.0, 144.8)
- added C317: 4.7uF, Capacitor_SMD:C_1206_3216Metric, F.Cu at (31.8, 155.3)
- added C318: 100nF, Capacitor_SMD:C_0603_1608Metric, F.Cu at (39.0, 147.3)
- added C319: 100nF, Capacitor_SMD:C_0603_1608Metric, F.Cu at (222.8, 106.4)
- added C320: 1uF, Capacitor_SMD:C_0805_2012Metric, F.Cu at (43.2, 142.6)
- added C321: 1uF, Capacitor_SMD:C_0805_2012Metric, F.Cu at (43.2, 145.6)
- added C501: 100nF, Capacitor_SMD:C_0603_1608Metric, B.Cu at (76.9, 98.6)
- added C601: 100nF, Capacitor_SMD:C_0603_1608Metric, B.Cu at (70.0, 90.8)
- added C701: 100nF, Capacitor_SMD:C_0603_1608Metric, B.Cu at (95.8, 103.1)
- added D1301: ~, LED_SMD:LED_1206_3216Metric, F.Cu at (250.8, 80.0)
- added D1302: ~, LED_SMD:LED_1206_3216Metric, F.Cu at (250.8, 83.4)
- added D1303: ~, LED_SMD:LED_1206_3216Metric, F.Cu at (250.8, 86.8)
- added D1304: ~, LED_SMD:LED_1206_3216Metric, F.Cu at (250.8, 90.2)
- added D201: BAT54C, Package_TO_SOT_SMD:SOT-23, F.Cu at (182.7, 15.5)
- added D202: B540C-13-F, Diode_SMD:D_SMC, F.Cu at (169.1, 17.1)
- added D203: ~, LED_SMD:LED_1206_3216Metric, F.Cu at (163.1, 100.6)
- added D204: ~, LED_SMD:LED_1206_3216Metric, F.Cu at (163.1, 104.0)
- added D205: ~, LED_SMD:LED_1206_3216Metric, F.Cu at (163.1, 107.4)
- added D206: ~, LED_SMD:LED_1206_3216Metric, F.Cu at (163.1, 110.8)
- added D207: ~, LED_SMD:LED_1206_3216Metric, F.Cu at (163.1, 114.2)
- added D208: ~, LED_SMD:LED_1206_3216Metric, F.Cu at (163.1, 117.6)
- added J1101: PPM, Connector_PinHeader_2.54mm:PinHeader_1x03_P2.54mm_Horizontal, F.Cu at (54.6, 116.3)
- added J1102: iBUS, Connector_PinHeader_2.54mm:PinHeader_1x03_P2.54mm_Horizontal, F.Cu at (63.5, 116.3)
- added J1201: S0, Connector_PinHeader_2.54mm:PinHeader_1x03_P2.54mm_Vertical, F.Cu at (99.1, 124.5)
- added J1202: S1, Connector_PinHeader_2.54mm:PinHeader_1x03_P2.54mm_Vertical, F.Cu at (103.1, 124.5)
- added J1203: S2, Connector_PinHeader_2.54mm:PinHeader_1x03_P2.54mm_Vertical, F.Cu at (107.2, 124.5)
- added J1204: S3, Connector_PinHeader_2.54mm:PinHeader_1x03_P2.54mm_Vertical, F.Cu at (111.3, 124.5)
- added J1205: S4, Connector_PinHeader_2.54mm:PinHeader_1x03_P2.54mm_Vertical, F.Cu at (115.3, 124.5)
- added J1206: S5, Connector_PinHeader_2.54mm:PinHeader_1x03_P2.54mm_Vertical, F.Cu at (119.4, 124.5)
- added J1207: S6, Connector_PinHeader_2.54mm:PinHeader_1x03_P2.54mm_Horizontal, F.Cu at (88.9, 36.1)
- added J1208: S7, Connector_PinHeader_2.54mm:PinHeader_1x03_P2.54mm_Horizontal, F.Cu at (94.0, 116.3)
- added J1209: S8, Connector_PinHeader_2.54mm:PinHeader_1x03_P2.54mm_Horizontal, F.Cu at (36.1, 59.7)
- added J1210: S9, Connector_PinHeader_2.54mm:PinHeader_1x03_P2.54mm_Horizontal, F.Cu at (36.1, 68.6)
- added J1211: S10, Connector_PinHeader_2.54mm:PinHeader_1x03_P2.54mm_Horizontal, F.Cu at (36.1, 77.5)
- added J1212: S11, Connector_PinHeader_2.54mm:PinHeader_1x03_P2.54mm_Horizontal, F.Cu at (36.1, 86.3)
- added J1213: S12, Connector_PinHeader_2.54mm:PinHeader_1x03_P2.54mm_Horizontal, F.Cu at (116.3, 54.6)
- added J1214: S13, Connector_PinHeader_2.54mm:PinHeader_1x03_P2.54mm_Horizontal, F.Cu at (116.3, 63.5)
- added J1215: S14, Connector_PinHeader_2.54mm:PinHeader_1x03_P2.54mm_Horizontal, F.Cu at (116.3, 72.4)
- added J1216: S15, Connector_PinHeader_2.54mm:PinHeader_1x03_P2.54mm_Horizontal, F.Cu at (116.3, 81.3)
- added J1401: LIDAR, Connector_PinHeader_2.54mm:PinHeader_1x08_P2.54mm_Horizontal, F.Cu at (85.1, 116.3)
- added J201: Battery, Connector_PinHeader_2.54mm:PinHeader_1x07_P2.54mm_Vertical, F.Cu at (73.2, 29.2)
- added J202: POWER IN, Connector_AMASS:AMASS_XT30UPB-M_1x02_P5.0mm_Vertical, F.Cu at (78.1, 29.2)
- added J203: 5V_SEL, Connector_PinHeader_2.54mm:PinHeader_2x03_P2.54mm_Vertical, F.Cu at (172.9, 101.3)
- added J204: E5V, Connector_PinHeader_2.54mm:PinHeader_1x02_P2.54mm_Vertical, F.Cu at (208.4, 114.8)
- added J401: STDC14, leptunKicadLib:FTSH-107-01-L-DV-K-A, F.Cu at (30.5, 113.0)
- added J701: SD_Card, leptunKicadLib:SDP-09L-SG, B.Cu at (98.1, 103.0)
- added J801: USB_C_Receptacle_USB2.0, leptunKicadLib:USB4110-GF-A, F.Cu at (30.5, 99.1)
- added L1001: 5.1nH, Inductor_SMD:L_0402_1005Metric_Pad0.77x0.64mm_HandSolder, F.Cu at (35.6, 34.3)
- added L201: SRP6530A-6R8M, leptunKicadLib:SRP6530A-6R8M, F.Cu at (168.6, 33.8)
- added Q1101: RE1C002UN, Package_TO_SOT_SMD:SOT-416, F.Cu at (52.1, 113.0)
- added Q1102: RE1C002UN, Package_TO_SOT_SMD:SOT-416, F.Cu at (61.0, 113.0)
- added Q1201: RE1C002UN, Package_TO_SOT_SMD:SOT-416, F.Cu at (99.1, 116.3)
- added Q1202: RE1C002UN, Package_TO_SOT_SMD:SOT-416, F.Cu at (103.1, 116.3)
- added Q1203: RE1C002UN, Package_TO_SOT_SMD:SOT-416, F.Cu at (107.2, 116.3)
- added Q1204: RE1C002UN, Package_TO_SOT_SMD:SOT-416, F.Cu at (111.3, 116.3)
- added Q1205: RE1C002UN, Package_TO_SOT_SMD:SOT-416, F.Cu at (115.3, 116.3)
- added Q1206: RE1C002UN, Package_TO_SOT_SMD:SOT-416, F.Cu at (119.4, 116.3)
- added Q1207: RE1C002UN, Package_TO_SOT_SMD:SOT-416, F.Cu at (91.4, 39.4)
- added Q1208: RE1C002UN, Package_TO_SOT_SMD:SOT-416, F.Cu at (91.4, 113.0)
- added Q1209: RE1C002UN, Package_TO_SOT_SMD:SOT-416, F.Cu at (39.4, 57.1)
- added Q1210: RE1C002UN, Package_TO_SOT_SMD:SOT-416, F.Cu at (39.4, 66.0)
- added Q1211: RE1C002UN, Package_TO_SOT_SMD:SOT-416, F.Cu at (39.4, 74.9)
- added Q1212: RE1C002UN, Package_TO_SOT_SMD:SOT-416, F.Cu at (39.4, 83.8)
- added Q1213: RE1C002UN, Package_TO_SOT_SMD:SOT-416, F.Cu at (113.0, 57.1)
- added Q1214: RE1C002UN, Package_TO_SOT_SMD:SOT-416, F.Cu at (113.0, 66.0)
- added Q1215: RE1C002UN, Package_TO_SOT_SMD:SOT-416, F.Cu at (113.0, 74.9)
- added Q1216: RE1C002UN, Package_TO_SOT_SMD:SOT-416, F.Cu at (113.0, 83.8)
- added Q1301: RE1C002UN, Package_TO_SOT_SMD:SOT-416, F.Cu at (255.4, 88.5)
- added Q1501: RE1C002UN, Package_TO_SOT_SMD:SOT-416, F.Cu at (63.4, 59.9)
- added Q1502: RE1C002UN, Package_TO_SOT_SMD:SOT-416, F.Cu at (63.4, 63.3)
- added Q1503: RE1C002UN, Package_TO_SOT_SMD:SOT-416, F.Cu at (63.4, 66.6)
- added Q1504: RE1C002UN, Package_TO_SOT_SMD:SOT-416, F.Cu at (63.4, 70.0)
- added Q1505: RE1C002UN, Package_TO_SOT_SMD:SOT-416, F.Cu at (63.4, 73.3)
- added Q201: RE1C002UN, Package_TO_SOT_SMD:SOT-416, F.Cu at (209.0, 88.5)
- added R1001: 0R, Resistor_SMD:R_0402_1005Metric_Pad0.72x0.64mm_HandSolder, F.Cu at (35.6, 37.9)
- added R1101: 2.2K, Resistor_SMD:R_0805_2012Metric, F.Cu at (49.5, 112.4)
- added R1102: 2.2K, Resistor_SMD:R_0805_2012Metric, F.Cu at (58.4, 112.4)
- added R1103: 2.2K, Resistor_SMD:R_0805_2012Metric, F.Cu at (54.6, 112.4)
- added R1104: 2.2K, Resistor_SMD:R_0805_2012Metric, F.Cu at (63.5, 112.4)
- added R1201: 2.2K, Resistor_SMD:R_0805_2012Metric, F.Cu at (100.1, 112.5)
- added R1202: 2.2K, Resistor_SMD:R_0805_2012Metric, F.Cu at (104.1, 112.5)
- added R1203: 2.2K, Resistor_SMD:R_0805_2012Metric, F.Cu at (108.2, 112.5)
- added R1204: 2.2K, Resistor_SMD:R_0805_2012Metric, F.Cu at (112.3, 112.5)
- added R1205: 2.2K, Resistor_SMD:R_0805_2012Metric, F.Cu at (98.0, 112.5)
- added R1206: 2.2K, Resistor_SMD:R_0805_2012Metric, F.Cu at (102.1, 112.5)
- added R1207: 2.2K, Resistor_SMD:R_0805_2012Metric, F.Cu at (106.2, 112.5)
- added R1208: 2.2K, Resistor_SMD:R_0805_2012Metric, F.Cu at (110.2, 112.5)
- added R1209: 2.2K, Resistor_SMD:R_0805_2012Metric, F.Cu at (116.3, 112.5)
- added R1210: 2.2K, Resistor_SMD:R_0805_2012Metric, F.Cu at (120.4, 112.5)
- added R1211: 2.2K, Resistor_SMD:R_0805_2012Metric, F.Cu at (94.0, 40.0)
- added R1212: 2.2K, Resistor_SMD:R_0805_2012Metric, F.Cu at (88.9, 112.4)
- added R1213: 2.2K, Resistor_SMD:R_0805_2012Metric, F.Cu at (114.3, 112.5)
- added R1214: 2.2K, Resistor_SMD:R_0805_2012Metric, F.Cu at (118.4, 112.5)
- added R1215: 2.2K, Resistor_SMD:R_0805_2012Metric, F.Cu at (88.9, 40.0)
- added R1216: 2.2K, Resistor_SMD:R_0805_2012Metric, F.Cu at (94.0, 112.4)
- added R1217: 2.2K, Resistor_SMD:R_0805_2012Metric, F.Cu at (40.0, 54.6)
- added R1218: 2.2K, Resistor_SMD:R_0805_2012Metric, F.Cu at (40.0, 63.5)
- added R1219: 2.2K, Resistor_SMD:R_0805_2012Metric, F.Cu at (40.0, 72.4)
- added R1220: 2.2K, Resistor_SMD:R_0805_2012Metric, F.Cu at (40.0, 81.3)
- added R1221: 2.2K, Resistor_SMD:R_0805_2012Metric, F.Cu at (40.0, 59.7)
- added R1222: 2.2K, Resistor_SMD:R_0805_2012Metric, F.Cu at (40.0, 68.6)
- added R1223: 2.2K, Resistor_SMD:R_0805_2012Metric, F.Cu at (40.0, 77.5)
- added R1224: 2.2K, Resistor_SMD:R_0805_2012Metric, F.Cu at (40.0, 86.4)
- added R1225: 2.2K, Resistor_SMD:R_0805_2012Metric, F.Cu at (112.4, 59.7)
- added R1226: 2.2K, Resistor_SMD:R_0805_2012Metric, F.Cu at (112.4, 68.6)
- added R1227: 2.2K, Resistor_SMD:R_0805_2012Metric, F.Cu at (112.4, 77.5)
- added R1228: 2.2K, Resistor_SMD:R_0805_2012Metric, F.Cu at (112.4, 86.4)
- added R1229: 2.2K, Resistor_SMD:R_0805_2012Metric, F.Cu at (112.4, 54.6)
- added R1230: 2.2K, Resistor_SMD:R_0805_2012Metric, F.Cu at (112.4, 63.5)
- added R1231: 2.2K, Resistor_SMD:R_0805_2012Metric, F.Cu at (112.4, 72.4)
- added R1232: 2.2K, Resistor_SMD:R_0805_2012Metric, F.Cu at (112.4, 81.3)
- added R1301: 100R, Resistor_SMD:R_0805_2012Metric, F.Cu at (245.8, 79.8)
- added R1302: 1K, Resistor_SMD:R_0805_2012Metric, F.Cu at (245.8, 82.7)
- added R1303: 1K, Resistor_SMD:R_0805_2012Metric, F.Cu at (245.8, 85.7)
- added R1304: 1K, Resistor_SMD:R_0805_2012Metric, F.Cu at (245.8, 88.6)
- added R1305: 1K, Resistor_SMD:R_0805_2012Metric, F.Cu at (245.8, 91.6)
- added R1306: 2.2K, Resistor_SMD:R_0805_2012Metric, F.Cu at (245.8, 94.5)
- added R1501: 2.2K, Resistor_SMD:R_0805_2012Metric, F.Cu at (67.3, 59.7)
- added R1502: 2.2K, Resistor_SMD:R_0805_2012Metric, F.Cu at (67.3, 62.7)
- added R1503: 2.2K, Resistor_SMD:R_0805_2012Metric, F.Cu at (67.3, 65.6)
- added R1504: 2.2K, Resistor_SMD:R_0805_2012Metric, F.Cu at (67.3, 68.6)
- added R1505: 2.2K, Resistor_SMD:R_0805_2012Metric, F.Cu at (67.3, 71.5)
- added R1506: 2.2K, Resistor_SMD:R_0805_2012Metric, F.Cu at (71.7, 59.7)
- added R1507: 2.2K, Resistor_SMD:R_0805_2012Metric, F.Cu at (71.7, 62.7)
- added R1508: 2.2K, Resistor_SMD:R_0805_2012Metric, F.Cu at (71.7, 65.6)
- added R1509: 2.2K, Resistor_SMD:R_0805_2012Metric, F.Cu at (71.7, 68.6)
- added R1510: 2.2K, Resistor_SMD:R_0805_2012Metric, F.Cu at (71.7, 71.5)
- added R201: 100K, Resistor_SMD:R_0805_2012Metric, F.Cu at (184.9, 32.0)
- added R202: 100K, Resistor_SMD:R_0805_2012Metric, F.Cu at (44.8, 124.5)
- added R203: 100K, Resistor_SMD:R_0805_2012Metric, F.Cu at (40.0, 124.1)
- added R204: 100K, Resistor_SMD:R_0805_2012Metric, F.Cu at (131.6, 104.1)
- added R205: 22K, Resistor_SMD:R_0805_2012Metric, F.Cu at (184.9, 35.0)
- added R206: 52.3K, Resistor_SMD:R_0603_1608Metric, F.Cu at (185.8, 24.8)
- added R207: 10K, Resistor_SMD:R_0603_1608Metric, F.Cu at (185.8, 27.3)
- added R208: 100K, Resistor_SMD:R_0805_2012Metric, F.Cu at (83.8, 74.1)
- added R209: 100K, Resistor_SMD:R_0805_2012Metric, F.Cu at (162.5, 94.5)
- added R210: 100K, Resistor_SMD:R_0805_2012Metric, F.Cu at (162.5, 97.5)
- added R211: 100K, Resistor_SMD:R_0805_2012Metric, F.Cu at (166.9, 79.8)
- added R212: 100K, Resistor_SMD:R_0805_2012Metric, F.Cu at (70.6, 32.8)
- added R213: 100K, Resistor_SMD:R_0805_2012Metric, F.Cu at (68.1, 32.8)
- added R214: 100K, Resistor_SMD:R_0805_2012Metric, F.Cu at (65.5, 32.8)
- added R215: 100K, Resistor_SMD:R_0805_2012Metric, F.Cu at (63.0, 32.8)
- added R216: 100K, Resistor_SMD:R_0805_2012Metric, F.Cu at (60.5, 32.8)
- added R217: 100K, Resistor_SMD:R_0805_2012Metric, F.Cu at (57.9, 32.8)
- added R218: 100K, Resistor_SMD:R_0805_2012Metric, F.Cu at (171.3, 79.8)
- added R219: 100K, Resistor_SMD:R_0805_2012Metric, F.Cu at (171.3, 82.7)
- added R220: 10K, Resistor_SMD:R_0603_1608Metric, F.Cu at (183.9, 95.7)
- added R221: 10K, Resistor_SMD:R_0603_1608Metric, F.Cu at (183.9, 98.2)
- added R222: 10K, Resistor_SMD:R_0603_1608Metric, F.Cu at (183.9, 100.7)
- added R223: 10K, Resistor_SMD:R_0603_1608Metric, F.Cu at (183.9, 103.2)
- added R224: 10K, Resistor_SMD:R_0603_1608Metric, F.Cu at (70.6, 36.6)
- added R225: 10K, Resistor_SMD:R_0603_1608Metric, F.Cu at (68.1, 36.6)
- added R226: 10K, Resistor_SMD:R_0603_1608Metric, F.Cu at (65.5, 36.6)
- added R227: 10K, Resistor_SMD:R_0603_1608Metric, F.Cu at (63.0, 36.6)
- added R228: 10K, Resistor_SMD:R_0603_1608Metric, F.Cu at (60.5, 36.6)
- added R229: 10K, Resistor_SMD:R_0603_1608Metric, F.Cu at (57.9, 36.6)
- added R230: 10K, Resistor_SMD:R_0603_1608Metric, F.Cu at (187.9, 103.2)
- added R231: 10K, Resistor_SMD:R_0603_1608Metric, F.Cu at (187.9, 105.7)
- added R232: 100K, Resistor_SMD:R_0805_2012Metric, F.Cu at (171.3, 85.7)
- added R233: 100R, Resistor_SMD:R_0805_2012Metric, F.Cu at (171.3, 88.6)
- added R234: 1K, Resistor_SMD:R_0805_2012Metric, F.Cu at (171.3, 91.6)
- added R235: 1K, Resistor_SMD:R_0805_2012Metric, F.Cu at (171.3, 94.5)
- added R236: 1K, Resistor_SMD:R_0805_2012Metric, F.Cu at (171.3, 97.5)
- added R237: 1K, Resistor_SMD:R_0805_2012Metric, F.Cu at (175.7, 79.8)
- added R238: 1K, Resistor_SMD:R_0805_2012Metric, F.Cu at (175.7, 82.7)
- added R239: 1K, Resistor_SMD:R_0805_2012Metric, F.Cu at (175.7, 85.7)
- added R301: 2.2K, Resistor_SMD:R_0805_2012Metric, F.Cu at (91.4, 96.3)
- added R302: 10K, Resistor_SMD:R_0603_1608Metric, F.Cu at (222.8, 108.9)
- added R501: 10K, Resistor_SMD:R_0603_1608Metric, B.Cu at (79.4, 98.6)
- added R502: 10K, Resistor_SMD:R_0603_1608Metric, B.Cu at (81.9, 98.6)
- added R503: 10K, Resistor_SMD:R_0603_1608Metric, B.Cu at (84.5, 98.6)
- added R601: 10K, Resistor_SMD:R_0603_1608Metric, B.Cu at (70.0, 93.3)
- added R602: 10K, Resistor_SMD:R_0603_1608Metric, B.Cu at (70.0, 95.8)
- added R603: 10K, Resistor_SMD:R_0603_1608Metric, B.Cu at (70.0, 98.3)
- added R701: 47K, Resistor_SMD:R_0805_2012Metric, B.Cu at (94.7, 93.0)
- added R702: 47K, Resistor_SMD:R_0805_2012Metric, B.Cu at (94.7, 95.0)
- added R703: 47K, Resistor_SMD:R_0805_2012Metric, B.Cu at (94.7, 107.7)
- added R704: 47K, Resistor_SMD:R_0805_2012Metric, B.Cu at (94.7, 109.7)
- added R705: 47K, Resistor_SMD:R_0805_2012Metric, B.Cu at (94.7, 111.8)
- added R706: 2.2K, Resistor_SMD:R_0805_2012Metric, B.Cu at (94.7, 105.7)
- added R707: 2.2K, Resistor_SMD:R_0805_2012Metric, B.Cu at (94.7, 90.9)
- added R801: 5.1K, Resistor_SMD:R_0603_1608Metric, B.Cu at (31.1, 97.8)
- added R802: 5.1K, Resistor_SMD:R_0603_1608Metric, B.Cu at (31.1, 100.3)
- added SW1301: SW_USER, Button_Switch_THT:SW_PUSH_6mm_H5mm, F.Cu at (255.7, 80.3)
- added SW201: START, Button_Switch_THT:SW_PUSH_6mm_H5mm, F.Cu at (165.7, 23.0)
- added SW301: RESET, Button_Switch_THT:SW_PUSH_6mm_H5mm, F.Cu at (226.8, 104.7)
- added SYM101: ~, leptunKicadLib:AMOGUS_exposed_copper, F.Cu at (76.2, 91.9)
- added TP1001: ~, TestPoint:TestPoint_Pad_D2.0mm, F.Cu at (214.8, 133.4)
- added TP201: ~, TestPoint:TestPoint_Pad_D2.0mm, F.Cu at (135.9, 103.1)
- added TP202: ~, TestPoint:TestPoint_Pad_D2.0mm, F.Cu at (45.5, 115.9)
- added TP203: ~, TestPoint:TestPoint_Pad_D2.0mm, F.Cu at (41.9, 20.3)
- added TP204: ~, TestPoint:TestPoint_Pad_D2.0mm, F.Cu at (88.1, 73.1)
- added TP205: ~, TestPoint:TestPoint_Pad_D2.0mm, F.Cu at (200.0, 114.5)
- added TP206: ~, TestPoint:TestPoint_Pad_D2.0mm, F.Cu at (207.0, 28.6)
- added TP207: ~, TestPoint:TestPoint_Pad_D2.0mm, F.Cu at (204.1, 114.5)
- added TP208: ~, TestPoint:TestPoint_Pad_D2.0mm, F.Cu at (204.1, 118.6)
- added TP801: ~, TestPoint:TestPoint_Pad_D2.0mm, F.Cu at (265.8, 65.7)
- added U1001: MAX-M10S, RF_GPS:ublox_MAX, F.Cu at (32.3, 45.7)
- added U1501: ICM-20948, Sensor_Motion:InvenSense_QFN-24_3x3mm_P0.4mm, F.Cu at (76.2, 76.2)
- added U201: AP2112K-3.3, Package_TO_SOT_SMD:SOT-23-5, F.Cu at (136.4, 98.9)
- added U202: AOZ1212AI, leptunKicadLib:AOZ1212AI, F.Cu at (178.5, 33.8)
- added U203: AP2151W, Package_TO_SOT_SMD:SOT-23-5, F.Cu at (40.4, 120.4)
- added U204: AP2112K-3.3, Package_TO_SOT_SMD:SOT-23-5, F.Cu at (42.5, 16.1)
- added U205: AP2112K-1.8, Package_TO_SOT_SMD:SOT-23-5, F.Cu at (88.6, 68.8)
- added U206: AP2112K-3.3, Package_TO_SOT_SMD:SOT-23-5, F.Cu at (185.6, 114.2)
- added U207: AP2112K-3.3, Package_TO_SOT_SMD:SOT-23-5, F.Cu at (207.6, 24.3)
- added U208: AP2171W, Package_TO_SOT_SMD:SOT-23-5, F.Cu at (185.6, 123.1)
- added U301: STM32F722ZETx, Package_QFP:LQFP-144_20x20mm_P0.5mm, F.Cu at (76.2, 91.9)
- added U501: W25Q128JVS, Package_SO:SOIC-8_5.23x5.23mm_P1.27mm, B.Cu at (81.9, 91.4)
- added U502: W25Q128JVPM, Package_SON:WSON-8-1EP_6x5mm_P1.27mm_EP3.4x4.3mm, B.Cu at (81.9, 91.4)
- added U601: W25Q128JVS, Package_SO:SOIC-8_5.23x5.23mm_P1.27mm, B.Cu at (73.2, 86.4)
- added U602: W25Q128JVPM, Package_SON:WSON-8-1EP_6x5mm_P1.27mm_EP3.4x4.3mm, B.Cu at (73.2, 86.4)
- added U801: USBLC6-2SC6, Package_TO_SOT_SMD:SOT-23-6, F.Cu at (39.2, 99.1)
- added Y301: 24MHz, leptunKicadLib:ATS240C, F.Cu at (91.4, 89.4)
Routing:
- net /MCU/LOOP: track 0.00 -> 1685.9 mm, vias 0 -> 6
- net GND: track 0.00 -> 4.16 mm
- net Net-(U301-PC15): track 0.00 -> 3.84 mm
- added copper zone on B.Cu, net GND
- added copper zone on F.Cu, net GND
- added copper zone on In1.Cu, net GND
- added copper zone on In2.Cu, net GND

Commit message: Checkpoint
Parts:
- moved U203 25.0 mm to (16.2, 126.7)
- moved C204 25.0 mm to (20.8, 125.8)
- moved C212 25.0 mm to (20.8, 128.3)
- moved R202 25.0 mm to (20.7, 130.8)
- moved C214 25.0 mm to (16.5, 122.4)
- moved R203 25.0 mm to (15.9, 130.4)
- moved TP202 25.0 mm to (21.3, 122.3)
Connections:
- U301 pad 75: /MCU/USB_OTG_HS_DM -> /USB_D-
- U301 pad 76: /MCU/USB_OTG_HS_DP -> /USB_D+
- U801 pad 1: /MCU/USB_OTG_HS_DM -> /USB_D+
- U801 pad 3: /MCU/USB_OTG_HS_DP -> /USB_D-
- U801 pad 4: /USB/CONN_D+ -> /USB/CONN_D-
- U801 pad 6: /USB/CONN_D- -> /USB/CONN_D+
Routing:
- net /USB_D-: track 0.00 -> 31.5 mm
- net /USB_D+: track 0.00 -> 31.5 mm
- net unconnected-(J801-SHIELD-PadS1): track 0.00 -> 30.0 mm
- net /USB/CONN_D-: track 0.00 -> 8.54 mm, vias 0 -> 2
- net /USB/CONN_D+: track 0.00 -> 8.54 mm, vias 0 -> 2
- net Net-(J801-CC2): track 0.00 -> 2.54 mm, vias 0 -> 1
- net Net-(J801-CC1): track 0.00 -> 2.23 mm, vias 0 -> 1

Commit message: Checkpoint
Parts:
- moved J204 140.5 mm to (91.4, 37.1)
- moved C206 106.0 mm to (77.4, 33.4), turned to 180 degrees
- moved C208 105.4 mm to (82.0, 40.7)
- moved C219 104.8 mm to (76.2, 46.0), turned to 180 degrees
- moved R206 101.5 mm to (85.4, 39.9), turned to 90 degrees
- moved R207 98.8 mm to (87.7, 39.2)
- moved C207 98.8 mm to (88.6, 35.0), turned to -90 degrees
- moved R205 98.6 mm to (86.4, 34.3), turned to 180 degrees
- moved J203 97.5 mm to (90.7, 48.8), turned to 180 degrees
- moved U202 96.6 mm to (81.9, 36.2), turned to 90 degrees
- moved D202 96.5 mm to (75.2, 39.4), turned to 90 degrees
- moved C205 87.7 mm to (89.7, 30.5)
- moved L201 87.2 mm to (82.2, 45.9), turned to -90 degrees
- moved R201 86.0 mm to (99.1, 37.1), turned to 180 degrees
- moved D201 81.6 mm to (103.5, 35.6), turned to 180 degrees
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
Commit message: Checkpoint
Parts:
- removed the J201 at (73.2, 29.2)
- removed the R214 at (65.5, 32.8)
- removed the R216 at (60.5, 32.8)
- removed the R218 at (171.3, 79.8)
- removed the R219 at (171.3, 82.7)
- removed the R224 at (70.6, 36.6)
- removed the R225 at (68.1, 36.6)
- removed the R226 at (65.5, 36.6)
- removed the R227 at (63.0, 36.6)
- removed the R228 at (60.5, 36.6)
- added C220: 100nF, Capacitor_SMD:C_0603_1608Metric, F.Cu at (152.7, 155.0)
- added C221: 100nF, Capacitor_SMD:C_0603_1608Metric, F.Cu at (152.7, 157.5)
- added C223: 1nF, Capacitor_SMD:C_0603_1608Metric, F.Cu at (152.7, 160.0)
- added C224: 1nF, Capacitor_SMD:C_0603_1608Metric, F.Cu at (152.7, 162.5)
- added R211: 10K, Resistor_SMD:R_0603_1608Metric, F.Cu at (152.7, 165.0)
- added R220: 10K, Resistor_SMD:R_0603_1608Metric, F.Cu at (156.7, 162.5)
- added R221: 10K, Resistor_SMD:R_0603_1608Metric, F.Cu at (156.7, 165.0)
- added R222: 15K, Resistor_SMD:R_1206_3216Metric, F.Cu at (153.5, 167.9)
- added R223: 15K, Resistor_SMD:R_1206_3216Metric, F.Cu at (153.5, 171.2)
- added TP207: ~, TestPoint:TestPoint_Pad_D2.0mm, F.Cu at (160.7, 155.7)
- added TP209: ~, TestPoint:TestPoint_Pad_D2.0mm, F.Cu at (160.7, 159.8)
- added U1101: USBLC6-4SC6, Package_TO_SOT_SMD:SOT-23-6, F.Cu at (72.1, 151.0)
- added U1201: USBLC6-4SC6, Package_TO_SOT_SMD:SOT-23-6, F.Cu at (64.9, 140.1)
- added U1202: USBLC6-4SC6, Package_TO_SOT_SMD:SOT-23-6, F.Cu at (64.9, 144.6)
- added U1203: USBLC6-4SC6, Package_TO_SOT_SMD:SOT-23-6, F.Cu at (64.9, 149.0)
- added U1204: USBLC6-4SC6, Package_TO_SOT_SMD:SOT-23-6, F.Cu at (64.9, 153.5)
- added U1401: USBLC6-4SC6, Package_TO_SOT_SMD:SOT-23-6, F.Cu at (79.2, 140.1)
- added U208: ACS714xLCTR-50A, Package_SO:SOIC-8_3.9x4.9mm_P1.27mm, F.Cu at (146.4, 156.9)
- added U209: ACS714xLCTR-50A, Package_SO:SOIC-8_3.9x4.9mm_P1.27mm, F.Cu at (146.4, 163.4)
- added U401: USBLC6-4SC6, Package_TO_SOT_SMD:SOT-23-6, F.Cu at (72.1, 140.1)
- added U402: USBLC6-4SC6, Package_TO_SOT_SMD:SOT-23-6, F.Cu at (72.1, 144.6)
- R212, R213, R215: value 100K -> 10K; footprint Resistor_SMD:R_0805_2012Metric -> Resistor_SMD:R_0603_1608Metric
- moved R215 158.0 mm to (156.7, 160.0), turned to 0 degrees
- moved R213 153.0 mm to (156.7, 157.5), turned to 0 degrees
- moved R212 149.5 mm to (156.7, 155.0), turned to 0 degrees
- moved R214 32.5 mm to (90.4, 38.1)
- moved R210 31.8 mm to (89.6, 35.6), turned to 0 degrees
- moved J1207 11.2 mm to (59.5, 36.1)
- moved Q1207 11.2 mm to (62.0, 39.4)
- moved R1211 11.2 mm to (64.5, 39.7)
- moved R1215 11.2 mm to (59.4, 39.7)
- moved C202 5.38 mm to (93.7, 35.0)
- moved C207 5.38 mm to (83.3, 35.1)
- moved C208 5.38 mm to (76.7, 40.8)
- moved C219 5.38 mm to (70.8, 46.0)
- moved J201 5.38 mm to (85.3, 48.8)
- moved J203 5.38 mm to (73.4, 29.3)
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- renumbered C220 to C222, C221 to C225, C222 to C226, J203 to J201, J204 to J202, J202 to J203, R217 to R210, R229 to R214, R230 to R216, R231 to R217, R210 to R218, R211 to R219, R220 to R224, R221 to R225, R222 to R226, R223 to R227, R232 to R228, R233 to R229, R234 to R230, R235 to R231, R236 to R232, R237 to R233, R238 to R234, R239 to R235, TP207 to TP210, U208 to U210
Connections:
- J1201 pad 2: /POWER/SERVO_5V5 -> /POWER/SERVO_ESC
- J201 pad 1: /POWER/D1_5V -> Net-(J201-Pin_1)
- J201 pad 3: /POWER/D1_5V -> Net-(J201-Pin_1)
- J201 pad 5: /POWER/D1_5V -> Net-(J201-Pin_1)
- J401 pad 11: unconnected-(J401-Pin_11-Pad11) -> /DEBUG/GNDDetect
- R1205 pad 2: /POWER/SERVO_5V5 -> /POWER/SERVO_ESC
- R210 pad 1: /POWER/BATT_S6 -> /POWER/PWR_IN
- R210 pad 2: /POWER/MEAS_S6 -> /MCU/ADC2_IN10
- R212 pad 1: /POWER/MEAS_S1 -> /POWER/SERVO_5V5
- R212 pad 2: /POWER/BATT_S1 -> /MCU/ADC3_IN15
- R213 pad 1: /POWER/BATT_S2 -> /POWER/D1_5V
- R213 pad 2: /POWER/MEAS_S2 -> /MCU/ADC2_IN12
- R214 pad 1: /POWER/MEAS_S6 -> /MCU/ADC2_IN10
- R215 pad 1: /POWER/BATT_S4 -> /MCU/ADC1_IN14
- R215 pad 2: /POWER/MEAS_S4 -> GND
- R216 pad 1: /MCU/ADC2_IN12 -> /MCU/ADC3_IN15
- R217 pad 1: /MCU/ADC2_IN13 -> /MCU/ADC2_IN12
- R224 pad 2: /MCU/ADC1_IN8 -> /MCU/ADC2_IN13
- R225 pad 2: /MCU/ADC1_IN9 -> /MCU/ADC3_IN8
- R226 pad 2: /MCU/ADC1_IN14 -> /MCU/ADC3_IN9
- R227 pad 2: /MCU/ADC1_IN15 -> /MCU/ADC3_IN14
- U301 pad 104: unconnected-(U301-PA12-Pad104) -> /DEBUG/GNDDetect
- U301 pad 13: /POWER/MEAS_S6 -> /MCU/ADC3_IN9
- U301 pad 14: /POWER/MEAS_S5 -> /MCU/ADC3_IN14
- U301 pad 15: /POWER/MEAS_S4 -> /MCU/ADC3_IN15
- U301 pad 22: /POWER/MEAS_S3 -> /MCU/ADC3_IN8
- U301 pad 26: /POWER/MEAS_S2 -> /MCU/ADC2_IN10
- U301 pad 27: /POWER/MEAS_S1 -> /MCU/ADC2_IN11
- U301 pad 46: /MCU/ADC1_IN8 -> unconnected-(U301-PB0-Pad46)
- U301 pad 47: /MCU/ADC1_IN9 -> unconnected-(U301-PB1-Pad47)

Commit message: Checkpoint
Parts:
- added J901: ~, Connector_Coaxial:SMA_Amphenol_132134_Vertical, F.Cu at (121.4, 46.2)
- added TP301: ~, TestPoint:TestPoint_Pad_D1.0mm, F.Cu at (146.3, 70.4)
- added TP302: ~, TestPoint:TestPoint_Pad_D1.0mm, F.Cu at (146.3, 73.4)
- added TP303: ~, TestPoint:TestPoint_Pad_D1.0mm, F.Cu at (146.3, 76.5)
- added TP304: ~, TestPoint:TestPoint_Pad_D1.0mm, F.Cu at (149.3, 70.4)
- added TP305: ~, TestPoint:TestPoint_Pad_D1.0mm, F.Cu at (149.3, 73.4)
- added TP306: ~, TestPoint:TestPoint_Pad_D1.0mm, F.Cu at (149.3, 76.5)
- added TP307: ~, TestPoint:TestPoint_Pad_D1.0mm, F.Cu at (152.4, 70.4)
- added TP308: ~, TestPoint:TestPoint_Pad_D1.0mm, F.Cu at (152.4, 73.4)
- added TP309: ~, TestPoint:TestPoint_Pad_D1.0mm, F.Cu at (152.4, 76.5)
- added TP310: ~, TestPoint:TestPoint_Pad_D1.0mm, F.Cu at (155.4, 70.4)
- added TP311: ~, TestPoint:TestPoint_Pad_D1.0mm, F.Cu at (155.4, 73.4)
- added TP312: ~, TestPoint:TestPoint_Pad_D1.0mm, F.Cu at (155.4, 76.5)
- added U901: LAMBDA62, leptunKicadLib:LAMBDA62, F.Cu at (107.2, 37.4)
- TP1001, TP201, TP202, TP203, TP204, TP205, TP206, TP207, TP208, TP209, TP210, TP801: footprint TestPoint:TestPoint_Pad_D2.0mm -> TestPoint:TestPoint_Pad_D1.0mm
- moved TP1001 208.8 mm to (28.6, 38.8)
- moved C205 4.59 mm to (79.7, 30.5)
- moved C206 4.59 mm to (67.4, 33.4)
- moved D201 4.59 mm to (93.5, 35.6)
- moved D202 4.59 mm to (65.2, 39.4)
- moved J1207 4.59 mm to (54.9, 36.1)
- moved J201 4.59 mm to (80.7, 48.8)
- moved J202 4.59 mm to (81.5, 37.1)
- moved L201 4.59 mm to (72.3, 45.9)
- moved R1211 4.59 mm to (59.9, 39.7)
- moved R1215 4.59 mm to (54.8, 39.7)
- moved R205 4.59 mm to (76.4, 34.3)
- moved R206 4.59 mm to (75.5, 39.9)
- moved R207 4.59 mm to (77.7, 39.2)
- moved R210 4.59 mm to (85.0, 35.6)
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Connections:
- U301 pad 1: unconnected-(U301-PE2-Pad1) -> Net-(U301-PE2)
- U301 pad 119: unconnected-(U301-PD5-Pad119) -> Net-(U301-PD5)
- U301 pad 134: unconnected-(U301-PB4-Pad134) -> Net-(U301-PB4)
- U301 pad 135: unconnected-(U301-PB5-Pad135) -> Net-(U301-PB5)
- U301 pad 137: unconnected-(U301-PB7-Pad137) -> Net-(U301-PB7)
- U301 pad 139: unconnected-(U301-PB8-Pad139) -> Net-(U301-PB8)
- U301 pad 46: unconnected-(U301-PB0-Pad46) -> Net-(U301-PB0)
- U301 pad 47: unconnected-(U301-PB1-Pad47) -> Net-(U301-PB1)
- U301 pad 87: unconnected-(U301-PG2-Pad87) -> Net-(U301-PG2)
- U301 pad 88: unconnected-(U301-PG3-Pad88) -> Net-(U301-PG3)
- U301 pad 92: unconnected-(U301-PG7-Pad92) -> Net-(U301-PG7)
- U301 pad 93: unconnected-(U301-PG8-Pad93) -> Net-(U301-PG8)
Routing:
- net /MCU/LOOP: track 1685.9 -> 1653.7 mm, vias 6 -> 4
- net Net-(U1001-~{SAFEBOOT}): track 0.00 -> 2.47 mm
- net /GPS/SCL: track 0.00 -> 1.30 mm, vias 0 -> 1
- net /GPS/SDA: track 0.00 -> 1.26 mm, vias 0 -> 1
- net GND: vias 0 -> 26

Commit message: Checkpoint routing
Parts:
- C301, C302, C310, C311, C314, C315, C317, C318, C319, C320, R1507, R1509, R1510: moved to B.Cu
- SYM101: footprint leptunKicadLib:AMOGUS_exposed_copper -> leptunKicadLib:AMOGUS
- moved SW1301 215.8 mm to (45.0, 33.6)
- moved R1306 211.1 mm to (42.4, 37.8), turned to -90 degrees
- moved SW301 192.6 mm to (45.0, 41.2)
- moved C226 158.6 mm to (54.2, 174.2)
- moved TP210 156.1 mm to (62.2, 179.6)
- moved U210 143.4 mm to (54.1, 180.3)
- moved C222 143.2 mm to (58.7, 179.4)
- moved C225 143.2 mm to (58.7, 181.9)
- moved R219 141.8 mm to (61.6, 174.7)
- moved R302 140.9 mm to (82.0, 105.2), turned to -90 degrees
- moved C319 139.5 mm to (84.8, 85.9)
- moved C217 129.1 mm to (89.6, 177.1)
- moved R218 125.3 mm to (61.6, 171.7)
- moved TP205 124.5 mm to (93.3, 178.6)
- moved C211 120.4 mm to (89.6, 174.1)
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Routing:
- net /DEBUG/T_VCC: track 0.00 -> 47.1 mm, vias 0 -> 6
- net GND: track 4.16 -> 33.7 mm, vias 26 -> 29
- net /IMU/VDD_1V8: track 0.00 -> 12.2 mm
- net /IMU/SDI_VIO: track 0.00 -> 11.7 mm
- net /MCU/QUADSPI_BK2_IO0: track 0.00 -> 9.98 mm, vias 0 -> 2
- net /MCU/QUADSPI_BK1_IO3: track 0.00 -> 9.78 mm, vias 0 -> 1
- net /MCU/QUADSPI_BK2_IO2: track 0.00 -> 9.64 mm, vias 0 -> 1
- net /IMU/SCLK_VIO: track 0.00 -> 9.00 mm
- net /MCU/QUADSPI_BK2_IO3: track 0.00 -> 8.91 mm, vias 0 -> 1
- net /MCU/QUADSPI_BK1_IO2: track 0.00 -> 8.67 mm, vias 0 -> 1
- net /MCU/QUADSPI_BK1_IO1: track 0.00 -> 7.26 mm, vias 0 -> 1
- net Net-(U301-PH1): track 0.00 -> 7.14 mm
- net Net-(U301-PH0): track 0.00 -> 7.12 mm
- net /IMU/NCS_VIO: track 0.00 -> 6.76 mm
- net /MCU/QUADSPI_BK2_IO1: track 0.00 -> 6.51 mm, vias 0 -> 1
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
Commit message: Checkpoint routing
Parts:
- moved R222 143.5 mm to (87.6, 40.4)
- moved R220 142.0 mm to (84.6, 40.1), turned to 90 degrees
- moved C223 130.1 mm to (90.7, 45.6), turned to -90 degrees
- moved C220 128.4 mm to (90.7, 42.5), turned to -90 degrees
- moved U208 127.7 mm to (86.2, 44.3)
- moved R223 79.2 mm to (98.2, 114.6)
- moved R221 75.6 mm to (98.0, 117.2), turned to 90 degrees
- moved C224 69.8 mm to (99.6, 117.2), turned to 90 degrees
- moved C221 69.1 mm to (96.5, 117.2), turned to -90 degrees
- moved U1202 67.3 mm to (121.7, 108.5), turned to 90 degrees
- moved U209 62.8 mm to (98.8, 122.4), turned to 90 degrees
- moved U1201 54.7 mm to (109.5, 108.5), turned to 90 degrees
- moved U1101 45.1 mm to (56.6, 108.7), turned to 90 degrees
- moved U1401 27.6 mm to (76.2, 112.7)
- moved J1201 4.35 mm to (103.4, 125.0)
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Connections:
- TP209 pad 1: /POWER/SERVO_ESC -> /POWER/SERVO_5V5
- U1401 pad 4: /GPS/SCL -> /GPS/SDA
- U1401 pad 6: /GPS/SDA -> /GPS/SCL
- U209 pad 1: /POWER/SERVO_ESC -> /POWER/SERVO_5V5
- U209 pad 2: /POWER/SERVO_ESC -> /POWER/SERVO_5V5
- U209 pad 3: /POWER/SERVO_5V5 -> /POWER/SERVO_ESC
- U209 pad 4: /POWER/SERVO_5V5 -> /POWER/SERVO_ESC
Routing:
- net /DEBUG/T_VCC: track 47.1 -> 103.5 mm, vias 6 -> 7
- net /POWER/SERVO_5V5: track 0.00 -> 40.6 mm, vias 0 -> 2
- net /SERVO/CH7_OUT: track 0.00 -> 37.4 mm
- net /MCU/SDMMC2_D2: track 0.00 -> 28.1 mm, vias 0 -> 1
- net /MCU/SDMMC2_CK: track 0.00 -> 27.2 mm, vias 0 -> 1
- net /MCU/SDMMC2_D1: track 0.00 -> 26.5 mm, vias 0 -> 1
- net /MCU/SDMMC2_D0: track 0.00 -> 26.4 mm, vias 0 -> 1
- net /MCU/SDMMC2_CMD: track 0.00 -> 25.8 mm, vias 0 -> 1
- net /MCU/SDMMC2_D3: track 0.00 -> 25.4 mm, vias 0 -> 1
- net /SERVO/CH3_OUT: track 0.00 -> 18.6 mm
- net Net-(J201-Pin_1): track 0.00 -> 17.1 mm
- net /SERVO/CH0_OUT: track 0.00 -> 15.9 mm
- net /SERVO/CH2_OUT: track 0.00 -> 14.1 mm
- net /SERVO/CH1_OUT: track 0.00 -> 13.9 mm
- net Net-(J1102-Pin_3): track 0.00 -> 13.5 mm
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
Commit message: Checkpoint routing
Parts:
- TP202, U1203, U1204: moved to B.Cu
- moved D1301 227.2 mm to (29.1, 129.8)
- moved D1302 227.2 mm to (29.1, 133.2)
- moved D1303 227.2 mm to (29.1, 136.6)
- moved D1304 227.2 mm to (29.1, 140.0)
- moved R1302 216.8 mm to (34.1, 129.6)
- moved R1303 216.8 mm to (34.1, 132.5)
- moved R1304 216.8 mm to (34.1, 135.5)
- moved R1305 216.8 mm to (34.1, 138.4)
- moved C211 162.2 mm to (110.2, 13.2)
- moved TP205 162.2 mm to (113.9, 17.7)
- moved U206 162.2 mm to (115.0, 13.9)
- moved C217 162.2 mm to (110.2, 16.2)
- moved R209 162.2 mm to (110.1, 19.2)
- moved C222 110.8 mm to (17.9, 76.3)
- moved C225 110.8 mm to (17.9, 78.8)
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Connections:
- U1203 pad 1: /SERVO/CH8_OUT -> /SERVO/CH11_OUT
- U1203 pad 3: /SERVO/CH9_OUT -> /SERVO/CH10_OUT
- U1203 pad 4: /SERVO/CH10_OUT -> /SERVO/CH9_OUT
- U1203 pad 6: /SERVO/CH11_OUT -> /SERVO/CH8_OUT
- U401 pad 1: /DEBUG/GNDDetect -> /DEBUG/T_VCP_RX
- U401 pad 3: /DEBUG/T_VCP_RX -> /DEBUG/T_VCP_TX
- U401 pad 4: /DEBUG/T_NRST  -> /DEBUG/T_JTDI
- U401 pad 6: /DEBUG/T_VCP_TX -> /DEBUG/T_NRST 
- U402 pad 1: /DEBUG/T_JTDI -> /DEBUG/GNDDetect
- U402 pad 3: /DEBUG/T_JTDO/T_SWO -> /DEBUG/T_JTMS/T_SWDIO
- U402 pad 4: /DEBUG/T_JTMS/T_SWDIO -> /DEBUG/T_JCLK/T_SWCLK
- U402 pad 6: /DEBUG/T_JCLK/T_SWCLK -> /DEBUG/T_JTDO/T_SWO
Routing:
- net /SERVO/CH15_OUT: track 0.00 -> 16.6 mm
- net /SERVO/CH8_OUT: track 0.00 -> 16.6 mm
- net /SERVO/CH12_OUT: track 0.00 -> 11.5 mm
- net /SERVO/CH11_OUT: track 0.00 -> 11.5 mm
- net /DEBUG/GNDDetect: track 0.00 -> 11.1 mm
- net /DEBUG/T_VCP_RX: track 0.00 -> 10.4 mm
- net /GPS/SCL: track 10.9 -> 1.30 mm
- net /DEBUG/T_JCLK/T_SWCLK: track 0.00 -> 9.08 mm
- net /DEBUG/T_VCP_TX: track 0.00 -> 7.48 mm
- net /SERVO/CH9_OUT: track 0.00 -> 6.97 mm
- net /SERVO/CH14_OUT: track 0.00 -> 6.97 mm
- net /GPS/SDA: track 7.54 -> 1.26 mm
- net /DEBUG/T_JTMS/T_SWDIO: track 0.00 -> 6.00 mm
- net /LIDAR/RX: track 5.78 -> 0.00 mm
- net /LIDAR/VDD: track 4.52 -> 0.00 mm
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