File: Hardware/Avionus_Flight_Controller.kicad_pcb (KiCad board)
At the start: 4 copper layers, 101.6 x 101.6 mm, 283 parts, among them J1101 PPM, J1102 iBUS, J1201 S0, J1202 S1, J1203 S2, J1204 S3, J1205 S4, J1206 S5, J1207 S6, J1208 S7, J1209 S8, J1210 S9, J1211 S10, J1212 S11, J1213 S12, J1214 S13, J1215 S14, J1216 S15, J1401 LIDAR, J201 5V_SEL, J202 E5V, J203 POWER IN, J401 STDC14, J701 SD_Card, J801 USB_C_Receptacle_USB2.0, Q1101 RE1C002UN, Q1102 RE1C002UN, Q1201 RE1C002UN, Q1202 RE1C002UN, Q1203 RE1C002UN, Q1204 RE1C002UN, Q1205 RE1C002UN, Q1206 RE1C002UN, Q1207 RE1C002UN, Q1208 RE1C002UN, Q1209 RE1C002UN, Q1210 RE1C002UN, Q1211 RE1C002UN, Q1212 RE1C002UN, Q1213 RE1C002UN, Q1214 RE1C002UN, Q1215 RE1C002UN, Q1216 RE1C002UN, Q1301 RE1C002UN, Q1501 RE1C002UN, Q1502 RE1C002UN, Q1503 RE1C002UN, Q1504 RE1C002UN, Q1505 RE1C002UN, Q201 RE1C002UN, SW1301 SW_USER, SW201 START, SW301 RESET, U1001 MAX-M10S, U1101 USBLC6-4SC6, U1201 USBLC6-4SC6, U1202 USBLC6-4SC6, U1203 USBLC6-4SC6, U1204 USBLC6-4SC6, U1401 USBLC6-4SC6, U1501 ICM-20948, U201 AP2112K-3.3, U202 AOZ1212AI, U203 AP2151W, U204 AP2112K-3.3, U205 AP2112K-1.8, U206 AP2112K-3.3, U207 AP2112K-3.3, U208 ACS714xLCTR-50A, U209 ACS714xLCTR-50A, U210 AP2171W, U301 STM32F722ZETx, U401 USBLC6-4SC6, U402 USBLC6-4SC6, U501 W25Q128JVS, U502 W25Q128JVPM, U601 W25Q128JVS, U602 W25Q128JVPM, U801 USBLC6-2SC6, U901 LAMBDA62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

Commit message: Finalize schematic and some more routing
Parts:
- added BZ1301: Buzzer, Buzzer_Beeper:Buzzer_12x9.5RM7.6, F.Cu at (242.6, 91.4)
- C211, C217, D1301, D1302, D1303, D1304, D206, R1302, R1303, R1304, R1305, R209, R233, TP205, U206: moved to B.Cu
- R1301, R229: value 100R -> 150R; footprint Resistor_SMD:R_0805_2012Metric -> Resistor_SMD:R_0603_1608Metric
- moved D1304 139.6 mm to (111.8, 27.4)
- moved D1303 134.2 mm to (107.2, 27.4)
- moved R1305 133.7 mm to (111.8, 29.6)
- moved D1302 128.8 mm to (102.6, 27.4)
- moved R1304 128.6 mm to (107.2, 29.6)
- moved R1303 123.6 mm to (102.6, 29.6)
- moved D1301 123.4 mm to (98.0, 27.4)
- moved R1302 118.7 mm to (98.0, 29.6)
- moved D203 104.0 mm to (88.3, 48.3), turned to 180 degrees
- moved R230 103.2 mm to (84.2, 48.0)
- moved D205 98.1 mm to (103.9, 98.4)
- moved R232 92.1 mm to (104.6, 101.3), turned to 90 degrees
- moved D206 85.1 mm to (110.6, 35.2)
- moved R233 80.4 mm to (111.3, 37.3)
- moved U207 40.0 mm to (84.5, 55.7)
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Routing:
- net GND: track 37.4 -> 51.3 mm, vias 29 -> 32
- net /POWER/D4_3V3: track 0.00 -> 11.2 mm, vias 0 -> 1
- net /POWER/D3_3V3: track 1.60 -> 11.9 mm, vias 0 -> 1
- net /POWER/D1_5V: track 5.73 -> 9.55 mm
- net Net-(D1302-A): track 0.00 -> 2.36 mm
- net Net-(D1304-A): track 0.00 -> 2.36 mm
- net Net-(D1303-A): track 0.00 -> 2.36 mm
- net Net-(D1301-A): track 0.00 -> 2.36 mm
- net Net-(D205-A): track 0.00 -> 2.27 mm
- net Net-(D206-A): track 0.00 -> 2.22 mm
- net /MCU/GPIO_PF12: track 0.00 -> 1.81 mm
- net /MCU/GPIO_PG15: track 0.00 -> 1.81 mm

Commit message: Misc routing
Parts:
- removed TP209: ~, TestPoint:TestPoint_Pad_D1.0mm
- added R303: 10K, Resistor_SMD:R_0603_1608Metric, F.Cu at (91.6, 96.3)
- C222, C225, Q1301, R1301, R211, R212, R215, R216, R218, R219, R224, R226, R227, U210: moved to B.Cu
- R301: value 2.2K -> 10K; footprint Resistor_SMD:R_0805_2012Metric -> Resistor_SMD:R_0603_1608Metric
- moved R1301 184.9 mm to (61.6, 59.1), turned to 90 degrees
- moved BZ1301 183.0 mm to (63.5, 54.0), turned to -90 degrees
- moved Q1301 182.9 mm to (63.5, 59.1), turned to -90 degrees
- moved D204 150.4 mm to (42.3, 41.9), turned to -90 degrees
- moved R231 148.5 mm to (39.4, 43.9)
- moved D207 140.4 mm to (59.6, 108.3), turned to -90 degrees
- moved TP208 138.7 mm to (83.5, 50.0)
- moved Q201 136.3 mm to (54.7, 42.7), turned to -90 degrees
- moved R234 132.0 mm to (62.5, 109.7), turned to 180 degrees
- moved R228 131.9 mm to (55.2, 44.8), turned to 180 degrees
- moved TP207 131.3 mm to (80.7, 51.6)
- moved R229 130.4 mm to (56.6, 42.3), turned to 90 degrees
- moved R213 126.1 mm to (80.9, 56.6), turned to 180 degrees
- moved R224 119.5 mm to (66.5, 72.9), turned to -90 degrees
- moved R216 119.4 mm to (68.8, 111.5), turned to -90 degrees
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Connections:
- R212 pad 1: /POWER/SERVO_5V5 -> /LIDAR/VDD
- R301 pad 2: Net-(U301-PC15) -> Net-(U301-PC14)
- U301 pad 8: /MCU/LOOP -> Net-(U301-PC14)
Routing:
- net /IMU/VDD_1V8: track 12.2 -> 51.1 mm
- net /POWER/D1_5V: track 9.55 -> 15.8 mm
- net /MCU/LOOP: track 1653.7 -> 1648.3 mm
- net /IMU/SDO_VIO: track 6.03 -> 1.72 mm
- net Net-(U301-PC14): track 0.00 -> 4.13 mm
- net Net-(J201-Pin_1): track 17.1 -> 19.9 mm
- net /POWER/D4_3V3: track 11.2 -> 12.9 mm
- net /POWER/D3_3V3: track 11.9 -> 13.6 mm
- net GND: track 51.3 -> 49.9 mm
- net /MCU/SDMMC2_D1: track 26.5 -> 27.0 mm

Commit message: Misc routing
Parts:
- moved TP312 90.5 mm to (71.4, 104.6)
- moved TP302 90.0 mm to (61.5, 90.5)
- moved TP303 89.8 mm to (61.5, 92.5)
- moved TP301 88.8 mm to (63.5, 90.5)
- moved TP304 87.2 mm to (63.5, 92.5)
- moved TP311 80.6 mm to (83.7, 104.6)
- moved TP309 78.0 mm to (80.2, 106.6)
- moved TP310 76.3 mm to (80.2, 104.6)
- moved TP308 76.1 mm to (83.7, 106.6)
- moved TP307 74.6 mm to (78.2, 79.2)
- moved TP306 73.0 mm to (80.3, 79.2)
- moved TP801 68.6 mm to (87.2, 81.0)
- moved TP305 63.9 mm to (88.8, 100.7)
- moved C313 1.87 mm to (86.1, 103.7)
- moved R217 0.09 mm to (81.0, 55.2)
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Routing:
- net /DEBUG/T_VCC: track 103.5 -> 470.4 mm, vias 7 -> 19
- net /POWER/SERVO_5V5: track 40.6 -> 396.9 mm, vias 2 -> 9
- net /POWER/D1_5V: track 15.8 -> 291.8 mm, vias 0 -> 7
- net /GPS/VCC: track 0.00 -> 90.3 mm, vias 0 -> 1
- net /GPS/V_BCKP: track 0.00 -> 87.6 mm, vias 0 -> 2
- net /LIDAR/VDD: track 0.00 -> 57.8 mm, vias 0 -> 1
- net /DEBUG/T_JCLK/T_SWCLK: track 9.08 -> 44.2 mm, vias 0 -> 2
- net /DEBUG/T_JTMS/T_SWDIO: track 6.00 -> 38.3 mm
- net /POWER/D3_3V3: track 13.6 -> 45.7 mm, vias 1 -> 3
- net Net-(R1306-Pad1): track 0.00 -> 9.56 mm
- net Net-(U301-PB4): track 0.00 -> 8.55 mm, vias 0 -> 2
- net /LIDAR/RX: track 0.00 -> 8.36 mm
- net /SERVO/CH10_OUT: track 2.99 -> 10.3 mm
- net /SERVO/CH11_OUT: track 11.5 -> 18.8 mm
- net /SERVO/CH13_OUT: track 2.99 -> 10.1 mm
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
Commit message: Finalize RF
Parts:
- moved C1001 0.07 mm to (35.0, 36.1)
- moved AE1001 0.06 mm to (30.2, 25.4)
Routing:
- net Net-(J901-In): track 0.00 -> 5.55 mm
- net Net-(AE1001-A): track 0.00 -> 3.24 mm
- net Net-(U1001-RF_IN): track 0.00 -> 2.51 mm
- net Net-(C1001-Pad2): track 0.00 -> 2.39 mm
- net GND: track 49.9 -> 52.2 mm, vias 32 -> 36

Commit message: Lots of routing
Parts:
- moved SYM101 31.4 mm to (101.1, 72.8)
- moved C315 0.65 mm to (77.6, 82.8)
- moved AE1001 0.29 mm to (30.2, 25.7)
- moved R225 0.20 mm to (83.3, 71.7)
- moved TP308 0.20 mm to (83.7, 106.8)
- moved TP309 0.20 mm to (80.2, 106.8)
- moved TP310 0.20 mm to (80.2, 104.8)
- moved TP311 0.15 mm to (83.7, 104.7)
Connections:
- U301 pad 34: /SERVO/CH12 -> /SERVO/CH15
- U301 pad 35: /SERVO/CH13 -> /SERVO/CH14
- U301 pad 36: /SERVO/CH14 -> /SERVO/CH13
- U301 pad 37: /SERVO/CH15 -> /SERVO/CH12
- U901 pad 4: /MCU/GPIO_PF14 -> /MCU/GPIO_PF13
- U901 pad 5: /MCU/GPIO_PF13 -> /MCU/GPIO_PF14
Routing:
- net /MCU/USB_OTG_HS_VBUS: track 0.00 -> 103.3 mm, vias 0 -> 2
- net /GPS/SCL: track 7.59 -> 99.4 mm, vias 1 -> 2
- net /GPS/SDA: track 4.44 -> 95.3 mm, vias 1 -> 2
- net /GPS/EXTINT: track 0.00 -> 82.5 mm, vias 0 -> 2
- net /GPS/TXD: track 0.00 -> 79.9 mm, vias 0 -> 2
- net /GPS/TIMEPULSE: track 0.00 -> 79.5 mm, vias 0 -> 2
- net /MCU/GPIO_PB11+EXTI11: track 0.00 -> 78.4 mm, vias 0 -> 2
- net /MCU/GPIO_PB10+EXTI10: track 0.00 -> 76.9 mm, vias 0 -> 2
- net Net-(D203-K): track 0.00 -> 76.7 mm, vias 0 -> 2
- net /MCU/GPIO_PD10: track 0.00 -> 76.2 mm, vias 0 -> 2
- net /MCU/GPIO_PD11: track 0.00 -> 76.1 mm, vias 0 -> 2
- net /GPS/RXD: track 0.00 -> 75.0 mm, vias 0 -> 2
- net /MCU/GPIO_PE15+EXTI15: track 0.00 -> 74.5 mm, vias 0 -> 2
- net /MCU/GPIO_PB12+EXTI12: track 0.00 -> 72.7 mm, vias 0 -> 2
- net /GPS/~{RESET}: track 0.00 -> 70.0 mm, vias 0 -> 2
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