File: Hardware/SERVO.kicad_sch (KiCad schematic)
At the start: 0 parts

Commit message: Checkpoint
Changed lines of the file:
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@@
 (kicad_sch (version 20230121) (generator eeschema)
   (paper "A4")
-  (hierarchical_label "CH1" (shape input) (at 114.3 78.74 180) (fields_autoplaced)
-    (effects (font (size 1.27 1.27)) (justify right))
+  (bus (pts (xy 241.3 25.4) (xy 266.7 25.4))
+    (stroke (width 0) (type default))
   )
-  (hierarchical_label "CH0" (shape input) (at 114.3 76.2 180) (fields_autoplaced)
-    (effects (font (size 1.27 1.27)) (justify right))
+  (label "CH[0..11]" (at 241.3 25.4 0) (fields_autoplaced)
+    (effects (font (size 1.27 1.27)) (justify left bottom))
   )
-  (hierarchical_label "CH4" (shape input) (at 114.3 86.36 180) (fields_autoplaced)
-    (effects (font (size 1.27 1.27)) (justify right))
+  (hierarchical_label "CH[0..11]" (shape input) (at 266.7 25.4 0) (fields_autoplaced)
+    (effects (font (size 1.27 1.27)) (justify left))
   )
-  (hierarchical_label "CH3" (shape input) (at 114.3 83.82 180) (fields_autoplaced)
-    (effects (font (size 1.27 1.27)) (justify right))
-  )
-  (hierarchical_label "CH10" (shape input) (at 114.3 101.6 180) (fields_autoplaced)
-    (effects (font (size 1.27 1.27)) (justify right))
-  )
-  (hierarchical_label "CH2" (shape input) (at 114.3 81.28 180) (fields_autoplaced)
-    (effects (font (size 1.27 1.27)) (justify right))
-  )
-  (hierarchical_label "CH6" (shape input) (at 114.3 91.44 180) (fields_autoplaced)
-    (effects (font (size 1.27 1.27)) (justify right))
-  )
-  (hierarchical_label "CH11" (shape input) (at 114.3 104.14 180) (fields_autoplaced)
-    (effects (font (size 1.27 1.27)) (justify right))
-  )
-  (hierarchical_label "CH7" (shape input) (at 114.3 93.98 180) (fields_autoplaced)
-    (effects (font (size 1.27 1.27)) (justify right))
-  )
-  (hierarchical_label "CH9" (shape input) (at 114.3 99.06 180) (fields_autoplaced)
-    (effects (font (size 1.27 1.27)) (justify right))
-  )
-  (hierarchical_label "CH8" (shape input) (at 114.3 96.52 180) (fields_autoplaced)
-    (effects (font (size 1.27 1.27)) (justify right))
-  )
-  (hierarchical_label "CH5" (shape input) (at 114.3 88.9 180) (fields_autoplaced)
-    (effects (font (size 1.27 1.27)) (justify right))
+  (hierarchical_label "PWR" (shape output) (at 152.4 25.4 0) (fields_autoplaced)
+    (effects (font (size 1.27 1.27)) (justify left))
   )
 )

Commit message: Checkpoint
Parts:
- added J10: S7, Connector_PinHeader_2.54mm:PinHeader_1x03_P2.54mm_Vertical, symbol Connector_Generic:Conn_01x03
- added J11: S8, Connector_PinHeader_2.54mm:PinHeader_1x03_P2.54mm_Vertical, symbol Connector_Generic:Conn_01x03
- added J12: S9, Connector_PinHeader_2.54mm:PinHeader_1x03_P2.54mm_Vertical, symbol Connector_Generic:Conn_01x03
- added J13: S10, Connector_PinHeader_2.54mm:PinHeader_1x03_P2.54mm_Vertical, symbol Connector_Generic:Conn_01x03
- added J14: S11, Connector_PinHeader_2.54mm:PinHeader_1x03_P2.54mm_Vertical, symbol Connector_Generic:Conn_01x03
- added J3: S0, Connector_PinHeader_2.54mm:PinHeader_1x03_P2.54mm_Vertical, symbol Connector_Generic:Conn_01x03
- added J4: S1, Connector_PinHeader_2.54mm:PinHeader_1x03_P2.54mm_Vertical, symbol Connector_Generic:Conn_01x03
- added J5: S2, Connector_PinHeader_2.54mm:PinHeader_1x03_P2.54mm_Vertical, symbol Connector_Generic:Conn_01x03
- added J6: S3, Connector_PinHeader_2.54mm:PinHeader_1x03_P2.54mm_Vertical, symbol Connector_Generic:Conn_01x03
- added J7: S4, Connector_PinHeader_2.54mm:PinHeader_1x03_P2.54mm_Vertical, symbol Connector_Generic:Conn_01x03
- added J8: S5, Connector_PinHeader_2.54mm:PinHeader_1x03_P2.54mm_Vertical, symbol Connector_Generic:Conn_01x03
- added J9: S6, Connector_PinHeader_2.54mm:PinHeader_1x03_P2.54mm_Vertical, symbol Connector_Generic:Conn_01x03
- added Q1, Q10, Q11, Q12, Q2, Q3, Q4, Q5, Q6, Q7, Q8, Q9: RE1C002UN, Package_TO_SOT_SMD:SOT-416, symbol Device:Q_NMOS_GSD
- added R10, R11, R12, R13, R14, R15, R16, R17, R18, R19, R20, R21, R22, R23, R24, R25, R26, R27, R28, R29, R30, R31, R8, R9: 2.2K, symbol Device:R_Small
Connections:
- new net CH0: Q1.2 (S), R14.1
- new net CH0_OUT: J3.3 (Pin_3), Q1.3 (D), R15.1
- new net CH1: Q2.2 (S), R12.1
- new net CH10: Q11.2 (S), R26.1
- new net CH10_OUT: J13.3 (Pin_3), Q11.3 (D), R30.1
- new net CH11: Q12.2 (S), R27.1
- new net CH11_OUT: J14.3 (Pin_3), Q12.3 (D), R31.1
- new net CH1_OUT: J4.3 (Pin_3), Q2.3 (D), R13.1
- new net CH2: Q3.2 (S), R10.1
- new net CH2_OUT: J5.3 (Pin_3), Q3.3 (D), R11.1
- new net CH3: Q4.2 (S), R8.1
- new net CH3_OUT: J6.3 (Pin_3), Q4.3 (D), R9.1
- new net CH4: Q5.2 (S), R16.1
- new net CH4_OUT: J7.3 (Pin_3), Q5.3 (D), R20.1
- new net CH5: Q6.2 (S), R17.1
- new net CH5_OUT: J8.3 (Pin_3), Q6.3 (D), R21.1
- new net CH6: Q7.2 (S), R18.1
- new net CH6_OUT: J9.3 (Pin_3), Q7.3 (D), R22.1
- new net CH7: Q8.2 (S), R19.1
- new net CH7_OUT: J10.3 (Pin_3), Q8.3 (D), R23.1
- new net CH8: Q9.2 (S), R24.1
- new net CH8_OUT: J11.3 (Pin_3), Q9.3 (D), R28.1
- new net CH9: Q10.2 (S), R25.1
- new net CH9_OUT: J12.3 (Pin_3), Q10.3 (D), R29.1
- new net GND: J10.1 (Pin_1), J11.1 (Pin_1), J12.1 (Pin_1), J13.1 (Pin_1), J14.1 (Pin_1), J3.1 (Pin_1), J4.1 (Pin_1), J5.1 (Pin_1), J6.1 (Pin_1), J7.1 (Pin_1), J8.1 (Pin_1), J9.1 (Pin_1)
- new net VDD_3V3: Q1.1 (G), Q10.1 (G), Q11.1 (G), Q12.1 (G), Q2.1 (G), Q3.1 (G), Q4.1 (G), Q5.1 (G), Q6.1 (G), Q7.1 (G), Q8.1 (G), Q9.1 (G), R10.2, R12.2, R14.2, R16.2, R17.2, R18.2, R19.2, R24.2, R25.2, R26.2, R27.2, R8.2
- new net VDD_SERVO: J10.2 (Pin_2), J11.2 (Pin_2), J12.2 (Pin_2), J13.2 (Pin_2), J14.2 (Pin_2), J3.2 (Pin_2), J4.2 (Pin_2), J5.2 (Pin_2), J6.2 (Pin_2), J7.2 (Pin_2), J8.2 (Pin_2), J9.2 (Pin_2), R11.2, R13.2, R15.2, R20.2, R21.2, R22.2, R23.2, R28.2, R29.2, R30.2, R31.2, R9.2

Commit message: Checkpoint
Parts:
- renumbered J3 to J1201, J4 to J1202, J5 to J1203, J6 to J1204, J7 to J1205, J8 to J1206, J9 to J1207, J10 to J1208, J11 to J1209, J12 to J1210, J13 to J1211, J14 to J1212, Q1 to Q1201, Q2 to Q1202, Q3 to Q1203, Q4 to Q1204, Q5 to Q1205, Q6 to Q1206, Q7 to Q1207, Q8 to Q1208, Q9 to Q1209, Q10 to Q1210, Q11 to Q1211, Q12 to Q1212, R14 to R1201, R12 to R1202, R10 to R1203, R8 to R1204, R15 to R1205, R13 to R1206, R11 to R1207, R9 to R1208, R16 to R1209, R17 to R1210, R18 to R1211, R19 to R1212, R20 to R1213, R21 to R1214, R22 to R1215, R23 to R1216, R24 to R1217, R25 to R1218, R26 to R1219, R27 to R1220, R28 to R1221, R29 to R1222, R30 to R1223, R31 to R1224

Commit message: Checkpoint
Parts:
- R1201, R1202, R1203, R1204, R1205, R1206, R1207, R1208, R1209, R1210, R1211, R1212, R1213, R1214, R1215, R1216, R1217, R1218, R1219, R1220, R1221, R1222, R1223, R1224: footprint (none) -> Resistor_SMD:R_0805_2012Metric
Changed lines of the file:
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@@
       (effects (font (size 1.27 1.27)) (justify right))
     )
-    (property "Footprint" "" (at 30.48 109.22 0)
+    (property "Footprint" "Resistor_SMD:R_0805_2012Metric" (at 30.48 109.22 0)
       (effects (font (size 1.27 1.27)) hide)
     )
@@
       (effects (font (size 1.27 1.27)) (justify right))
     )
-    (property "Footprint" "" (at 45.72 58.42 0)
+    (property "Footprint" "Resistor_SMD:R_0805_2012Metric" (at 45.72 58.42 0)
       (effects (font (size 1.27 1.27)) hide)
     )
@@
       (effects (font (size 1.27 1.27)) (justify right))
     )
-    (property "Footprint" "" (at 96.52 109.22 0)
+    (property "Footprint" "Resistor_SMD:R_0805_2012Metric" (at 96.52 109.22 0)
       (effects (font (size 1.27 1.27)) hide)
     )
@@
       (effects (font (size 1.27 1.27)) (justify right))
     )
-    (property "Footprint" "" (at 132.08 83.82 0)
+    (property "Footprint" "Resistor_SMD:R_0805_2012Metric" (at 132.08 83.82 0)
       (effects (font (size 1.27 1.27)) hide)
     )
@@
       (effects (font (size 1.27 1.27)) (justify right))
     )
-    (property "Footprint" "" (at 81.28 33.02 0)
+    (property "Footprint" "Resistor_SMD:R_0805_2012Metric" (at 81.28 33.02 0)
       (effects (font (size 1.27 1.27)) hide)
     )
@@
       (effects (font (size 1.27 1.27)) (justify right))
     )
-    (property "Footprint" "" (at 96.52 58.42 0)
+    (property "Footprint" "Resistor_SMD:R_0805_2012Metric" (at 96.52 58.42 0)
       (effects (font (size 1.27 1.27)) hide)
     )
@@
       (effects (font (size 1.27 1.27)) (justify right))
     )
-    (property "Footprint" "" (at 147.32 58.42 0)
+    (property "Footprint" "Resistor_SMD:R_0805_2012Metric" (at 147.32 58.42 0)
       (effects (font (size 1.27 1.27)) hide)
     )
@@
       (effects (font (size 1.27 1.27)) (justify right))
     )
-    (property "Footprint" "" (at 132.08 33.02 0)
+    (property "Footprint" "Resistor_SMD:R_0805_2012Metric" (at 132.08 33.02 0)
       (effects (font (size 1.27 1.27)) hide)
     )
@@
       (effects (font (size 1.27 1.27)) (justify right))
     )
-    (property "Footprint" "" (at 81.28 58.42 0)
+    (property "Footprint" "Resistor_SMD:R_0805_2012Metric" (at 81.28 58.42 0)
       (effects (font (size 1.27 1.27)) hide)
     )
@@
       (effects (font (size 1.27 1.27)) (justify right))
     )
-    (property "Footprint" "" (at 132.08 58.42 0)
+    (property "Footprint" "Resistor_SMD:R_0805_2012Metric" (at 132.08 58.42 0)
       (effects (font (size 1.27 1.27)) hide)
     )
@@
       (effects (font (size 1.27 1.27)) (justify right))
     )
-    (property "Footprint" "" (at 30.48 58.42 0)
+    (property "Footprint" "Resistor_SMD:R_0805_2012Metric" (at 30.48 58.42 0)
       (effects (font (size 1.27 1.27)) hide)
     )
@@
       (effects (font (size 1.27 1.27)) (justify right))
     )
-    (property "Footprint" "" (at 96.52 83.82 0)
+    (property "Footprint" "Resistor_SMD:R_0805_2012Metric" (at 96.52 83.82 0)
       (effects (font (size 1.27 1.27)) hide)
     )
@@
       (effects (font (size 1.27 1.27)) (justify right))
     )
-    (property "Footprint" "" (at 147.32 33.02 0)
+    (property "Footprint" "Resistor_SMD:R_0805_2012Metric" (at 147.32 33.02 0)
       (effects (font (size 1.27 1.27)) hide)
     )
@@
       (effects (font (size 1.27 1.27)) (justify right))
     )
-    (property "Footprint" "" (at 147.32 109.22 0)
+    (property "Footprint" "Resistor_SMD:R_0805_2012Metric" (at 147.32 109.22 0)
       (effects (font (size 1.27 1.27)) hide)
     )
@@
       (effects (font (size 1.27 1.27)) (justify right))
     )
-    (property "Footprint" "" (at 147.32 83.82 0)
+    (property "Footprint" "Resistor_SMD:R_0805_2012Metric" (at 147.32 83.82 0)
       (effects (font (size 1.27 1.27)) hide)
     )
@@
       (effects (font (size 1.27 1.27)) (justify right))
     )
-    (property "Footprint" "" (at 45.72 109.22 0)
+    (property "Footprint" "Resistor_SMD:R_0805_2012Metric" (at 45.72 109.22 0)
       (effects (font (size 1.27 1.27)) hide)
     )
@@
       (effects (font (size 1.27 1.27)) (justify right))
     )
-    (property "Footprint" "" (at 45.72 33.02 0)
+    (property "Footprint" "Resistor_SMD:R_0805_2012Metric" (at 45.72 33.02 0)
       (effects (font (size 1.27 1.27)) hide)
     )
@@
       (effects (font (size 1.27 1.27)) (justify right))
     )
-    (property "Footprint" "" (at 81.28 83.82 0)
+    (property "Footprint" "Resistor_SMD:R_0805_2012Metric" (at 81.28 83.82 0)
       (effects (font (size 1.27 1.27)) hide)
     )
@@
       (effects (font (size 1.27 1.27)) (justify right))
     )
-    (property "Footprint" "" (at 45.72 83.82 0)
+    (property "Footprint" "Resistor_SMD:R_0805_2012Metric" (at 45.72 83.82 0)
       (effects (font (size 1.27 1.27)) hide)
     )
@@
       (effects (font (size 1.27 1.27)) (justify right))
     )
-    (property "Footprint" "" (at 81.28 109.22 0)
+    (property "Footprint" "Resistor_SMD:R_0805_2012Metric" (at 81.28 109.22 0)
       (effects (font (size 1.27 1.27)) hide)
     )
@@
       (effects (font (size 1.27 1.27)) (justify right))
     )
-    (property "Footprint" "" (at 96.52 33.02 0)
+    (property "Footprint" "Resistor_SMD:R_0805_2012Metric" (at 96.52 33.02 0)
       (effects (font (size 1.27 1.27)) hide)
     )
@@
       (effects (font (size 1.27 1.27)) (justify right))
     )
-    (property "Footprint" "" (at 132.08 109.22 0)
+    (property "Footprint" "Resistor_SMD:R_0805_2012Metric" (at 132.08 109.22 0)
       (effects (font (size 1.27 1.27)) hide)
     )
@@
       (effects (font (size 1.27 1.27)) (justify right))
     )
-    (property "Footprint" "" (at 30.48 33.02 0)
+    (property "Footprint" "Resistor_SMD:R_0805_2012Metric" (at 30.48 33.02 0)
       (effects (font (size 1.27 1.27)) hide)
     )
@@
       (effects (font (size 1.27 1.27)) (justify right))
     )
-    (property "Footprint" "" (at 30.48 83.82 0)
-      (effects (font (size 1.27 1.27)) hide)
-    )
+    (property "Footprint" "Resistor_SMD:R_0805_2012Metric" (at 30.48 83.82 0)
+      (effects (font (size 1.27 1.27)) hide)
+    )

Commit message: Checkpoint
Parts:
- added J1213, J1214, J1215, J1216: S11, Connector_PinHeader_2.54mm:PinHeader_1x03_P2.54mm_Vertical, symbol Connector_Generic:Conn_01x03
- added Q1213, Q1214, Q1215, Q1216: RE1C002UN, Package_TO_SOT_SMD:SOT-416, symbol Device:Q_NMOS_GSD
- added R1225, R1226, R1227, R1228, R1229, R1230, R1231, R1232: 2.2K, Resistor_SMD:R_0805_2012Metric, symbol Device:R_Small
Connections:
- net GND: now also J1213.1 (Pin_1), J1214.1 (Pin_1), J1215.1 (Pin_1), J1216.1 (Pin_1)
- net VDD_3V3: now also Q1213.1 (G), Q1214.1 (G), Q1215.1 (G), Q1216.1 (G), R1225.2, R1226.2, R1227.2, R1228.2
- net VDD_SERVO: now also J1213.2 (Pin_2), J1214.2 (Pin_2), J1215.2 (Pin_2), J1216.2 (Pin_2), R1229.2, R1230.2, R1231.2, R1232.2
- new net CH12: Q1213.2 (S), R1225.1
- new net CH12_OUT: J1213.3 (Pin_3), Q1213.3 (D), R1229.1
- new net CH13: Q1214.2 (S), R1226.1
- new net CH13_OUT: J1214.3 (Pin_3), Q1214.3 (D), R1230.1
- new net CH14: Q1215.2 (S), R1227.1
- new net CH14_OUT: J1215.3 (Pin_3), Q1215.3 (D), R1231.1
- new net CH15: Q1216.2 (S), R1228.1
- new net CH15_OUT: J1216.3 (Pin_3), Q1216.3 (D), R1232.1
Other:
- moved on the sheet: J1201, J1202, J1203, J1204, J1205, J1206, J1207, J1208, J1209, J1210, J1211, J1212

Commit message: Checkpoint
Parts:
- J1207, J1208, J1209, J1210, J1211, J1212: footprint Connector_PinHeader_2.54mm:PinHeader_1x03_P2.54mm_Vertical -> Connector_PinHeader_2.54mm:PinHeader_1x03_P2.54mm_Horizontal
- J1213: value S11 -> S12; footprint Connector_PinHeader_2.54mm:PinHeader_1x03_P2.54mm_Vertical -> Connector_PinHeader_2.54mm:PinHeader_1x03_P2.54mm_Horizontal
- J1214: value S11 -> S13; footprint Connector_PinHeader_2.54mm:PinHeader_1x03_P2.54mm_Vertical -> Connector_PinHeader_2.54mm:PinHeader_1x03_P2.54mm_Horizontal
- J1215: value S11 -> S14; footprint Connector_PinHeader_2.54mm:PinHeader_1x03_P2.54mm_Vertical -> Connector_PinHeader_2.54mm:PinHeader_1x03_P2.54mm_Horizontal
- J1216: value S11 -> S15; footprint Connector_PinHeader_2.54mm:PinHeader_1x03_P2.54mm_Vertical -> Connector_PinHeader_2.54mm:PinHeader_1x03_P2.54mm_Horizontal

Commit message: Checkpoint
Parts:
- added U1201, U1202, U1203, U1204: USBLC6-4SC6, Package_TO_SOT_SMD:SOT-23-6, symbol Power_Protection:USBLC6-4SC6
Connections:
- net CH0_OUT: now also U1201.1 (I/O1)
- net CH10_OUT: now also U1203.4 (I/O3)
- net CH11_OUT: now also U1203.6 (I/O4)
- net CH12_OUT: now also U1204.1 (I/O1)
- net CH13_OUT: now also U1204.3 (I/O2)
- net CH14_OUT: now also U1204.4 (I/O3)
- net CH15_OUT: now also U1204.6 (I/O4)
- net CH1_OUT: now also U1201.3 (I/O2)
- net CH2_OUT: now also U1201.4 (I/O3)
- net CH3_OUT: now also U1201.6 (I/O4)
- net CH4_OUT: now also U1202.1 (I/O1)
- net CH5_OUT: now also U1202.3 (I/O2)
- net CH6_OUT: now also U1202.4 (I/O3)
- net CH7_OUT: now also U1202.6 (I/O4)
- net CH8_OUT: now also U1203.1 (I/O1)
- net CH9_OUT: now also U1203.3 (I/O2)
- net GND: now also U1201.2 (GND), U1202.2 (GND), U1203.2 (GND), U1204.2 (GND)
- net VDD_SERVO: now also U1201.5 (VBUS), U1202.5 (VBUS), U1203.5 (VBUS), U1204.5 (VBUS); no longer J1201.2 (Pin_2), R1205.2
- new net VDD_ESC: J1201.2 (Pin_2), R1205.2
Other:
- moved on the sheet: J1201, J1202, J1203, J1204, J1205, J1206, J1207, J1208, J1209, J1210, J1211, J1212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

Commit message: Checkpoint routing
Connections:
- net CH10_OUT: now also U1203.3 (I/O2); no longer U1203.4 (I/O3)
- net CH11_OUT: now also U1203.1 (I/O1); no longer U1203.6 (I/O4)
- net CH8_OUT: now also U1203.6 (I/O4); no longer U1203.1 (I/O1)
- net CH9_OUT: now also U1203.4 (I/O3); no longer U1203.3 (I/O2)
Changed lines of the file:
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@@
     (effects (font (size 1.27 1.27)) (justify right bottom))
   )
-  (label "CH9_OUT" (at 233.68 114.3 0) (fields_autoplaced)
-    (effects (font (size 1.27 1.27)) (justify left bottom))
+  (label "CH9_OUT" (at 274.32 109.22 180) (fields_autoplaced)
+    (effects (font (size 1.27 1.27)) (justify right bottom))
   )
   (label "CH12_OUT" (at 208.28 40.64 180) (fields_autoplaced)
@@
     (effects (font (size 1.27 1.27)) (justify left bottom))
   )
-  (label "CH11_OUT" (at 274.32 114.3 180) (fields_autoplaced)
-    (effects (font (size 1.27 1.27)) (justify right bottom))
+  (label "CH11_OUT" (at 233.68 109.22 0) (fields_autoplaced)
+    (effects (font (size 1.27 1.27)) (justify left bottom))
   )
   (label "CH10" (at 124.46 91.44 0) (fields_autoplaced)
@@
     (effects (font (size 1.27 1.27)) (justify right bottom))
   )
-  (label "CH8_OUT" (at 233.68 109.22 0) (fields_autoplaced)
-    (effects (font (size 1.27 1.27)) (justify left bottom))
+  (label "CH8_OUT" (at 274.32 114.3 180) (fields_autoplaced)
+    (effects (font (size 1.27 1.27)) (justify right bottom))
   )
   (label "CH1_OUT" (at 233.68 48.26 0) (fields_autoplaced)
@@
     (effects (font (size 1.27 1.27)) (justify right bottom))
   )
-  (label "CH10_OUT" (at 274.32 109.22 180) (fields_autoplaced)
-    (effects (font (size 1.27 1.27)) (justify right bottom))
+  (label "CH10_OUT" (at 233.68 114.3 0) (fields_autoplaced)
+    (effects (font (size 1.27 1.27)) (justify left bottom))
   )
   (hierarchical_label "VDD_SERVO" (shape passive) (at 27.94 104.14 180) (fields_autoplaced)
