File: Hardware/SERVO.kicad_sch (KiCad schematic)
At the start: 68 parts, among them J1201 S0, J1202 S1, J1203 S2, J1204 S3, J1205 S4, J1206 S5, J1207 S6, J1208 S7, J1209 S8, J1210 S9, J1211 S10, J1212 S11, J1213 S12, J1214 S13, J1215 S14, J1216 S15, Q1201 RE1C002UN, Q1202 RE1C002UN, Q1203 RE1C002UN, Q1204 RE1C002UN, Q1205 RE1C002UN, Q1206 RE1C002UN, Q1207 RE1C002UN, Q1208 RE1C002UN, Q1209 RE1C002UN, Q1210 RE1C002UN, Q1211 RE1C002UN, Q1212 RE1C002UN, Q1213 RE1C002UN, Q1214 RE1C002UN, Q1215 RE1C002UN, Q1216 RE1C002UN, U1201 USBLC6-4SC6, U1202 USBLC6-4SC6, U1203 USBLC6-4SC6, U1204 USBLC6-4SC6

Commit message: Finalize silkscreen
Other:
- title: (none) -> Avionus_Flight_Controller
Changed lines of the file:
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@@
 (kicad_sch (version 20230121) (generator eeschema)
   (paper "A4")
+  (title_block
+    (title "Avionus_Flight_Controller")
+    (date "2023-11-25")
+    (rev "1.0")
+  )
   (junction (at 96.52 66.04) (diameter 0) (color 0 0 0 0)
   )

Commit message: Misc fixes
Parts:
- J1201: value S0 -> CH0
- J1202: value S1 -> CH1
- J1203: value S2 -> CH2
- J1204: value S3 -> CH3
- J1205: value S4 -> CH4
- J1206: value S5 -> CH5
- J1207: value S6 -> CH6
- J1208: value S7 -> CH7
- J1209: value S8 -> CH8
- J1210: value S9 -> CH9
- J1211: value S10 -> CH10
- J1212: value S11 -> CH11
- J1213: value S12 -> CH12
- J1214: value S13 -> CH13
- J1215: value S14 -> CH14
- J1216: value S15 -> CH15
Changed lines of the file:
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@@
       (effects (font (size 1.27 1.27)))
     )
-    (property "Value" "S4" (at 63.5 133.35 90)
+    (property "Value" "CH4" (at 63.5 133.35 90)
       (effects (font (size 1.27 1.27)))
     )
@@
       (effects (font (size 1.27 1.27)))
     )
-    (property "Value" "S12" (at 144.78 133.35 90)
+    (property "Value" "CH12" (at 144.78 133.35 90)
       (effects (font (size 1.27 1.27)))
     )
@@
       (effects (font (size 1.27 1.27)))
     )
-    (property "Value" "S8" (at 104.14 133.35 90)
+    (property "Value" "CH8" (at 104.14 133.35 90)
       (effects (font (size 1.27 1.27)))
     )
@@
       (effects (font (size 1.27 1.27)))
     )
-    (property "Value" "S2" (at 43.18 133.35 90)
+    (property "Value" "CH2" (at 43.18 133.35 90)
       (effects (font (size 1.27 1.27)))
     )
@@
       (effects (font (size 1.27 1.27)))
     )
-    (property "Value" "S5" (at 73.66 133.35 90)
+    (property "Value" "CH5" (at 73.66 133.35 90)
       (effects (font (size 1.27 1.27)))
     )
@@
       (effects (font (size 1.27 1.27)))
     )
-    (property "Value" "S10" (at 124.46 133.35 90)
+    (property "Value" "CH10" (at 124.46 133.35 90)
       (effects (font (size 1.27 1.27)))
     )
@@
       (effects (font (size 1.27 1.27)))
     )
-    (property "Value" "S15" (at 175.26 133.35 90)
+    (property "Value" "CH15" (at 175.26 133.35 90)
       (effects (font (size 1.27 1.27)))
     )
@@
       (effects (font (size 1.27 1.27)))
     )
-    (property "Value" "S7" (at 93.98 133.35 90)
+    (property "Value" "CH7" (at 93.98 133.35 90)
       (effects (font (size 1.27 1.27)))
     )
@@
       (effects (font (size 1.27 1.27)))
     )
-    (property "Value" "S11" (at 134.62 133.35 90)
+    (property "Value" "CH11" (at 134.62 133.35 90)
       (effects (font (size 1.27 1.27)))
     )
@@
       (effects (font (size 1.27 1.27)))
     )
-    (property "Value" "S6" (at 83.82 133.35 90)
+    (property "Value" "CH6" (at 83.82 133.35 90)
       (effects (font (size 1.27 1.27)))
     )
@@
       (effects (font (size 1.27 1.27)))
     )
-    (property "Value" "S9" (at 114.3 133.35 90)
+    (property "Value" "CH9" (at 114.3 133.35 90)
       (effects (font (size 1.27 1.27)))
     )
@@
       (effects (font (size 1.27 1.27)))
     )
-    (property "Value" "S0" (at 22.86 133.35 90)
+    (property "Value" "CH0" (at 22.86 133.35 90)
       (effects (font (size 1.27 1.27)))
     )
@@
       (effects (font (size 1.27 1.27)))
     )
-    (property "Value" "S3" (at 53.34 133.35 90)
+    (property "Value" "CH3" (at 53.34 133.35 90)
       (effects (font (size 1.27 1.27)))
     )
@@
       (effects (font (size 1.27 1.27)))
     )
-    (property "Value" "S13" (at 154.94 133.35 90)
+    (property "Value" "CH13" (at 154.94 133.35 90)
       (effects (font (size 1.27 1.27)))
     )
@@
       (effects (font (size 1.27 1.27)))
     )
-    (property "Value" "S1" (at 33.02 133.35 90)
+    (property "Value" "CH1" (at 33.02 133.35 90)
       (effects (font (size 1.27 1.27)))
     )
@@
       (effects (font (size 1.27 1.27)))
     )
-    (property "Value" "S14" (at 165.1 133.35 90)
-      (effects (font (size 1.27 1.27)))
-    )
+    (property "Value" "CH14" (at 165.1 133.35 90)
+      (effects (font (size 1.27 1.27)))
+    )
