File: Hardware/USB.kicad_sch (KiCad schematic)
At the start: 7 parts, among them J1 USB_C_Receptacle_USB2.0, U10 USBLC6-2SC6

Commit message: Checkpoint
Parts:
- removed C3: 100nF, symbol Device:C
- removed R1: 330R, Resistor_SMD:R_0805_2012Metric, symbol Device:R
Connections:
- net D-: now also U10.1 (I/O1); no longer U10.4 (I/O2)
- net CONN_D+: now reaches J1.A6 (D+), J1.B6 (D+)
- net CONN_D+: now also U10.4 (I/O2); no longer U10.1 (I/O1)
- net CONN_D-: now reaches J1.A7 (D-), J1.B7 (D-), U10.6 (I/O1)
- no-connect marks 2 -> 3
Other:
- moved on the sheet: R44, R45, U10

Commit message: Checkpoint
Changed lines of the file:
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@@
+    (stroke (width 0) (type default))
+  )
+  (wire (pts (xy 193.04 93.98) (xy 198.12 93.98))
     (stroke (width 0) (type default))
   )
@@
   )
   (wire (pts (xy 147.32 96.52) (xy 157.48 96.52))
+    (stroke (width 0) (type default))
+  )
+  (wire (pts (xy 223.52 93.98) (xy 218.44 93.98))
     (stroke (width 0) (type default))
   )
@@
     (effects (font (size 1.27 1.27)) (justify left))
   )
-  (hierarchical_label "D-" (shape bidirectional) (at 198.12 93.98 180) (fields_autoplaced)
+  (hierarchical_label "D-" (shape bidirectional) (at 193.04 93.98 180) (fields_autoplaced)
     (effects (font (size 1.27 1.27)) (justify right))
   )
@@
     (effects (font (size 1.27 1.27)) (justify left))
   )
-  (hierarchical_label "D+" (shape bidirectional) (at 218.44 93.98 0) (fields_autoplaced)
+  (hierarchical_label "D+" (shape bidirectional) (at 223.52 93.98 0) (fields_autoplaced)
     (effects (font (size 1.27 1.27)) (justify left))
   )
+  (netclass_flag "" (length 2.54) (shape round) (at 195.58 93.98 180) (fields_autoplaced)
+    (effects (font (size 1.27 1.27)) (justify right bottom))
+    (property "Netclass" "USB" (at 196.2785 96.52 0)
+      (effects (font (size 1.27 1.27) italic) (justify left))
+    )
+  )
+  (netclass_flag "" (length 2.54) (shape round) (at 220.98 93.98 180) (fields_autoplaced)
+    (effects (font (size 1.27 1.27)) (justify right bottom))
+    (property "Netclass" "USB" (at 221.6785 96.52 0)
+      (effects (font (size 1.27 1.27) italic) (justify left))
+    )
+  )
+  (netclass_flag "" (length 2.54) (shape round) (at 195.58 88.9 180) (fields_autoplaced)
+    (effects (font (size 1.27 1.27)) (justify right bottom))
+    (property "Netclass" "USB" (at 196.2785 91.44 0)
+      (effects (font (size 1.27 1.27) italic) (justify left))
+    )
+  )
+  (netclass_flag "" (length 2.54) (shape round) (at 220.98 88.9 180) (fields_autoplaced)
+    (effects (font (size 1.27 1.27)) (justify right bottom))
+    (property "Netclass" "USB" (at 221.6785 91.44 0)
+      (effects (font (size 1.27 1.27) italic) (justify left))
+    )
+  )
   (symbol (lib_id "Device:R_Small") (at 160.02 83.82 270) (mirror x) (unit 1)

Commit message: Checkpoint
Parts:
- renumbered J1 to J?, R44 to R801, R45 to R802, TP8 to TP801, U10 to U801
Changed lines of the file:
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@@
   (symbol (lib_id "Device:R_Small") (at 160.02 83.82 270) (mirror x) (unit 1)
     (in_bom yes) (on_board yes) (dnp no) (fields_autoplaced)
-    (property "Reference" "R45" (at 160.02 86.36 90)
+    (property "Reference" "R802" (at 160.02 86.36 90)
       (effects (font (size 1.27 1.27)))
     )
@@
       (project "Avionus_Flight_Controller"
         (path "/ddc7e940-0588-4587-8902-8ced9e615ace/d19046d9-5fb5-41f1-9a98-30f2d85e54f8"
-          (reference "R45") (unit 1)
+          (reference "R802") (unit 1)
         )
       )
@@
   (symbol (lib_id "power:GND") (at 167.64 83.82 90) (unit 1)
     (in_bom yes) (on_board yes) (dnp no)
-    (property "Reference" "#PWR033" (at 173.99 83.82 0)
+    (property "Reference" "#PWR0802" (at 173.99 83.82 0)
       (effects (font (size 1.27 1.27)) hide)
     )
@@
       (project "Avionus_Flight_Controller"
         (path "/ddc7e940-0588-4587-8902-8ced9e615ace/d19046d9-5fb5-41f1-9a98-30f2d85e54f8"
-          (reference "#PWR033") (unit 1)
+          (reference "#PWR0802") (unit 1)
         )
       )
@@
   (symbol (lib_id "power:GND") (at 129.54 114.3 0) (unit 1)
     (in_bom yes) (on_board yes) (dnp no) (fields_autoplaced)
-    (property "Reference" "#PWR031" (at 129.54 120.65 0)
+    (property "Reference" "#PWR0801" (at 129.54 120.65 0)
       (effects (font (size 1.27 1.27)) hide)
     )
@@
       (project "Avionus_Flight_Controller"
         (path "/ddc7e940-0588-4587-8902-8ced9e615ace/d19046d9-5fb5-41f1-9a98-30f2d85e54f8"
-          (reference "#PWR031") (unit 1)
+          (reference "#PWR0801") (unit 1)
         )
       )
@@
   (symbol (lib_id "Device:R_Small") (at 160.02 81.28 270) (unit 1)
     (in_bom yes) (on_board yes) (dnp no) (fields_autoplaced)
-    (property "Reference" "R44" (at 160.02 74.93 90)
+    (property "Reference" "R801" (at 160.02 74.93 90)
       (effects (font (size 1.27 1.27)))
     )
@@
       (project "Avionus_Flight_Controller"
         (path "/ddc7e940-0588-4587-8902-8ced9e615ace/d19046d9-5fb5-41f1-9a98-30f2d85e54f8"
-          (reference "R44") (unit 1)
+          (reference "R801") (unit 1)
         )
       )
@@
   (symbol (lib_id "Power_Protection:USBLC6-2SC6") (at 208.28 91.44 0) (unit 1)
     (in_bom yes) (on_board yes) (dnp no) (fields_autoplaced)
-    (property "Reference" "U10" (at 209.9311 78.74 0)
+    (property "Reference" "U801" (at 209.9311 78.74 0)
       (effects (font (size 1.27 1.27)) (justify left))
     )
@@
       (project "Avionus_Flight_Controller"
         (path "/ddc7e940-0588-4587-8902-8ced9e615ace/d19046d9-5fb5-41f1-9a98-30f2d85e54f8"
-          (reference "U10") (unit 1)
+          (reference "U801") (unit 1)
         )
       )
@@
   (symbol (lib_id "Connector:TestPoint") (at 266.7 20.32 90) (unit 1)
     (in_bom yes) (on_board yes) (dnp no) (fields_autoplaced)
-    (property "Reference" "TP8" (at 263.398 17.78 90)
+    (property "Reference" "TP801" (at 263.398 17.78 90)
       (effects (font (size 1.27 1.27)))
     )
@@
       (project "Avionus_Flight_Controller"
         (path "/ddc7e940-0588-4587-8902-8ced9e615ace/d19046d9-5fb5-41f1-9a98-30f2d85e54f8"
-          (reference "TP8") (unit 1)
+          (reference "TP801") (unit 1)
         )
       )
@@
   (symbol (lib_id "Connector:USB_C_Receptacle_USB2.0") (at 129.54 91.44 0) (unit 1)
     (in_bom yes) (on_board yes) (dnp no)
-    (property "Reference" "J1" (at 132.2578 69.4182 0)
+    (property "Reference" "J?" (at 132.2578 69.4182 0)
       (effects (font (size 1.27 1.27)))
     )
@@
       (project "MUXUS"
         (path "/4790d15d-8fc7-4350-9ac5-2cdedd8248a8"
-          (reference "J1") (unit 1)
-        )
-      )
-      (project "Avionus_Flight_Controller"
-        (path "/ddc7e940-0588-4587-8902-8ced9e615ace/d19046d9-5fb5-41f1-9a98-30f2d85e54f8"
-          (reference "J16") (unit 1)
+          (reference "J?") (unit 1)
+        )
+      )
+      (project "Avionus_Flight_Controller"
+        (path "/ddc7e940-0588-4587-8902-8ced9e615ace/d19046d9-5fb5-41f1-9a98-30f2d85e54f8"
+          (reference "J801") (unit 1)
         )
       )
@@
   (symbol (lib_name "GND_1") (lib_id "power:GND") (at 208.28 104.14 0) (unit 1)
     (in_bom yes) (on_board yes) (dnp no) (fields_autoplaced)
-    (property "Reference" "#PWR032" (at 208.28 110.49 0)
+    (property "Reference" "#PWR0803" (at 208.28 110.49 0)
       (effects (font (size 1.27 1.27)) hide)
     )
@@
       (project "Avionus_Flight_Controller"
         (path "/ddc7e940-0588-4587-8902-8ced9e615ace/d19046d9-5fb5-41f1-9a98-30f2d85e54f8"
-          (reference "#PWR032") (unit 1)
-        )
-      )
+          (reference "#PWR0803") (unit 1)
+        )
+      )

Commit message: Checkpoint
Parts:
- R801, R802: footprint (none) -> Resistor_SMD:R_0603_1608Metric
Changed lines of the file:
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@@
       (effects (font (size 1.27 1.27)))
     )
-    (property "Footprint" "" (at 160.02 83.82 0)
+    (property "Footprint" "Resistor_SMD:R_0603_1608Metric" (at 160.02 83.82 0)
       (effects (font (size 1.27 1.27)) hide)
     )
@@
       (effects (font (size 1.27 1.27)))
     )
-    (property "Footprint" "" (at 160.02 81.28 0)
+    (property "Footprint" "Resistor_SMD:R_0603_1608Metric" (at 160.02 81.28 0)
       (effects (font (size 1.27 1.27)) hide)
     )

Commit message: Checkpoint
Parts:
- TP801: footprint (none) -> TestPoint:TestPoint_Pad_D2.0mm
Changed lines of the file:
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@@
       (effects (font (size 1.27 1.27)) hide)
     )
-    (property "Footprint" "" (at 266.7 15.24 0)
+    (property "Footprint" "TestPoint:TestPoint_Pad_D2.0mm" (at 266.7 15.24 0)
       (effects (font (size 1.27 1.27)) hide)
     )

Commit message: Checkpoint
Connections:
- net CONN_D+: now also U801.6 (I/O1); no longer U801.4 (I/O2)
- net CONN_D-: now also U801.4 (I/O2); no longer U801.6 (I/O1)
- net D+: now also U801.1 (I/O1); no longer U801.3 (I/O2)
- net D-: now also U801.3 (I/O2); no longer U801.1 (I/O1)
Changed lines of the file:
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@@
     (stroke (width 0) (type default))
   )
-  (label "CONN_D-" (at 187.96 88.9 0) (fields_autoplaced)
-    (effects (font (size 1.27 1.27)) (justify left bottom))
+  (label "CONN_D-" (at 228.6 88.9 180) (fields_autoplaced)
+    (effects (font (size 1.27 1.27)) (justify right bottom))
   )
   (label "CONN_D+" (at 157.48 96.52 180) (fields_autoplaced)
@@
     (effects (font (size 1.27 1.27)) (justify right bottom))
   )
-  (label "CONN_D+" (at 228.6 88.9 180) (fields_autoplaced)
-    (effects (font (size 1.27 1.27)) (justify right bottom))
+  (label "CONN_D+" (at 187.96 88.9 0) (fields_autoplaced)
+    (effects (font (size 1.27 1.27)) (justify left bottom))
   )
   (hierarchical_label "SOF" (shape input) (at 266.7 20.32 0) (fields_autoplaced)
@@
     (effects (font (size 1.27 1.27)) (justify left))
   )
-  (hierarchical_label "D-" (shape bidirectional) (at 193.04 93.98 180) (fields_autoplaced)
-    (effects (font (size 1.27 1.27)) (justify right))
+  (hierarchical_label "D-" (shape bidirectional) (at 223.52 93.98 0) (fields_autoplaced)
+    (effects (font (size 1.27 1.27)) (justify left))
   )
   (hierarchical_label "VBUS" (shape output) (at 208.28 81.28 90) (fields_autoplaced)
     (effects (font (size 1.27 1.27)) (justify left))
   )
-  (hierarchical_label "D+" (shape bidirectional) (at 223.52 93.98 0) (fields_autoplaced)
-    (effects (font (size 1.27 1.27)) (justify left))
+  (hierarchical_label "D+" (shape bidirectional) (at 193.04 93.98 180) (fields_autoplaced)
+    (effects (font (size 1.27 1.27)) (justify right))
   )
   (netclass_flag "" (length 2.54) (shape round) (at 195.58 93.98 180) (fields_autoplaced)

Commit message: Checkpoint
Parts:
- TP801: footprint TestPoint:TestPoint_Pad_D2.0mm -> TestPoint:TestPoint_Pad_D1.0mm
Changed lines of the file:
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@@
       (effects (font (size 1.27 1.27)) hide)
     )
-    (property "Footprint" "TestPoint:TestPoint_Pad_D2.0mm" (at 266.7 15.24 0)
+    (property "Footprint" "TestPoint:TestPoint_Pad_D1.0mm" (at 266.7 15.24 0)
       (effects (font (size 1.27 1.27)) hide)
     )
