File: Hardware/USB.kicad_sch (KiCad schematic)
At the start: 5 parts, among them U801 USBLC6-2SC6

Commit message: Finalize silkscreen
Other:
- title: (none) -> Avionus_Flight_Controller
Changed lines of the file:
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@@
 (kicad_sch (version 20230121) (generator eeschema)
   (paper "A4")
+  (title_block
+    (title "Avionus_Flight_Controller")
+    (date "2023-11-25")
+    (rev "1.0")
+  )
   (junction (at 147.32 96.52) (diameter 0) (color 0 0 0 0)
   )
