File: Hardware/GPS.kicad_sch (KiCad schematic)
At the start: 0 parts

Commit message: Checkpoint
Parts:
- added AE1: GPS antenna, symbol Device:Antenna_Shield
- added TP1: ~{SAFEBOOT}, symbol Connector:TestPoint
- added U2: MAX-M10S, RF_GPS:ublox_MAX, symbol RF_GPS:MAX-M10S
Connections:
- new net: TP1.1, U2.18 (~{SAFEBOOT})
- new net: AE1.1 (A), U2.11 (RF_IN)
- new net EXTINT: U2.5 (EXTINT)
- new net GND: AE1.2 (Shield), U2.1 (GND), U2.10 (GND), U2.12 (GND)
- new net RXD: U2.3 (RXD)
- new net SCL: U2.17 (SCL)
- new net SDA: U2.16 (SDA)
- new net TIMEPULSE: U2.4 (TIMEPULSE)
- new net TXD: U2.2 (TXD)
- new net VCC: U2.7 (VCC_IO), U2.8 (VCC)
- new net V_BCKP: U2.6 (V_BCKP)
- new net ~{RESET}: U2.9 (~{RESET})
- no-connect marks 0 -> 3
Changed lines of the file:
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@@
 (kicad_sch (version 20230121) (generator eeschema)
   (paper "A4")
+  (junction (at 109.22 71.12) (diameter 0) (color 0 0 0 0)
+  )
+  (no_connect (at 99.06 104.14))
+  (no_connect (at 119.38 73.66))
+  (no_connect (at 129.54 86.36))
+  (wire (pts (xy 93.98 96.52) (xy 99.06 96.52))
+    (stroke (width 0) (type default))
+  )
+  (wire (pts (xy 111.76 73.66) (xy 111.76 71.12))
+    (stroke (width 0) (type default))
+  )
+  (wire (pts (xy 114.3 68.58) (xy 114.3 73.66))
+    (stroke (width 0) (type default))
+  )
+  (wire (pts (xy 144.78 91.44) (xy 129.54 91.44))
+    (stroke (width 0) (type default))
+  )
+  (wire (pts (xy 88.9 99.06) (xy 99.06 99.06))
+    (stroke (width 0) (type default))
+  )
+  (wire (pts (xy 144.78 86.36) (xy 144.78 91.44))
+    (stroke (width 0) (type default))
+  )
+  (wire (pts (xy 93.98 91.44) (xy 99.06 91.44))
+    (stroke (width 0) (type default))
+  )
+  (wire (pts (xy 109.22 68.58) (xy 109.22 71.12))
+    (stroke (width 0) (type default))
+  )
+  (wire (pts (xy 147.32 86.36) (xy 147.32 88.9))
+    (stroke (width 0) (type default))
+  )
+  (wire (pts (xy 93.98 83.82) (xy 99.06 83.82))
+    (stroke (width 0) (type default))
+  )
+  (wire (pts (xy 93.98 88.9) (xy 99.06 88.9))
+    (stroke (width 0) (type default))
+  )
+  (wire (pts (xy 109.22 71.12) (xy 109.22 73.66))
+    (stroke (width 0) (type default))
+  )
+  (wire (pts (xy 93.98 101.6) (xy 99.06 101.6))
+    (stroke (width 0) (type default))
+  )
+  (wire (pts (xy 111.76 71.12) (xy 109.22 71.12))
+    (stroke (width 0) (type default))
+  )
+  (wire (pts (xy 93.98 81.28) (xy 99.06 81.28))
+    (stroke (width 0) (type default))
+  )
+  (hierarchical_label "TXD" (shape output) (at 93.98 83.82 180) (fields_autoplaced)
+    (effects (font (size 1.27 1.27)) (justify right))
+  )
+  (hierarchical_label "VCC" (shape passive) (at 109.22 68.58 90) (fields_autoplaced)
+    (effects (font (size 1.27 1.27)) (justify left))
+  )
+  (hierarchical_label "V_BCKP" (shape passive) (at 114.3 68.58 90) (fields_autoplaced)
+    (effects (font (size 1.27 1.27)) (justify left))
+  )
+  (hierarchical_label "RXD" (shape input) (at 93.98 81.28 180) (fields_autoplaced)
+    (effects (font (size 1.27 1.27)) (justify right))
+  )
+  (hierarchical_label "TIMEPULSE" (shape output) (at 129.54 99.06 0) (fields_autoplaced)
+    (effects (font (size 1.27 1.27)) (justify left))
+  )
+  (hierarchical_label "~{RESET}" (shape input) (at 93.98 101.6 180) (fields_autoplaced)
+    (effects (font (size 1.27 1.27)) (justify right))
+  )
+  (hierarchical_label "SDA" (shape bidirectional) (at 93.98 88.9 180) (fields_autoplaced)
+    (effects (font (size 1.27 1.27)) (justify right))
+  )
+  (hierarchical_label "SCL" (shape bidirectional) (at 93.98 91.44 180) (fields_autoplaced)
+    (effects (font (size 1.27 1.27)) (justify right))
+  )
+  (hierarchical_label "EXTINT" (shape bidirectional) (at 93.98 96.52 180) (fields_autoplaced)
+    (effects (font (size 1.27 1.27)) (justify right))
+  )
+  (symbol (lib_id "power:GND") (at 147.32 88.9 0) (unit 1)
+    (in_bom yes) (on_board yes) (dnp no) (fields_autoplaced)
+    (property "Reference" "#PWR05" (at 147.32 95.25 0)
+      (effects (font (size 1.27 1.27)) hide)
+    )
+    (property "Value" "GND" (at 147.32 93.98 0)
+      (effects (font (size 1.27 1.27)))
+    )
+    (property "Footprint" "" (at 147.32 88.9 0)
+      (effects (font (size 1.27 1.27)) hide)
+    )
+    (property "Datasheet" "" (at 147.32 88.9 0)
+      (effects (font (size 1.27 1.27)) hide)
+    )
+    (pin "1")
+    (instances
+      (project "Avionus_Flight_Controller"
+        (path "/ddc7e940-0588-4587-8902-8ced9e615ace/3a158364-4219-4eb3-b5df-68fe4e695c96"
+          (reference "#PWR05") (unit 1)
+        )
+      )
+    )
+  )
+  (symbol (lib_id "Connector:TestPoint") (at 88.9 99.06 90) (mirror x) (unit 1)
+    (in_bom yes) (on_board yes) (dnp no) (fields_autoplaced)
+    (property "Reference" "TP1" (at 83.82 97.79 90)
+      (effects (font (size 1.27 1.27)) (justify left))
+    )
+    (property "Value" "~{SAFEBOOT}" (at 83.82 100.33 90)
+      (effects (font (size 1.27 1.27)) (justify left))
+    )
+    (property "Footprint" "" (at 88.9 104.14 0)
+      (effects (font (size 1.27 1.27)) hide)
+    )
+    (property "Datasheet" "~" (at 88.9 104.14 0)
+      (effects (font (size 1.27 1.27)) hide)
+    )
+    (pin "1")
+    (instances
+      (project "Avionus_Flight_Controller"
+        (path "/ddc7e940-0588-4587-8902-8ced9e615ace/3a158364-4219-4eb3-b5df-68fe4e695c96"
+          (reference "TP1") (unit 1)
+        )
+        (path "/ddc7e940-0588-4587-8902-8ced9e615ace"
+          (reference "TP1") (unit 1)
+        )
+      )
+    )
+  )
+  (symbol (lib_id "power:GND") (at 114.3 109.22 0) (unit 1)
+    (in_bom yes) (on_board yes) (dnp no) (fields_autoplaced)
+    (property "Reference" "#PWR03" (at 114.3 115.57 0)
+      (effects (font (size 1.27 1.27)) hide)
+    )
+    (property "Value" "GND" (at 114.3 114.3 0)
+      (effects (font (size 1.27 1.27)))
+    )
+    (property "Footprint" "" (at 114.3 109.22 0)
+      (effects (font (size 1.27 1.27)) hide)
+    )
+    (property "Datasheet" "" (at 114.3 109.22 0)
+      (effects (font (size 1.27 1.27)) hide)
+    )
+    (pin "1")
+    (instances
+      (project "Avionus_Flight_Controller"
+        (path "/ddc7e940-0588-4587-8902-8ced9e615ace/3a158364-4219-4eb3-b5df-68fe4e695c96"
+          (reference "#PWR03") (unit 1)
+        )
+      )
+    )
+  )
+  (symbol (lib_id "RF_GPS:MAX-M10S") (at 114.3 91.44 0) (unit 1)
+    (in_bom yes) (on_board yes) (dnp no) (fields_autoplaced)
+    (property "Reference" "U2" (at 116.2559 109.22 0)
+      (effects (font (size 1.27 1.27)) (justify left))
+    )
+    (property "Value" "MAX-M10S" (at 116.2559 111.76 0)
+      (effects (font (size 1.27 1.27)) (justify left))
+    )
+    (property "Footprint" "RF_GPS:ublox_MAX" (at 124.46 107.95 0)
+      (effects (font (size 1.27 1.27)) hide)
+    )
+    (property "Datasheet" "https://content.u-blox.com/sites/default/files/MAX-M10S_DataSheet_UBX-20035208.pdf" (at 114.3 91.44 0)
+      (effects (font (size 1.27 1.27)) hide)
+    )
+    (pin "1")
+    (pin "10")
+    (pin "11")
+    (pin "12")
+    (pin "13")
+    (pin "14")
+    (pin "15")
+    (pin "16")
+    (pin "17")
+    (pin "18")
+    (pin "2")
+    (pin "3")
+    (pin "4")
+    (pin "5")
+    (pin "6")
+    (pin "7")
+    (pin "8")
+    (pin "9")
+    (instances
+      (project "Avionus_Flight_Controller"
+        (path "/ddc7e940-0588-4587-8902-8ced9e615ace/3a158364-4219-4eb3-b5df-68fe4e695c96"
+          (reference "U2") (unit 1)
+        )
+      )
+    )
+  )
+  (symbol (lib_id "Device:Antenna_Shield") (at 144.78 81.28 0) (unit 1)
+    (in_bom yes) (on_board yes) (dnp no) (fields_autoplaced)
+    (property "Reference" "AE1" (at 148.59 79.375 0)
+      (effects (font (size 1.27 1.27)) (justify left))
+    )
+    (property "Value" "GPS antenna" (at 148.59 81.915 0)
+      (effects (font (size 1.27 1.27)) (justify left))
+    )
+    (property "Footprint" "" (at 144.78 78.74 0)
+      (effects (font (size 1.27 1.27)) hide)
+    )
+    (property "Datasheet" "~" (at 144.78 78.74 0)
+      (effects (font (size 1.27 1.27)) hide)
+    )
+    (pin "1")
+    (pin "2")
+    (instances
+      (project "Avionus_Flight_Controller"
+        (path "/ddc7e940-0588-4587-8902-8ced9e615ace/3a158364-4219-4eb3-b5df-68fe4e695c96"
+          (reference "AE1") (unit 1)
+        )
+      )
+    )
+  )
 )

Commit message: Checkpoint
Parts:
- added C24, C52: ~, symbol Device:C_Small
- added L1: ~, symbol Device:L_Small
- added R43: ~, symbol Device:R_Small
- AE1: value GPS antenna -> SR4G080
Connections:
- net GND: now also C24.2, C52.1
- net at AE1.1 (A): now also C24.1, L1.1; no longer U2.11 (RF_IN)
- new net: C52.2, L1.2, R43.1
- new net: R43.2, U2.11 (RF_IN)
Changed lines of the file:
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@@
 (kicad_sch (version 20230121) (generator eeschema)
   (paper "A4")
+  (junction (at 144.78 81.28) (diameter 0) (color 0 0 0 0)
+  )
+  (junction (at 144.78 71.12) (diameter 0) (color 0 0 0 0)
+  )
   (junction (at 109.22 71.12) (diameter 0) (color 0 0 0 0)
   )
@@
   (no_connect (at 119.38 73.66))
   (no_connect (at 129.54 86.36))
+  (wire (pts (xy 147.32 71.12) (xy 144.78 71.12))
+    (stroke (width 0) (type default))
+  )
   (wire (pts (xy 93.98 96.52) (xy 99.06 96.52))
     (stroke (width 0) (type default))
@@
     (stroke (width 0) (type default))
   )
-  (wire (pts (xy 144.78 86.36) (xy 144.78 91.44))
+  (wire (pts (xy 144.78 81.28) (xy 147.32 81.28))
+    (stroke (width 0) (type default))
+  )
+  (wire (pts (xy 144.78 71.12) (xy 144.78 73.66))
+    (stroke (width 0) (type default))
+  )
+  (wire (pts (xy 144.78 81.28) (xy 144.78 83.82))
+    (stroke (width 0) (type default))
+  )
+  (wire (pts (xy 144.78 58.42) (xy 144.78 71.12))
+    (stroke (width 0) (type default))
+  )
+  (wire (pts (xy 144.78 78.74) (xy 144.78 81.28))
     (stroke (width 0) (type default))
   )
@@
     (stroke (width 0) (type default))
   )
-  (wire (pts (xy 147.32 86.36) (xy 147.32 88.9))
+  (wire (pts (xy 144.78 88.9) (xy 144.78 91.44))
     (stroke (width 0) (type default))
   )
@@
     (effects (font (size 1.27 1.27)) (justify right))
   )
-  (symbol (lib_id "power:GND") (at 147.32 88.9 0) (unit 1)
-    (in_bom yes) (on_board yes) (dnp no) (fields_autoplaced)
-    (property "Reference" "#PWR05" (at 147.32 95.25 0)
-      (effects (font (size 1.27 1.27)) hide)
-    )
-    (property "Value" "GND" (at 147.32 93.98 0)
+  (netclass_flag "" (length 2.54) (shape round) (at 144.78 71.12 90) (fields_autoplaced)
+    (effects (font (size 1.27 1.27)) (justify left bottom))
+    (property "Netclass" "GPS_RF" (at 142.24 70.4215 90)
+      (effects (font (size 1.27 1.27) italic) (justify left))
+    )
+  )
+  (netclass_flag "" (length 2.54) (shape round) (at 144.78 81.28 90) (fields_autoplaced)
+    (effects (font (size 1.27 1.27)) (justify left bottom))
+    (property "Netclass" "GPS_RF" (at 142.24 80.5815 90)
+      (effects (font (size 1.27 1.27) italic) (justify left))
+    )
+  )
+  (netclass_flag "" (length 2.54) (shape round) (at 134.62 91.44 0) (fields_autoplaced)
+    (effects (font (size 1.27 1.27)) (justify left bottom))
+    (property "Netclass" "GPS_RF" (at 135.3185 88.9 0)
+      (effects (font (size 1.27 1.27) italic) (justify left))
+    )
+  )
+  (symbol (lib_id "power:GND") (at 147.32 58.42 0) (unit 1)
+    (in_bom yes) (on_board yes) (dnp no) (fields_autoplaced)
+    (property "Reference" "#PWR05" (at 147.32 64.77 0)
+      (effects (font (size 1.27 1.27)) hide)
+    )
+    (property "Value" "GND" (at 147.32 63.5 0)
       (effects (font (size 1.27 1.27)))
     )
-    (property "Footprint" "" (at 147.32 88.9 0)
-      (effects (font (size 1.27 1.27)) hide)
-    )
-    (property "Datasheet" "" (at 147.32 88.9 0)
+    (property "Footprint" "" (at 147.32 58.42 0)
+      (effects (font (size 1.27 1.27)) hide)
+    )
+    (property "Datasheet" "" (at 147.32 58.42 0)
       (effects (font (size 1.27 1.27)) hide)
     )
@@
         (path "/ddc7e940-0588-4587-8902-8ced9e615ace/3a158364-4219-4eb3-b5df-68fe4e695c96"
           (reference "#PWR05") (unit 1)
+        )
+      )
+    )
+  )
+  (symbol (lib_id "Device:L_Small") (at 144.78 76.2 0) (unit 1)
+    (in_bom yes) (on_board yes) (dnp no)
+    (property "Reference" "L1" (at 146.05 76.2 0)
+      (effects (font (size 1.27 1.27)) (justify left))
+    )
+    (property "Value" "~" (at 146.05 77.47 0)
+      (effects (font (size 1.27 1.27)) (justify left))
+    )
+    (property "Footprint" "" (at 144.78 76.2 0)
+      (effects (font (size 1.27 1.27)) hide)
+    )
+    (property "Datasheet" "~" (at 144.78 76.2 0)
+      (effects (font (size 1.27 1.27)) hide)
+    )
+    (pin "1")
+    (pin "2")
+    (instances
+      (project "Avionus_Flight_Controller"
+        (path "/ddc7e940-0588-4587-8902-8ced9e615ace/3a158364-4219-4eb3-b5df-68fe4e695c96"
+          (reference "L1") (unit 1)
+        )
+      )
+    )
+  )
+  (symbol (lib_id "Device:C_Small") (at 149.86 81.28 270) (unit 1)
+    (in_bom yes) (on_board yes) (dnp no) (fields_autoplaced)
+    (property "Reference" "C52" (at 149.8536 77.47 90)
+      (effects (font (size 1.27 1.27)))
+    )
+    (property "Value" "~" (at 148.5837 83.6148 0)
+      (effects (font (size 1.27 1.27)) (justify left))
+    )
+    (property "Footprint" "" (at 149.86 81.28 0)
+      (effects (font (size 1.27 1.27)) hide)
+    )
+    (property "Datasheet" "~" (at 149.86 81.28 0)
+      (effects (font (size 1.27 1.27)) hide)
+    )
+    (pin "1")
+    (pin "2")
+    (instances
+      (project "Avionus_Flight_Controller"
+        (path "/ddc7e940-0588-4587-8902-8ced9e615ace/3a158364-4219-4eb3-b5df-68fe4e695c96"
+          (reference "C52") (unit 1)
+        )
+      )
+    )
+  )
+  (symbol (lib_id "power:GND") (at 152.4 71.12 90) (unit 1)
+    (in_bom yes) (on_board yes) (dnp no) (fields_autoplaced)
+    (property "Reference" "#PWR057" (at 158.75 71.12 0)
+      (effects (font (size 1.27 1.27)) hide)
+    )
+    (property "Value" "GND" (at 156.21 71.12 90)
+      (effects (font (size 1.27 1.27)) (justify right))
+    )
+    (property "Footprint" "" (at 152.4 71.12 0)
+      (effects (font (size 1.27 1.27)) hide)
+    )
+    (property "Datasheet" "" (at 152.4 71.12 0)
+      (effects (font (size 1.27 1.27)) hide)
+    )
+    (pin "1")
+    (instances
+      (project "Avionus_Flight_Controller"
+        (path "/ddc7e940-0588-4587-8902-8ced9e615ace/3a158364-4219-4eb3-b5df-68fe4e695c96"
+          (reference "#PWR057") (unit 1)
         )
       )
@@
         (path "/ddc7e940-0588-4587-8902-8ced9e615ace/3a158364-4219-4eb3-b5df-68fe4e695c96"
           (reference "#PWR03") (unit 1)
+        )
+      )
+    )
+  )
+  (symbol (lib_id "Device:C_Small") (at 149.86 71.12 90) (unit 1)
+    (in_bom yes) (on_board yes) (dnp no) (fields_autoplaced)
+    (property "Reference" "C24" (at 149.8663 67.31 90)
+      (effects (font (size 1.27 1.27)))
+    )
+    (property "Value" "~" (at 151.1363 68.7852 0)
+      (effects (font (size 1.27 1.27)) (justify left))
+    )
+    (property "Footprint" "" (at 149.86 71.12 0)
+      (effects (font (size 1.27 1.27)) hide)
+    )
+    (property "Datasheet" "~" (at 149.86 71.12 0)
+      (effects (font (size 1.27 1.27)) hide)
+    )
+    (pin "1")
+    (pin "2")
+    (instances
+      (project "Avionus_Flight_Controller"
+        (path "/ddc7e940-0588-4587-8902-8ced9e615ace/3a158364-4219-4eb3-b5df-68fe4e695c96"
+          (reference "C24") (unit 1)
+        )
+      )
+    )
+  )
+  (symbol (lib_id "Device:R_Small") (at 144.78 86.36 0) (unit 1)
+    (in_bom yes) (on_board yes) (dnp no)
+    (property "Reference" "R43" (at 147.32 86.36 0)
+      (effects (font (size 1.27 1.27)) (justify left))
+    )
+    (property "Value" "~" (at 147.32 87.63 0)
+      (effects (font (size 1.27 1.27)) (justify left))
+    )
+    (property "Footprint" "" (at 144.78 86.36 0)
+      (effects (font (size 1.27 1.27)) hide)
+    )
+    (property "Datasheet" "~" (at 144.78 86.36 0)
+      (effects (font (size 1.27 1.27)) hide)
+    )
+    (pin "1")
+    (pin "2")
+    (instances
+      (project "Avionus_Flight_Controller"
+        (path "/ddc7e940-0588-4587-8902-8ced9e615ace/3a158364-4219-4eb3-b5df-68fe4e695c96"
+          (reference "R43") (unit 1)
         )
       )
@@
     )
   )
-  (symbol (lib_id "Device:Antenna_Shield") (at 144.78 81.28 0) (unit 1)
-    (in_bom yes) (on_board yes) (dnp no) (fields_autoplaced)
-    (property "Reference" "AE1" (at 148.59 79.375 0)
-      (effects (font (size 1.27 1.27)) (justify left))
-    )
-    (property "Value" "GPS antenna" (at 148.59 81.915 0)
-      (effects (font (size 1.27 1.27)) (justify left))
-    )
-    (property "Footprint" "" (at 144.78 78.74 0)
-      (effects (font (size 1.27 1.27)) hide)
-    )
-    (property "Datasheet" "~" (at 144.78 78.74 0)
-      (effects (font (size 1.27 1.27)) hide)
-    )
+  (symbol (lib_id "power:GND") (at 152.4 81.28 90) (unit 1)
+    (in_bom yes) (on_board yes) (dnp no) (fields_autoplaced)
+    (property "Reference" "#PWR058" (at 158.75 81.28 0)
+      (effects (font (size 1.27 1.27)) hide)
+    )
+    (property "Value" "GND" (at 156.21 81.28 90)
+      (effects (font (size 1.27 1.27)) (justify right))
+    )
+    (property "Footprint" "" (at 152.4 81.28 0)
+      (effects (font (size 1.27 1.27)) hide)
+    )
+    (property "Datasheet" "" (at 152.4 81.28 0)
+      (effects (font (size 1.27 1.27)) hide)
+    )
+    (pin "1")
+    (instances
+      (project "Avionus_Flight_Controller"
+        (path "/ddc7e940-0588-4587-8902-8ced9e615ace/3a158364-4219-4eb3-b5df-68fe4e695c96"
+          (reference "#PWR058") (unit 1)
+        )
+      )
+    )
+  )
+  (symbol (lib_id "Device:Antenna_Shield") (at 144.78 53.34 0) (unit 1)
+    (in_bom yes) (on_board yes) (dnp no) (fields_autoplaced)
+    (property "Reference" "AE1" (at 148.59 51.435 0)
+      (effects (font (size 1.27 1.27)) (justify left))
+    )
+    (property "Value" "SR4G080" (at 148.59 53.975 0)
+      (effects (font (size 1.27 1.27)) (justify left))
+    )
+    (property "Footprint" "" (at 144.78 50.8 0)
+      (effects (font (size 1.27 1.27)) hide)
+    )
+    (property "Datasheet" "~" (at 144.78 50.8 0)
+      (effects (font (size 1.27 1.27)) hide)
+    )
