File: Hardware/GPS.kicad_sch (KiCad schematic)
At the start: 7 parts, among them U2 MAX-M10S

Commit message: Checkpoint
Parts:
- renumbered AE1 to AE1001, C24 to C1001, C52 to C1002, L1 to L1001, R43 to R1001, TP1 to TP1001, U2 to U1001
Changed lines of the file:
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@@
   (symbol (lib_id "power:GND") (at 147.32 58.42 0) (unit 1)
     (in_bom yes) (on_board yes) (dnp no) (fields_autoplaced)
-    (property "Reference" "#PWR05" (at 147.32 64.77 0)
+    (property "Reference" "#PWR01002" (at 147.32 64.77 0)
       (effects (font (size 1.27 1.27)) hide)
     )
@@
       (project "Avionus_Flight_Controller"
         (path "/ddc7e940-0588-4587-8902-8ced9e615ace/3a158364-4219-4eb3-b5df-68fe4e695c96"
-          (reference "#PWR05") (unit 1)
+          (reference "#PWR01002") (unit 1)
         )
       )
@@
   (symbol (lib_id "Device:L_Small") (at 144.78 76.2 0) (unit 1)
     (in_bom yes) (on_board yes) (dnp no)
-    (property "Reference" "L1" (at 146.05 76.2 0)
+    (property "Reference" "L1001" (at 146.05 76.2 0)
       (effects (font (size 1.27 1.27)) (justify left))
     )
@@
       (project "Avionus_Flight_Controller"
         (path "/ddc7e940-0588-4587-8902-8ced9e615ace/3a158364-4219-4eb3-b5df-68fe4e695c96"
-          (reference "L1") (unit 1)
+          (reference "L1001") (unit 1)
         )
       )
@@
   (symbol (lib_id "Device:C_Small") (at 149.86 81.28 270) (unit 1)
     (in_bom yes) (on_board yes) (dnp no) (fields_autoplaced)
-    (property "Reference" "C52" (at 149.8536 77.47 90)
+    (property "Reference" "C1002" (at 149.8536 77.47 90)
       (effects (font (size 1.27 1.27)))
     )
@@
       (project "Avionus_Flight_Controller"
         (path "/ddc7e940-0588-4587-8902-8ced9e615ace/3a158364-4219-4eb3-b5df-68fe4e695c96"
-          (reference "C52") (unit 1)
+          (reference "C1002") (unit 1)
         )
       )
@@
   (symbol (lib_id "power:GND") (at 152.4 71.12 90) (unit 1)
     (in_bom yes) (on_board yes) (dnp no) (fields_autoplaced)
-    (property "Reference" "#PWR057" (at 158.75 71.12 0)
+    (property "Reference" "#PWR01003" (at 158.75 71.12 0)
       (effects (font (size 1.27 1.27)) hide)
     )
@@
       (project "Avionus_Flight_Controller"
         (path "/ddc7e940-0588-4587-8902-8ced9e615ace/3a158364-4219-4eb3-b5df-68fe4e695c96"
-          (reference "#PWR057") (unit 1)
+          (reference "#PWR01003") (unit 1)
         )
       )
@@
   (symbol (lib_id "Connector:TestPoint") (at 88.9 99.06 90) (mirror x) (unit 1)
     (in_bom yes) (on_board yes) (dnp no) (fields_autoplaced)
-    (property "Reference" "TP1" (at 83.82 97.79 90)
+    (property "Reference" "TP1001" (at 83.82 97.79 90)
       (effects (font (size 1.27 1.27)) (justify left))
     )
@@
       (project "Avionus_Flight_Controller"
         (path "/ddc7e940-0588-4587-8902-8ced9e615ace/3a158364-4219-4eb3-b5df-68fe4e695c96"
-          (reference "TP1") (unit 1)
+          (reference "TP1001") (unit 1)
         )
         (path "/ddc7e940-0588-4587-8902-8ced9e615ace"
-          (reference "TP1") (unit 1)
+          (reference "TP?") (unit 1)
         )
       )
@@
   (symbol (lib_id "power:GND") (at 114.3 109.22 0) (unit 1)
     (in_bom yes) (on_board yes) (dnp no) (fields_autoplaced)
-    (property "Reference" "#PWR03" (at 114.3 115.57 0)
+    (property "Reference" "#PWR01001" (at 114.3 115.57 0)
       (effects (font (size 1.27 1.27)) hide)
     )
@@
       (project "Avionus_Flight_Controller"
         (path "/ddc7e940-0588-4587-8902-8ced9e615ace/3a158364-4219-4eb3-b5df-68fe4e695c96"
-          (reference "#PWR03") (unit 1)
+          (reference "#PWR01001") (unit 1)
         )
       )
@@
   (symbol (lib_id "Device:C_Small") (at 149.86 71.12 90) (unit 1)
     (in_bom yes) (on_board yes) (dnp no) (fields_autoplaced)
-    (property "Reference" "C24" (at 149.8663 67.31 90)
+    (property "Reference" "C1001" (at 149.8663 67.31 90)
       (effects (font (size 1.27 1.27)))
     )
@@
       (project "Avionus_Flight_Controller"
         (path "/ddc7e940-0588-4587-8902-8ced9e615ace/3a158364-4219-4eb3-b5df-68fe4e695c96"
-          (reference "C24") (unit 1)
+          (reference "C1001") (unit 1)
         )
       )
@@
   (symbol (lib_id "Device:R_Small") (at 144.78 86.36 0) (unit 1)
     (in_bom yes) (on_board yes) (dnp no)
-    (property "Reference" "R43" (at 147.32 86.36 0)
+    (property "Reference" "R1001" (at 147.32 86.36 0)
       (effects (font (size 1.27 1.27)) (justify left))
     )
@@
       (project "Avionus_Flight_Controller"
         (path "/ddc7e940-0588-4587-8902-8ced9e615ace/3a158364-4219-4eb3-b5df-68fe4e695c96"
-          (reference "R43") (unit 1)
+          (reference "R1001") (unit 1)
         )
       )
@@
   (symbol (lib_id "RF_GPS:MAX-M10S") (at 114.3 91.44 0) (unit 1)
     (in_bom yes) (on_board yes) (dnp no) (fields_autoplaced)
-    (property "Reference" "U2" (at 116.2559 109.22 0)
+    (property "Reference" "U1001" (at 116.2559 109.22 0)
       (effects (font (size 1.27 1.27)) (justify left))
     )
@@
       (project "Avionus_Flight_Controller"
         (path "/ddc7e940-0588-4587-8902-8ced9e615ace/3a158364-4219-4eb3-b5df-68fe4e695c96"
-          (reference "U2") (unit 1)
+          (reference "U1001") (unit 1)
         )
       )
@@
   (symbol (lib_id "power:GND") (at 152.4 81.28 90) (unit 1)
     (in_bom yes) (on_board yes) (dnp no) (fields_autoplaced)
-    (property "Reference" "#PWR058" (at 158.75 81.28 0)
+    (property "Reference" "#PWR01004" (at 158.75 81.28 0)
       (effects (font (size 1.27 1.27)) hide)
     )
@@
       (project "Avionus_Flight_Controller"
         (path "/ddc7e940-0588-4587-8902-8ced9e615ace/3a158364-4219-4eb3-b5df-68fe4e695c96"
-          (reference "#PWR058") (unit 1)
+          (reference "#PWR01004") (unit 1)
         )
       )
@@
   (symbol (lib_id "Device:Antenna_Shield") (at 144.78 53.34 0) (unit 1)
     (in_bom yes) (on_board yes) (dnp no) (fields_autoplaced)
-    (property "Reference" "AE1" (at 148.59 51.435 0)
+    (property "Reference" "AE1001" (at 148.59 51.435 0)
       (effects (font (size 1.27 1.27)) (justify left))
     )
@@
       (project "Avionus_Flight_Controller"
         (path "/ddc7e940-0588-4587-8902-8ced9e615ace/3a158364-4219-4eb3-b5df-68fe4e695c96"
-          (reference "AE1") (unit 1)
-        )
-      )
+          (reference "AE1001") (unit 1)
+        )
+      )

Commit message: Checkpoint
Parts:
- renumbered C1002 to C1001, C1001 to C1002
Connections:
- net at AE1001.1 (A), C1002.1: now also L1001.2; no longer L1001.1
- net at C1001.2, R1001.1: now also L1001.1; no longer L1001.2
Other:
- moved on the sheet: AE1001, C1001, C1002, L1001, R1001

Commit message: Checkpoint
Parts:
- TP1001: value ~{SAFEBOOT} -> ~; footprint (none) -> TestPoint:TestPoint_Pad_D2.0mm
Changed lines of the file:
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@@
   (symbol (lib_id "Connector:TestPoint") (at 88.9 99.06 90) (mirror x) (unit 1)
     (in_bom yes) (on_board yes) (dnp no) (fields_autoplaced)
-    (property "Reference" "TP1001" (at 83.82 97.79 90)
+    (property "Reference" "TP1001" (at 83.82 99.06 90)
       (effects (font (size 1.27 1.27)) (justify left))
     )
-    (property "Value" "~{SAFEBOOT}" (at 83.82 100.33 90)
+    (property "Value" "~" (at 83.82 100.33 90)
       (effects (font (size 1.27 1.27)) (justify left))
     )
-    (property "Footprint" "" (at 88.9 104.14 0)
+    (property "Footprint" "TestPoint:TestPoint_Pad_D2.0mm" (at 88.9 104.14 0)
       (effects (font (size 1.27 1.27)) hide)
     )

Commit message: Checkpoint
Parts:
- AE1001: footprint (none) -> leptunKicadLib:SR4G080
- C1001: value ~ -> 4.3pF; footprint (none) -> Capacitor_SMD:C_0402_1005Metric_Pad0.74x0.62mm_HandSolder
- C1002: value ~ -> 3.6pF; footprint (none) -> Capacitor_SMD:C_0402_1005Metric_Pad0.74x0.62mm_HandSolder
- L1001: value ~ -> 5.1nH; footprint (none) -> Inductor_SMD:L_0402_1005Metric_Pad0.77x0.64mm_HandSolder
- R1001: value ~ -> 0R; footprint (none) -> Resistor_SMD:R_0402_1005Metric_Pad0.72x0.64mm_HandSolder
Changed lines of the file:
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@@
   (symbol (lib_id "Device:L_Small") (at 160.02 91.44 90) (unit 1)
     (in_bom yes) (on_board yes) (dnp no) (fields_autoplaced)
-    (property "Reference" "L1001" (at 160.02 88.9 90)
-      (effects (font (size 1.27 1.27)))
-    )
-    (property "Value" "~" (at 161.29 90.17 0)
-      (effects (font (size 1.27 1.27)) (justify left))
-    )
-    (property "Footprint" "" (at 160.02 91.44 0)
+    (property "Reference" "L1001" (at 160.02 86.36 90)
+      (effects (font (size 1.27 1.27)))
+    )
+    (property "Value" "5.1nH" (at 160.02 88.9 90)
+      (effects (font (size 1.27 1.27)))
+    )
+    (property "Footprint" "Inductor_SMD:L_0402_1005Metric_Pad0.77x0.64mm_HandSolder" (at 160.02 91.44 0)
       (effects (font (size 1.27 1.27)) hide)
     )
@@
   (symbol (lib_id "Device:C_Small") (at 152.4 96.52 180) (unit 1)
     (in_bom yes) (on_board yes) (dnp no) (fields_autoplaced)
-    (property "Reference" "C1001" (at 154.94 96.5136 0)
+    (property "Reference" "C1001" (at 154.94 95.2436 0)
       (effects (font (size 1.27 1.27)) (justify right))
     )
-    (property "Value" "~" (at 150.0652 95.2437 0)
-      (effects (font (size 1.27 1.27)) (justify left))
-    )
-    (property "Footprint" "" (at 152.4 96.52 0)
+    (property "Value" "4.3pF" (at 154.94 97.7836 0)
+      (effects (font (size 1.27 1.27)) (justify right))
+    )
+    (property "Footprint" "Capacitor_SMD:C_0402_1005Metric_Pad0.74x0.62mm_HandSolder" (at 152.4 96.52 0)
       (effects (font (size 1.27 1.27)) hide)
     )
@@
   (symbol (lib_id "Device:C_Small") (at 167.64 96.52 0) (unit 1)
     (in_bom yes) (on_board yes) (dnp no) (fields_autoplaced)
-    (property "Reference" "C1002" (at 170.18 96.5263 0)
-      (effects (font (size 1.27 1.27)) (justify left))
-    )
-    (property "Value" "~" (at 169.9748 97.7963 0)
-      (effects (font (size 1.27 1.27)) (justify left))
-    )
-    (property "Footprint" "" (at 167.64 96.52 0)
+    (property "Reference" "C1002" (at 170.18 95.2563 0)
+      (effects (font (size 1.27 1.27)) (justify left))
+    )
+    (property "Value" "3.6pF" (at 170.18 97.7963 0)
+      (effects (font (size 1.27 1.27)) (justify left))
+    )
+    (property "Footprint" "Capacitor_SMD:C_0402_1005Metric_Pad0.74x0.62mm_HandSolder" (at 167.64 96.52 0)
       (effects (font (size 1.27 1.27)) hide)
     )
@@
   (symbol (lib_id "Device:R_Small") (at 147.32 91.44 270) (unit 1)
     (in_bom yes) (on_board yes) (dnp no) (fields_autoplaced)
-    (property "Reference" "R1001" (at 147.32 88.9 90)
-      (effects (font (size 1.27 1.27)))
-    )
-    (property "Value" "~" (at 146.05 93.98 0)
-      (effects (font (size 1.27 1.27)) (justify left))
-    )
-    (property "Footprint" "" (at 147.32 91.44 0)
+    (property "Reference" "R1001" (at 147.32 86.36 90)
+      (effects (font (size 1.27 1.27)))
+    )
+    (property "Value" "0R" (at 147.32 88.9 90)
+      (effects (font (size 1.27 1.27)))
+    )
+    (property "Footprint" "Resistor_SMD:R_0402_1005Metric_Pad0.72x0.64mm_HandSolder" (at 147.32 91.44 0)
       (effects (font (size 1.27 1.27)) hide)
     )
@@
       (effects (font (size 1.27 1.27)) (justify left))
     )
-    (property "Footprint" "" (at 190.5 91.44 0)
-      (effects (font (size 1.27 1.27)) hide)
-    )
+    (property "Footprint" "leptunKicadLib:SR4G080" (at 190.5 91.44 0)
+      (effects (font (size 1.27 1.27)) hide)
+    )

Commit message: Checkpoint
Parts:
- TP1001: footprint TestPoint:TestPoint_Pad_D2.0mm -> TestPoint:TestPoint_Pad_D1.0mm
Changed lines of the file:
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@@
       (effects (font (size 1.27 1.27)) (justify left))
     )
-    (property "Footprint" "TestPoint:TestPoint_Pad_D2.0mm" (at 88.9 104.14 0)
+    (property "Footprint" "TestPoint:TestPoint_Pad_D1.0mm" (at 88.9 104.14 0)
       (effects (font (size 1.27 1.27)) hide)
     )

Commit message: Finalize silkscreen
Other:
- title: (none) -> Avionus_Flight_Controller
Changed lines of the file:
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@@
 (kicad_sch (version 20230121) (generator eeschema)
   (paper "A4")
+  (title_block
+    (title "Avionus_Flight_Controller")
+    (date "2023-11-25")
+    (rev "1.0")
+  )
   (junction (at 152.4 91.44) (diameter 0) (color 0 0 0 0)
   )
