File: Hardware/IMU.kicad_sch (KiCad schematic)
At the start: 19 parts, among them U1501 ICM-20948

Commit message: Finalize silkscreen
Other:
- title: (none) -> Avionus_Flight_Controller
Changed lines of the file:
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@@
 (kicad_sch (version 20230121) (generator eeschema)
   (paper "A4")
+  (title_block
+    (title "Avionus_Flight_Controller")
+    (date "2023-11-25")
+    (rev "1.0")
+  )
   (junction (at 50.8 134.62) (diameter 0) (color 0 0 0 0)
   )
