File: Hardware/LIDAR.kicad_sch (KiCad schematic)
At the start: 4 parts, among them J1401 LIDAR1, J1402 LIDAR2, U1401 USBLC6-4SC6, U801 USBLC6-2SC6

Commit message: Finalize silkscreen
Other:
- title: (none) -> Avionus_Flight_Controller
Changed lines of the file:
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@@
 (kicad_sch (version 20230121) (generator eeschema)
   (paper "A4")
+  (title_block
+    (title "Avionus_Flight_Controller")
+    (date "2023-11-25")
+    (rev "1.0")
+  )
   (wire (pts (xy 208.28 129.54) (xy 203.2 129.54))
     (stroke (width 0) (type default))
