File: Hardware/REMOTE.kicad_sch (KiCad schematic)
At the start: 0 parts

Commit message: Checkpoint
Changed lines of the file:
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@@
     (effects (font (size 1.27 1.27)) (justify left))
   )
-  (hierarchical_label "VCC" (shape passive) (at 101.6 53.34 0) (fields_autoplaced)
+  (hierarchical_label "VDD_5V" (shape passive) (at 101.6 53.34 0) (fields_autoplaced)
     (effects (font (size 1.27 1.27)) (justify left))
   )
+  (hierarchical_label "VDD_3V3" (shape passive) (at 101.6 50.8 0) (fields_autoplaced)
+    (effects (font (size 1.27 1.27)) (justify left))
+  )

Commit message: Checkpoint
Parts:
- added J?: PPM, Connector_PinHeader_2.54mm:PinHeader_1x03_P2.54mm_Horizontal, symbol Connector_Generic:Conn_01x03
- added J?: iBUS, Connector_PinHeader_2.54mm:PinHeader_1x03_P2.54mm_Horizontal, symbol Connector_Generic:Conn_01x03
- added Q? (x2): RE1C002UN, Package_TO_SOT_SMD:SOT-416, symbol Device:Q_NMOS_GSD
- added R? (x4): 2.2K, Resistor_SMD:R_0805_2012Metric, symbol Device:R_Small
Connections:
- net PPM: now also Q?.2 (S), R?.1
- net VDD_3V3: now also Q?.1 (G), Q?.1 (G), R?.2, R?.2
- net VDD_5V: now also J?.2 (Pin_2), J?.2 (Pin_2), R?.2, R?.2
- net iBUS: now also Q?.2 (S), R?.1
- new net: J?.3 (Pin_3), Q?.3 (D), R?.1 (x2)
- new net GND: J?.1 (Pin_1), J?.1 (Pin_1)

Commit message: Checkpoint
Parts:
- added U1101: USBLC6-4SC6, Package_TO_SOT_SMD:SOT-23-6, symbol Power_Protection:USBLC6-4SC6
Connections:
- net GND: now also U1101.2 (GND)
- net VDD_5V: now also U1101.5 (VBUS)
- net at J?.3 (Pin_3), Q?.3 (D), R?.1: now also U1101.1 (I/O1)
- net at J?.3 (Pin_3), Q?.3 (D), R?.1: now also U1101.3 (I/O2)
- no-connect marks 0 -> 2
Changed lines of the file:
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@@
   (junction (at 60.96 55.88) (diameter 0) (color 0 0 0 0)
   )
+  (junction (at 78.74 55.88) (diameter 0) (color 0 0 0 0)
+  )
   (junction (at 60.96 81.28) (diameter 0) (color 0 0 0 0)
   )
+  (junction (at 78.74 81.28) (diameter 0) (color 0 0 0 0)
+  )
   (junction (at 45.72 81.28) (diameter 0) (color 0 0 0 0)
   )
   (junction (at 45.72 55.88) (diameter 0) (color 0 0 0 0)
   )
+  (no_connect (at 127 63.5))
+  (no_connect (at 127 68.58))
   (wire (pts (xy 60.96 81.28) (xy 58.42 81.28))
     (stroke (width 0) (type default))
   )
-  (wire (pts (xy 60.96 55.88) (xy 88.9 55.88))
+  (wire (pts (xy 60.96 55.88) (xy 78.74 55.88))
     (stroke (width 0) (type default))
   )
@@
     (stroke (width 0) (type default))
   )
-  (wire (pts (xy 60.96 81.28) (xy 88.9 81.28))
+  (wire (pts (xy 60.96 81.28) (xy 78.74 81.28))
     (stroke (width 0) (type default))
   )
@@
     (stroke (width 0) (type default))
   )
+  (wire (pts (xy 78.74 68.58) (xy 78.74 81.28))
+    (stroke (width 0) (type default))
+  )
   (wire (pts (xy 43.18 68.58) (xy 60.96 68.58))
     (stroke (width 0) (type default))
@@
     (stroke (width 0) (type default))
   )
+  (wire (pts (xy 78.74 55.88) (xy 88.9 55.88))
+    (stroke (width 0) (type default))
+  )
   (wire (pts (xy 60.96 55.88) (xy 58.42 55.88))
     (stroke (width 0) (type default))
@@
     (stroke (width 0) (type default))
   )
+  (wire (pts (xy 78.74 55.88) (xy 78.74 63.5))
+    (stroke (width 0) (type default))
+  )
   (wire (pts (xy 53.34 71.12) (xy 45.72 71.12))
     (stroke (width 0) (type default))
   )
+  (wire (pts (xy 78.74 81.28) (xy 88.9 81.28))
+    (stroke (width 0) (type default))
+  )
+  (wire (pts (xy 106.68 68.58) (xy 78.74 68.58))
+    (stroke (width 0) (type default))
+  )
   (wire (pts (xy 53.34 73.66) (xy 53.34 71.12))
     (stroke (width 0) (type default))
@@
     (stroke (width 0) (type default))
   )
+  (wire (pts (xy 78.74 63.5) (xy 106.68 63.5))
+    (stroke (width 0) (type default))
+  )
   (hierarchical_label "VDD_5V" (shape passive) (at 88.9 53.34 180) (fields_autoplaced)
     (effects (font (size 1.27 1.27)) (justify right))
@@
     (effects (font (size 1.27 1.27)) (justify right))
   )
+  (hierarchical_label "VDD_5V" (shape passive) (at 116.84 55.88 90) (fields_autoplaced)
+    (effects (font (size 1.27 1.27)) (justify left))
+  )
   (hierarchical_label "PPM" (shape output) (at 43.18 55.88 180) (fields_autoplaced)
     (effects (font (size 1.27 1.27)) (justify right))
+  )
+  (symbol (lib_id "power:GND") (at 116.84 76.2 0) (unit 1)
+    (in_bom yes) (on_board yes) (dnp no) (fields_autoplaced)
+    (property "Reference" "#PWR01103" (at 116.84 82.55 0)
+      (effects (font (size 1.27 1.27)) hide)
+    )
+    (property "Value" "GND" (at 116.84 81.28 0)
+      (effects (font (size 1.27 1.27)))
+    )
+    (property "Footprint" "" (at 116.84 76.2 0)
+      (effects (font (size 1.27 1.27)) hide)
+    )
+    (property "Datasheet" "" (at 116.84 76.2 0)
+      (effects (font (size 1.27 1.27)) hide)
+    )
+    (pin "1")
+    (instances
+      (project "Avionus_Flight_Controller"
+        (path "/ddc7e940-0588-4587-8902-8ced9e615ace/e1d6da77-64eb-4d15-b8a2-13dabb15172d"
+          (reference "#PWR01103") (unit 1)
+        )
+      )
+    )
   )
   (symbol (lib_id "Device:R_Small") (at 45.72 73.66 180) (unit 1)
@@
         )
       )
+    )
+  )
+  (symbol (lib_id "Power_Protection:USBLC6-4SC6") (at 116.84 66.04 0) (unit 1)
+    (in_bom yes) (on_board yes) (dnp no) (fields_autoplaced)
+    (property "Reference" "U1101" (at 118.4911 53.34 0)
+      (effects (font (size 1.27 1.27)) (justify left))
+    )
+    (property "Value" "USBLC6-4SC6" (at 118.4911 55.88 0)
+      (effects (font (size 1.27 1.27)) (justify left))
+    )
+    (property "Footprint" "Package_TO_SOT_SMD:SOT-23-6" (at 116.84 78.74 0)
+      (effects (font (size 1.27 1.27)) hide)
+    )
+    (property "Datasheet" "https://www.st.com/resource/en/datasheet/usblc6-4.pdf" (at 121.92 57.15 0)
+      (effects (font (size 1.27 1.27)) hide)
+    )
+    (pin "1")
+    (pin "2")
+    (pin "3")
+    (pin "4")
+    (pin "5")
+    (pin "6")
+    (instances
+      (project "Avionus_Flight_Controller"
+        (path "/ddc7e940-0588-4587-8902-8ced9e615ace/e1d6da77-64eb-4d15-b8a2-13dabb15172d"
+          (reference "U1101") (unit 1)
+        )
+      )

Commit message: Finalize silkscreen
Other:
- title: (none) -> Avionus_Flight_Controller
Changed lines of the file:
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@@
 (kicad_sch (version 20230121) (generator eeschema)
   (paper "A4")
+  (title_block
+    (title "Avionus_Flight_Controller")
+    (date "2023-11-25")
+    (rev "1.0")
+  )
   (junction (at 45.72 45.72) (diameter 0) (color 0 0 0 0)
   )
