File: Hardware/RF.kicad_sch (KiCad schematic)
At the start: 2 parts, among them U901 LAMBDA62

Commit message: Finalize silkscreen
Other:
- title: (none) -> Avionus_Flight_Controller
Changed lines of the file:
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@@
 (kicad_sch (version 20230121) (generator eeschema)
   (paper "A4")
+  (title_block
+    (title "Avionus_Flight_Controller")
+    (date "2023-11-25")
+    (rev "1.0")
+  )
   (wire (pts (xy 162.56 83.82) (xy 175.26 83.82))
     (stroke (width 0) (type default))
